File: VDJoulemeter/HighPowerJoulemeter/HighPowerJoulemeter.kicad_sch (KiCad schematic)
At the start: 45 parts, among them J1 XT60-M, J2 XT60-M, J3 22035035, J4 22035035, U2 TMCS1107A1BQDR, U3 MCP2551-E/P, U5 MCP6286T-E/OT, U6 PTPSM365R6FRDN, U8 ADS1118QDGSRQ1, U9 MIC5219-3.3YM5-TR

Commit message: 9/24 feedback stuff
Connections:
- net MISO is gone; now on net STM_MISO: U1.51 (PA6)
- net MOSI is gone; now on net STM_MOSI: U1.53 (PA7)
- no-connect marks 0 -> 58
Changed lines of the file:
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@@
 	(text "Leaving these unnconnected because only two things being measured"
 		(exclude_from_sim no)
-		(at 166.116 197.104 0)
+		(at 176.784 197.104 0)
 		(effects
 			(font
@@
 		(color 0 0 0 0)
 	)
+	(no_connect
+		(at 340.36 199.39)
+	)
+	(no_connect
+		(at 340.36 194.31)
+	)
+	(no_connect
+		(at 381 173.99)
+	)
+	(no_connect
+		(at 381 148.59)
+	)
+	(no_connect
+		(at 340.36 110.49)
+	)
+	(no_connect
+		(at 381 191.77)
+	)
+	(no_connect
+		(at 381 120.65)
+	)
+	(no_connect
+		(at 340.36 118.11)
+	)
+	(no_connect
+		(at 340.36 153.67)
+	)
+	(no_connect
+		(at 340.36 115.57)
+	)
+	(no_connect
+		(at 381 168.91)
+	)
+	(no_connect
+		(at 381 156.21)
+	)
+	(no_connect
+		(at 340.36 143.51)
+	)
+	(no_connect
+		(at 340.36 168.91)
+	)
+	(no_connect
+		(at 381 176.53)
+	)
+	(no_connect
+		(at 340.36 166.37)
+	)
+	(no_connect
+		(at 381 194.31)
+	)
+	(no_connect
+		(at 381 179.07)
+	)
+	(no_connect
+		(at 340.36 151.13)
+	)
+	(no_connect
+		(at 340.36 181.61)
+	)
+	(no_connect
+		(at 381 196.85)
+	)
+	(no_connect
+		(at 340.36 186.69)
+	)
+	(no_connect
+		(at 245.11 68.58)
+	)
+	(no_connect
+		(at 153.67 198.12)
+	)
+	(no_connect
+		(at 381 128.27)
+	)
+	(no_connect
+		(at 340.36 191.77)
+	)
+	(no_connect
+		(at 245.11 66.04)
+	)
+	(no_connect
+		(at 381 110.49)
+	)
+	(no_connect
+		(at 245.11 60.96)
+	)
+	(no_connect
+		(at 340.36 125.73)
+	)
+	(no_connect
+		(at 340.36 161.29)
+	)
+	(no_connect
+		(at 340.36 138.43)
+	)
+	(no_connect
+		(at 340.36 123.19)
+	)
+	(no_connect
+		(at 381 181.61)
+	)
+	(no_connect
+		(at 340.36 179.07)
+	)
+	(no_connect
+		(at 381 163.83)
+	)
+	(no_connect
+		(at 381 186.69)
+	)
+	(no_connect
+		(at 340.36 146.05)
+	)
+	(no_connect
+		(at 381 123.19)
+	)
+	(no_connect
+		(at 381 171.45)
+	)
+	(no_connect
+		(at 381 201.93)
+	)
+	(no_connect
+		(at 340.36 184.15)
+	)
+	(no_connect
+		(at 340.36 204.47)
+	)
+	(no_connect
+		(at 381 113.03)
+	)
+	(no_connect
+		(at 381 184.15)
+	)
+	(no_connect
+		(at 381 166.37)
+	)
+	(no_connect
+		(at 340.36 196.85)
+	)
+	(no_connect
+		(at 513.08 157.48)
+	)
+	(no_connect
+		(at 381 115.57)
+	)
+	(no_connect
+		(at 340.36 113.03)
+	)
+	(no_connect
+		(at 340.36 201.93)
+	)
+	(no_connect
+		(at 340.36 176.53)
+	)
+	(no_connect
+		(at 381 151.13)
+	)
+	(no_connect
+		(at 340.36 140.97)
+	)
+	(no_connect
+		(at 340.36 171.45)
+	)
+	(no_connect
+		(at 153.67 195.58)
+	)
+	(no_connect
+		(at 381 118.11)
+	)
+	(no_connect
+		(at 340.36 189.23)
+	)
 	(wire
 		(pts
@@
 	(wire
 		(pts
+			(xy 383.54 157.48) (xy 383.54 158.75)
+		)
+		(stroke
+			(width 0)
+			(type default)
+		)
+	)
+	(wire
+		(pts
 			(xy 212.09 181.61) (xy 217.17 181.61)
 		)
@@
 	(wire
 		(pts
-			(xy 381 158.75) (xy 383.54 158.75)
+			(xy 383.54 157.48) (xy 389.89 157.48)
 		)
 		(stroke
@@
 	(wire
 		(pts
+			(xy 387.35 163.83) (xy 387.35 161.29)
+		)
+		(stroke
+			(width 0)
+			(type default)
+		)
+	)
+	(wire
+		(pts
 			(xy 510.54 140.97) (xy 516.89 140.97)
 		)
@@
 	(wire
 		(pts
+			(xy 387.35 161.29) (xy 381 161.29)
+		)
+		(stroke
+			(width 0)
+			(type default)
+		)
+	)
+	(wire
+		(pts
 			(xy 140.97 186.69) (xy 143.51 186.69)
 		)
@@
 	(wire
 		(pts
-			(xy 381 161.29) (xy 388.62 161.29)
+			(xy 387.35 163.83) (xy 391.16 163.83)
 		)
 		(stroke
@@
 	(wire
 		(pts
+			(xy 383.54 158.75) (xy 381 158.75)
+		)
+		(stroke
+			(width 0)
+			(type default)
+		)
+	)
+	(wire
+		(pts
 			(xy 190.5 73.66) (xy 190.5 66.04)
 		)
@@
 	)
 	(label "STM32ChipSelectSignal"
-		(at 388.62 161.29 0)
+		(at 391.16 163.83 0)
 		(effects
 			(font
@@
 		)
 	)
-	(label "MISO"
+	(label "STM_MISO"
 		(at 388.62 140.97 0)
 		(effects
@@
 		)
 	)
-	(label "MOSI"
+	(label "STM_MOSI"
 		(at 389.89 146.05 0)
 		(effects
@@
 	(symbol
 		(lib_id "power:GND")
-		(at 383.54 158.75 0)
+		(at 389.89 157.48 0)
 		(unit 1)
 		(exclude_from_sim no)
@@
 		(on_board yes)
 		(dnp no)
-		(fields_autoplaced yes)
 		(property "Reference" "#PWR035"
-			(at 383.54 165.1 0)
+			(at 389.89 163.83 0)
 			(effects
 				(font
@@
 		)
 		(property "Value" "GND"
-			(at 383.54 163.83 0)
+			(at 389.89 160.274 0)
 			(effects
 				(font
@@
 		)
 		(property "Footprint" ""
-			(at 383.54 158.75 0)
+			(at 389.89 157.48 0)
 			(effects
 				(font
@@
 		)
 		(property "Datasheet" ""
-			(at 383.54 158.75 0)
+			(at 389.89 157.48 0)
 			(effects
 				(font
@@
 		)
 		(property "Description" "Power symbol creates a global label with name \"GND\" , ground"
-			(at 383.54 158.75 0)
+			(at 389.89 157.48 0)
 			(effects
 				(font

Commit message: patrick feedback
Parts:
- added TP15, TP16: TestPoint, symbol Connector:TestPoint
- U6: value PTPSM365R6FRDN -> PTPSM365R6V5RDNR
Connections:
- net GND: now also TP15.1
- net at U6.1 (PGOOD): now also TP16.1
Other:
- note added: "48Vto5V DCDC Converter"
- note added: "ADC"
- note added: "CAN Subcircuit"
- note added: "Hall Sensor"
- note added: "LDO 5 to 3.3V"
- note added: "STM_32"
- note added: "TPSM365R6V5RDNR"
- note added: "Voltage Divider"
- note added: "XT60 Connectors"
- note removed: "Maybe put a testing pad here"
- note removed: "TPSM365R6"
- moved on the sheet: C10, C11, C12, C13, C14, C15, C16, C17, C2, C3, C4, C5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
