File: VDJoulemeter/HighPowerJoulemeter/HighPowerJoulemeter.kicad_sch (KiCad schematic)
At the start: 47 parts, among them J1 XT60-M, J2 XT60-M, J3 22035035, J4 22035035, U2 TMCS1107A1BQDR, U3 MCP2551-E/P, U5 MCP6286T-E/OT, U6 PTPSM365R6V5RDNR, U8 ADS1118QDGSRQ1, U9 MIC5219-3.3YM5-TR

Commit message: final draftish
Parts:
- added C1, C18, C19, C20, C23: 0.1uF, symbol Device:C
- added R5: 4k7, symbol Device:R
- added R6, R7: 50Ω, symbol Device:R
- added R8: 500Ω, symbol Device:R
- added TP17, TP18: TestPoint, symbol Connector:TestPoint
- added U4: TMCS1126A1BQDVGR, SOIC10_DVG_TEX, symbol SMV_Custom:PMCS1126A1BQDVGR
- R3: value 1kΩ -> 500Ω
- R4: value 1kΩ -> 500uF
- U3: value MCP2551-E/P -> MCP2562
Connections:
- net +3.3V: now also U3.8 (V_IO), C18.1, C23.1, R5.1, U4.4 (VS), U4.5 (VOC)
- net +5V: now also C1.1
- net 48V_IN: now also U4.1 (IN+)
- net 48V_OUT: now also U4.2 (IN-)
- net GND: now also C1.2, C18.2, C19.2, C23.2, U4.3 (*OC), U4.9 (GND); no longer U3.8
- net I_Sense: now also R3.1, TP17.1, U4.6 (VOUT); no longer R4.1
- net STM32ChipSelectSignal: now also R5.2
- net STM_MISO: now also R6.2; no longer U8.9 (DOUT_DRDY_N)
- net STM_MOSI: now also R7.2; no longer U1.53 (PA7)
- net V_Sense: now also R4.1; no longer R3.1
- net at C16.1, R3.2, U8.4 (AIN0): now also C20.1
- net at C17.1, R4.2: now also U8.6 (AIN2); no longer U8.5 (AIN1)
- new net: C19.1, C20.2, R8.2, U8.5 (AIN1)
- new net: R6.1, U8.9 (DOUT_DRDY_N)
- new net: R7.1, U1.53 (PA7)
- new net: TP18.1, U4.7 (VREF)
- new net V_Ref: R8.1
Other:
- note added: "Pull-up Resistor for CS Pin"
- note removed: "Leaving these unnconnected because only two things being measured"
- moved on the sheet: C16, C17, R3, R4, TP10, TP11, TP6

Commit message: fix
Other:
- note added: "Old Hall Sensor"
- moved on the sheet: C23, C4, TP17, TP18, TP9, U2, U4

Commit message: some changes from 10/11 feedbackk
Parts:
- removed C4: 0.1uF, symbol Device:C
- removed TP9: TestPoint, symbol Connector:TestPoint
- removed U2: TMCS1107A1BQDR, D0008A-IPC_A, symbol SMV_Custom:TMCS1107A1BQDR
- added C21, C24, C25: 10uF, symbol Device:C
- added C22, C4: 470uF, 63V, SMV_Passives:Big_Chunky_Cap, symbol SMV_Custom:Big_Chunky_Cap2
- added R10, R9: 50Ω, symbol Device:R
Connections:
- net +3.3V: now also C25.2
- net GND: now also C21.1, C21.2, C22.1, C22.2, C24.1, C24.2, C25.1, C4.1, C4.2
- net SCK: now also R9.2; no longer U1.49 (PA5)
- net STM32ChipSelectSignal: now also R10.1; no longer U1.59 (PA9)
- new net: R9.1, U1.49 (PA5)
- new net: R10.2, U1.59 (PA9)
Other:
- note removed: "HallSensor"
- note removed: "Old Hall Sensor"

Commit message: more changes
Parts:
- removed R10: 50Ω, symbol Device:R
- added R11: 0Ω, symbol Device:R
- added R12: 50Ω, symbol Device:R
Connections:
- net +3.3V: now also R11.1
- net STM32ChipSelectSignal: now also R12.2
- net at U1.32 (PA4): now also R12.1
- net at U1.34 (PB0): now also R11.2
- no-connect marks 58 -> 57
Other:
- note added: "Jumper for VBAT"
- note added: "VBAT"
- moved on the sheet: C12, C25, C3, R1, R2, TP1, TP8

Commit message: added it
Parts:
- R1: value 270kΩ -> 500kΩ
- R2: value 10kΩ -> 20kΩ
Other:
- moved on the sheet: C1
Changed lines of the file:
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@@
 	)
 	(junction
+		(at 386.08 44.45)
+		(diameter 0)
+		(color 0 0 0 0)
+	)
+	(junction
 		(at 62.23 176.53)
 		(diameter 0)
@@
 	)
 	(junction
-		(at 384.81 44.45)
-		(diameter 0)
-		(color 0 0 0 0)
-	)
-	(junction
 		(at 93.98 328.93)
 		(diameter 0)
@@
 	(wire
 		(pts
-			(xy 384.81 44.45) (xy 384.81 41.91)
-		)
-		(stroke
-			(width 0)
-			(type default)
-		)
-	)
-	(wire
-		(pts
 			(xy 373.38 346.71) (xy 373.38 349.25)
 		)
@@
 	(wire
 		(pts
+			(xy 386.08 41.91) (xy 386.08 44.45)
+		)
+		(stroke
+			(width 0)
+			(type default)
+		)
+	)
+	(wire
+		(pts
 			(xy 36.83 71.12) (xy 46.99 71.12)
 		)
@@
 	(wire
 		(pts
-			(xy 396.24 44.45) (xy 396.24 46.99)
+			(xy 398.78 44.45) (xy 398.78 46.99)
 		)
 		(stroke
@@
 	(wire
 		(pts
-			(xy 386.08 44.45) (xy 384.81 44.45)
+			(xy 388.62 44.45) (xy 386.08 44.45)
 		)
 		(stroke
@@
 	(wire
 		(pts
-			(xy 372.11 41.91) (xy 374.65 41.91)
-		)
-		(stroke
-			(width 0)
-			(type default)
-		)
-	)
-	(wire
-		(pts
 			(xy 447.04 58.42) (xy 447.04 62.23)
 		)
@@
 	(wire
 		(pts
-			(xy 384.81 58.42) (xy 386.08 58.42)
-		)
-		(stroke
-			(width 0)
-			(type default)
-		)
-	)
-	(wire
-		(pts
 			(xy 220.98 190.5) (xy 226.06 190.5)
 		)
@@
 	(wire
 		(pts
-			(xy 374.65 41.91) (xy 384.81 41.91)
+			(xy 374.65 41.91) (xy 386.08 41.91)
 		)
 		(stroke
@@
 	(wire
 		(pts
-			(xy 372.11 40.64) (xy 372.11 41.91)
-		)
-		(stroke
-			(width 0)
-			(type default)
-		)
-	)
-	(wire
-		(pts
 			(xy 283.21 83.82) (xy 298.45 83.82)
 		)
@@
 	(wire
 		(pts
-			(xy 368.3 40.64) (xy 372.11 40.64)
+			(xy 368.3 41.91) (xy 374.65 41.91)
 		)
 		(stroke
@@
 	(wire
 		(pts
-			(xy 393.7 44.45) (xy 396.24 44.45)
+			(xy 396.24 44.45) (xy 398.78 44.45)
 		)
 		(stroke
@@
 	(wire
 		(pts
-			(xy 384.81 44.45) (xy 384.81 58.42)
+			(xy 386.08 44.45) (xy 386.08 59.69)
 		)
 		(stroke
@@
 	(wire
 		(pts
-			(xy 386.08 58.42) (xy 386.08 59.69)
-		)
-		(stroke
-			(width 0)
-			(type default)
-		)
-	)
-	(wire
-		(pts
 			(xy 85.09 328.93) (xy 85.09 332.74)
 		)
@@
 	(symbol
 		(lib_id "power:GND")
-		(at 396.24 46.99 0)
+		(at 398.78 46.99 0)
 		(unit 1)
 		(exclude_from_sim no)
@@
 		(fields_autoplaced yes)
 		(property "Reference" "#PWR055"
-			(at 396.24 53.34 0)
+			(at 398.78 53.34 0)
 			(effects
 				(font
@@
 		)
 		(property "Value" "GND"
-			(at 396.24 52.07 0)
+			(at 398.78 52.07 0)
 			(effects
 				(font
@@
 		)
 		(property "Footprint" ""
-			(at 396.24 46.99 0)
+			(at 398.78 46.99 0)
 			(effects
 				(font
@@
 		)
 		(property "Datasheet" ""
-			(at 396.24 46.99 0)
+			(at 398.78 46.99 0)
 			(effects
 				(font
@@
 		)
 		(property "Description" "Power symbol creates a global label with name \"GND\" , ground"
-			(at 396.24 46.99 0)
+			(at 398.78 46.99 0)
 			(effects
 				(font
@@
 			)
 		)
-		(property "Value" "10kΩ"
+		(property "Value" "20kΩ"
 			(at 154.94 185.4199 0)
 			(effects
@@
 	(symbol
 		(lib_id "power:+5V")
-		(at 368.3 40.64 0)
+		(at 368.3 41.91 0)
 		(unit 1)
 		(exclude_from_sim no)
@@
 		(fields_autoplaced yes)
 		(property "Reference" "#PWR047"
-			(at 368.3 44.45 0)
+			(at 368.3 45.72 0)
 			(effects
 				(font
@@
 		)
 		(property "Value" "+5V"
-			(at 368.3 35.56 0)
+			(at 368.3 36.83 0)
 			(effects
 				(font
@@
 		)
 		(property "Footprint" ""
-			(at 368.3 40.64 0)
+			(at 368.3 41.91 0)
 			(effects
 				(font
@@
 		)
 		(property "Datasheet" ""
-			(at 368.3 40.64 0)
+			(at 368.3 41.91 0)
 			(effects
 				(font
@@
 		)
 		(property "Description" "Power symbol creates a global label with name \"+5V\""
-			(at 368.3 40.64 0)
+			(at 368.3 41.91 0)
 			(effects
 				(font
@@
 	(symbol
 		(lib_id "Device:C")
-		(at 389.89 44.45 90)
+		(at 392.43 44.45 90)
 		(unit 1)
 		(exclude_from_sim no)
@@
 		(fields_autoplaced yes)
 		(property "Reference" "C1"
-			(at 389.89 36.83 90)
+			(at 392.43 36.83 90)
 			(effects
 				(font
@@
 		)
 		(property "Value" "0.1uF"
-			(at 389.89 39.37 90)
+			(at 392.43 39.37 90)
 			(effects
 				(font
@@
 		)
 		(property "Footprint" ""
-			(at 393.7 43.4848 0)
+			(at 396.24 43.4848 0)
 			(effects
 				(font
@@
 		)
 		(property "Datasheet" "~"
-			(at 389.89 44.45 0)
+			(at 392.43 44.45 0)
 			(effects
 				(font
@@
 		)
 		(property "Description" "Unpolarized capacitor"
-			(at 389.89 44.45 0)
+			(at 392.43 44.45 0)
 			(effects
 				(font
@@
 			)
 		)
-		(property "Value" "270kΩ"
+		(property "Value" "500kΩ"
 			(at 154.94 173.9899 0)
 			(effects

Commit message: changes
Parts:
- added TP19, TP20, TP21, TP22, TP23, TP24, TP25, TP26, TP27, TP28, TP29, TP30, TP31, TP32, TP33, TP34, TP35, TP36, TP37, TP38, TP39, TP40, TP41, TP42, TP43, TP44, TP45, TP46, TP47, TP48, TP49, TP50, TP51, TP52, TP53, TP54, TP55, TP56, TP57, TP58, TP59, TP60, TP61, TP62, TP63, TP64, TP65, TP66, TP9: TestPoint, symbol Connector:TestPoint
- U4: value TMCS1126A1BQDVGR -> TMCS1126B6AQDVGRQ1
Connections:
- net +3.3V: now also TP22.1, TP26.1, TP35.1, TP40.1, TP42.1, TP55.1, TP58.1
- net +5V: now also TP48.1, TP64.1
- net 48V_IN: now also TP9.1
- net 48V_OUT: now also TP19.1, TP66.1
- net CAN_H: now also TP51.1, TP53.1, TP56.1
- net CAN_L: now also TP50.1, TP52.1, TP57.1
- net GND: now also TP20.1, TP21.1, TP24.1, TP25.1, TP28.1, TP29.1, TP31.1, TP32.1, TP33.1, TP41.1, TP44.1, TP45.1, TP47.1, TP54.1, TP62.1, TP63.1
- net STM_CAN_RX_PIN: now also TP36.1, TP49.1
- net STM_CAN_TX_PIN: now also TP39.1, TP46.1
- net STM_MISO: now also TP37.1; no longer TP11.1
- net VoltageDividerOut: now also TP27.1
- net at C19.1, C20.2, R8.2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: now also TP60.1
- net at C7.2, U6.8 (VCC): now also TP23.1
- net at R11.2, U1.34 (PB0): now also TP43.1
- net at C16.1, C20.1, R3.2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: now also TP59.1
- net at C17.1, R4.2, U8.6 (AIN2): now also TP61.1
- net at R6.1, U8.9 (DOUT_DRDY_N): now also TP11.1
- net at C10.1, U9.4 (BYP): now also TP65.1
- net at R12.1, U1.32 (PA4): now also TP34.1
- net at R9.1, U1.49 (PA5): now also TP38.1
- net at R7.1, U1.53 (PA7): now also TP30.1
Other:
- moved on the sheet: C7, R12, R7

Commit message: all feedback implemented except footprints
Parts:
- removed C20: 0.1uF, symbol Device:C
- R4: value 500uF -> 500Ω
Connections:
- net +3.3V: now also U3.5 (V_IO); no longer U3.8 (V_IO)
- net GND: now also U3.8 (STBY)
- no-connect marks 57 -> 56
Other:
- note removed: "Leave Pin 5 unconnected!! It is a reference voltage output"
Changed lines of the file:
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@@
 		)
 	)
-	(text "Leave Pin 5 unconnected!! It is a reference voltage output"
-		(exclude_from_sim no)
-		(at 406.4 314.706 0)
-		(effects
-			(font
-				(size 1.27 1.27)
-			)
-		)
-	)
 	(text "Jumper for VBAT"
 		(exclude_from_sim no)
@@
 	)
 	(junction
-		(at 93.98 323.85)
-		(diameter 0)
-		(color 0 0 0 0)
-	)
-	(junction
 		(at 360.68 346.71)
 		(diameter 0)
@@
 	)
 	(junction
-		(at 93.98 328.93)
-		(diameter 0)
-		(color 0 0 0 0)
-	)
-	(junction
 		(at 410.21 355.6)
 		(diameter 0)
@@
 	)
 	(no_connect
-		(at 387.35 309.88)
-	)
-	(no_connect
 		(at 457.2 133.35)
 	)
@@
 	(wire
 		(pts
-			(xy 85.09 323.85) (xy 93.98 323.85)
-		)
-		(stroke
-			(width 0)
-			(type default)
-		)
-	)
-	(wire
-		(pts
 			(xy 203.2 40.64) (xy 208.28 40.64)
 		)
@@
 	(wire
 		(pts
-			(xy 93.98 323.85) (xy 115.57 323.85)
+			(xy 85.09 323.85) (xy 115.57 323.85)
 		)
 		(stroke
@@
 	(wire
 		(pts
-			(xy 107.95 328.93) (xy 93.98 328.93)
+			(xy 85.09 328.93) (xy 107.95 328.93)
 		)
 		(stroke
@@
 	(wire
 		(pts
-			(xy 391.16 124.46) (xy 391.16 127)
+			(xy 387.35 309.88) (xy 387.35 313.69)
 		)
 		(stroke
@@
 	(wire
 		(pts
-			(xy 384.81 307.34) (xy 392.43 307.34)
+			(xy 391.16 124.46) (xy 391.16 127)
 		)
 		(stroke
@@
 	(wire
 		(pts
-			(xy 384.81 304.8) (xy 387.35 304.8)
+			(xy 384.81 307.34) (xy 392.43 307.34)
 		)
 		(stroke
@@
 	(wire
 		(pts
-			(xy 241.3 198.12) (xy 241.3 199.39)
+			(xy 384.81 304.8) (xy 387.35 304.8)
 		)
 		(stroke
@@
 	(wire
 		(pts
-			(xy 392.43 204.47) (xy 392.43 207.01)
+			(xy 241.3 198.12) (xy 241.3 199.39)
 		)
 		(stroke
@@
 	(wire
 		(pts
-			(xy 46.99 72.39) (xy 46.99 73.66)
+			(xy 392.43 204.47) (xy 392.43 207.01)
 		)
 		(stroke
@@
 	(wire
 		(pts
-			(xy 97.79 325.12) (xy 93.98 325.12)
+			(xy 46.99 72.39) (xy 46.99 73.66)
 		)
 		(stroke
@@
 	(wire
 		(pts
-			(xy 93.98 325.12) (xy 93.98 323.85)
-		)
-		(stroke
-			(width 0)
-			(type default)
-		)
-	)
-	(wire
-		(pts
 			(xy 279.4 81.28) (xy 279.4 76.2)
 		)
@@
 	(wire
 		(pts
-			(xy 93.98 332.74) (xy 93.98 328.93)
-		)
-		(stroke
-			(width 0)
-			(type default)
-		)
-	)
-	(wire
-		(pts
 			(xy 476.25 156.21) (xy 482.6 156.21)
 		)
@@
 	(wire
 		(pts
-			(xy 97.79 332.74) (xy 93.98 332.74)
-		)
-		(stroke
-			(width 0)
-			(type default)
-		)
-	)
-	(wire
-		(pts
 			(xy 85.09 332.74) (xy 85.09 336.55)
 		)
@@
 	(wire
 		(pts
-			(xy 85.09 328.93) (xy 93.98 328.93)
-		)
-		(stroke
-			(width 0)
-			(type default)
-		)
-	)
-	(wire
-		(pts
 			(xy 312.42 304.8) (xy 344.17 304.8)
 		)
@@
 	(symbol
 		(lib_id "power:GND")
+		(at 387.35 313.69 0)
+		(unit 1)
+		(exclude_from_sim no)
+		(in_bom yes)
+		(on_board yes)
+		(dnp no)
+		(fields_autoplaced yes)
+		(property "Reference" "#PWR04"
+			(at 387.35 320.04 0)
+			(effects
+				(font
+					(size 1.27 1.27)
+				)
+				(hide yes)
+			)
+		)
+		(property "Value" "GND"
+			(at 387.35 318.77 0)
+			(effects
+				(font
+					(size 1.27 1.27)
+				)
+			)
+		)
+		(property "Footprint" ""
+			(at 387.35 313.69 0)
+			(effects
+				(font
+					(size 1.27 1.27)
+				)
+				(hide yes)
+			)
+		)
+		(property "Datasheet" ""
+			(at 387.35 313.69 0)
+			(effects
+				(font
+					(size 1.27 1.27)
+				)
+				(hide yes)
+			)
+		)
+		(property "Description" "Power symbol creates a global label with name \"GND\" , ground"
+			(at 387.35 313.69 0)
+			(effects
+				(font
+					(size 1.27 1.27)
+				)
+				(hide yes)
+			)
+		)
+		(pin "1"
+		)
+		(instances
+			(project ""
+				(path "/d9b1233e-8a2d-46d3-b6ba-86b7db1904e8"
+					(reference "#PWR04")
+					(unit 1)
+				)
+			)
+		)
+	)
+	(symbol
+		(lib_id "power:GND")
 		(at 26.67 172.72 0)
 		(unit 1)
@@
 			)
 		)
-		(property "Value" "500uF"
+		(property "Value" "500Ω"
 			(at 105.41 345.44 90)
 			(effects
@@
 					(unit 1)
 				)
-			)
-		)
-	)
-	(symbol
-		(lib_id "Device:C")
-		(at 97.79 328.93 0)
-		(unit 1)
-		(exclude_from_sim no)
-		(in_bom yes)
-		(on_board yes)
-		(dnp no)
-		(fields_autoplaced yes)
-		(property "Reference" "C20"
-			(at 101.6 327.6599 0)
-			(effects
-				(font
-					(size 1.27 1.27)
-				)
-				(justify left)
-			)
-		)
-		(property "Value" "0.1uF"
-			(at 101.6 330.1999 0)
-			(effects
-				(font
-					(size 1.27 1.27)
-				)
-				(justify left)
-			)
-		)
-		(property "Footprint" ""
-			(at 98.7552 332.74 0)
-			(effects
-				(font
-					(size 1.27 1.27)
-				)
-				(hide yes)
-			)
-		)
-		(property "Datasheet" "~"
-			(at 97.79 328.93 0)
-			(effects
-				(font
-					(size 1.27 1.27)
-				)
-				(hide yes)
-			)
-		)
-		(property "Description" "Unpolarized capacitor"
-			(at 97.79 328.93 0)
-			(effects
-				(font
-					(size 1.27 1.27)
-				)
-				(hide yes)
-			)
-		)
-		(pin "2"
-		)
-		(pin "1"
-		)
-		(instances
-			(project ""
-				(path "/d9b1233e-8a2d-46d3-b6ba-86b7db1904e8"
-					(reference "C20")
-					(unit 1)
-				)

Commit message: changes
Parts:
- added TP67: TestPoint, TestPoint:TestPoint_Pad_4.0x4.0mm, symbol Connector:TestPoint
- TP1, TP10, TP11, TP12, TP13, TP16, TP17, TP18, TP19, TP2, TP22, TP26, TP27, TP3, TP30, TP34, TP35, TP36, TP37, TP38, TP39, TP4, TP40, TP42, TP43, TP46, TP48, TP49, TP5, TP50, TP51, TP52, TP53, TP55, TP56, TP57, TP58, TP59, TP6, TP60, TP61, TP64, TP66, TP7, TP8, TP9: footprint (none) -> TestPoint:TestPoint_Pad_1.0x1.0mm
- TP14, TP15, TP20, TP21, TP23, TP24, TP25, TP28, TP29, TP31, TP32, TP33, TP41, TP44, TP45, TP47, TP54, TP62, TP63, TP65: footprint (none) -> TestPoint:TestPoint_Pad_4.0x4.0mm
- U5: footprint SOT-23-5_MC_MCH -> SMV_ICs:SOT-23-5_MC_MCH
Connections:
- net GND: now also TP67.1
- net V_Ref: now also TP18.1, U4.7 (VREF)
- no-connect marks 56 -> 55
