File: VDJoulemeter/HighPowerJoulemeter/HighPowerJoulemeter.kicad_pcb (KiCad board)
At the start: 4 copper layers, 771 x 448.5 mm, 113 parts, among them J1 XT60-M, J2 XT60-M, J3 22035035, J4 22035035, U3 MCP2562, U4 TMCS1126B6AQDVGRQ1, U5 MCP6286T-E/OT, U6 PTPSM365R6V5RDNR, U8 ADS1118QDGSRQ1, U9 MIC5219-3.3YM5-TR

Commit message: all 9 components down except voltage divider lost in the jumble :'(
Parts:
- U5: value MCP6286T-E/OT -> VoltageBuffer
- moved J3 352.3 mm to (514.8, 309.6), turned to 180 degrees
Changed lines of the file:
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@@
 	(footprint "SMV_Connectors:3pin_CON_22035035_MOL"
 		(layer "F.Cu")
-		(at 242.5 86)
+		(at 514.75401 309.649998 180)
 		(tags "22035035 ")
 		(property "Reference" "J3"
-			(at -2.49999 -6.35 0)
+			(at -2.49999 -6.35 180)
 			(unlocked yes)
 			(layer "F.SilkS")
@@
 		)
 		(property "Value" "22035035"
-			(at -2.49999 -6.35 0)
+			(at -2.49999 -6.35 180)
 			(unlocked yes)
 			(layer "F.Fab")
@@
 		(attr through_hole)
 		(fp_line
-			(start -7.44998 -1.800002)
-			(end -7.44998 3.099999)
+			(start 4.228 0.635)
+			(end 2.704 0)
 			(stroke
 				(width 0.127)
@@
 		)
 		(fp_line
-			(start -7.44998 3.099999)
-			(end 2.45 3.099999)
+			(start 4.228 -0.635)
+			(end 4.228 0.635)
 			(stroke
 				(width 0.127)
@@
 		)
 		(fp_line
-			(start 2.45 -1.800002)
-			(end -7.44998 -1.800002)
+			(start 2.704 0)
+			(end 4.228 -0.635)
 			(stroke
 				(width 0.127)
@@
 		)
 		(fp_line
-			(start 2.704 0)
-			(end 4.228 -0.635)
+			(start 2.45 -1.800002)
+			(end -7.44998 -1.800002)
 			(stroke
 				(width 0.127)
@@
 		)
 		(fp_line
-			(start 4.228 -0.635)
-			(end 4.228 0.635)
+			(start -7.44998 3.099999)
+			(end 2.45 3.099999)
 			(stroke
 				(width 0.127)
@@
 		)
 		(fp_line
-			(start 4.228 0.635)
-			(end 2.704 0)
+			(start -7.44998 -1.800002)
+			(end -7.44998 3.099999)
 			(stroke
 				(width 0.127)
@@
 		)
 		(fp_line
-			(start -8.71998 -3.070002)
-			(end -8.71998 4.369999)
+			(start 3.72 4.369999)
+			(end 3.72 -3.070002)
 			(stroke
 				(width 0.127)
@@
 		)
 		(fp_line
-			(start -8.71998 4.369999)
-			(end 3.72 4.369999)
+			(start 3.72 -3.070002)
+			(end -8.71998 -3.070002)
 			(stroke
 				(width 0.127)
@@
 		)
 		(fp_line
-			(start 3.72 -3.070002)
-			(end -8.71998 -3.070002)
+			(start -8.71998 4.369999)
+			(end 3.72 4.369999)
 			(stroke
 				(width 0.127)
@@
 		)
 		(fp_line
-			(start 3.72 4.369999)
-			(end 3.72 -3.070002)
+			(start -8.71998 -3.070002)
+			(end -8.71998 4.369999)
 			(stroke
 				(width 0.127)
@@
 		)
 		(fp_line
-			(start -7.44998 -1.800002)
-			(end -7.44998 3.099999)
+			(start 4.228 0.635)
+			(end 2.704 0)
 			(stroke
 				(width 0.127)
@@
 		)
 		(fp_line
-			(start -7.44998 3.099999)
-			(end 2.45 3.099999)
+			(start 4.228 -0.635)
+			(end 4.228 0.635)
 			(stroke
 				(width 0.127)
@@
 		)
 		(fp_line
-			(start 2.45 -1.800002)
-			(end -7.44998 -1.800002)
+			(start 2.704 0)
+			(end 4.228 -0.635)
 			(stroke
 				(width 0.127)
@@
 		)
 		(fp_line
-			(start 2.704 0)
-			(end 4.228 -0.635)
+			(start 2.45 -1.800002)
+			(end -7.44998 -1.800002)
 			(stroke
 				(width 0.127)
@@
 		)
 		(fp_line
-			(start 4.228 -0.635)
-			(end 4.228 0.635)
+			(start -7.44998 3.099999)
+			(end 2.45 3.099999)
 			(stroke
 				(width 0.127)
@@
 		)
 		(fp_line
-			(start 4.228 0.635)
-			(end 2.704 0)
+			(start -7.44998 -1.800002)
+			(end -7.44998 3.099999)
 			(stroke
 				(width 0.127)
@@
 		)
 		(fp_text user "WITHOUT_COIN,_COPPER_UNDERPLATING"
-			(at -2.49999 -10.780001 0)
+			(at -2.49999 -10.780001 180)
 			(unlocked yes)
 			(layer "F.SilkS")
@@
 		)
 		(fp_text user "22035035"
-			(at -2.49999 -15.860001 0)
+			(at -2.49999 -15.860001 180)
 			(unlocked yes)
 			(layer "F.SilkS")
@@
 		)
 		(fp_text user "MINI-SPOX_2.5_W/B_VERT_PLUG_ASSY_-3_CKT"
-			(at -2.49999 -13.320001 0)
+			(at -2.49999 -13.320001 180)
 			(unlocked yes)
 			(layer "F.SilkS")
@@
 		)
 		(fp_text user "NOTE"
-			(at -7.44998 8.359998 0)
+			(at -7.44998 8.359998 180)
 			(unlocked yes)
 			(layer "Cmts.User")
@@
 		)
 		(fp_text user "MAXIMUM_PACKAGE_HEIGHT:_5.9_MM"
-			(at -7.44998 10.899998 0)
+			(at -7.44998 10.899998 180)
 			(unlocked yes)
 			(layer "Cmts.User")
@@
 		)
 		(fp_text user "MINI-SPOX_2.5_W/B_VERT_PLUG_ASSY_-3_CKT"
-			(at -2.49999 -13.320001 0)
+			(at -2.49999 -13.320001 180)
 			(unlocked yes)
 			(layer "F.Fab")
@@
 		)
 		(fp_text user "WITHOUT_COIN,_COPPER_UNDERPLATING"
-			(at -2.49999 -10.780001 0)
+			(at -2.49999 -10.780001 180)
 			(unlocked yes)
 			(layer "F.Fab")
@@
 		)
 		(fp_text user "22035035"
-			(at -2.49999 -15.860001 0)
+			(at -2.49999 -15.860001 180)
 			(unlocked yes)
 			(layer "F.Fab")
@@
 		)
 		(fp_text user "${REFERENCE}"
-			(at -2.49999 -6.35 0)
+			(at -2.49999 -6.35 180)
 			(unlocked yes)
 			(layer "F.Fab")
@@
 		)
 		(pad "1" thru_hole rect
-			(at 0 0)
+			(at 0 0 180)
 			(size 1.15 1.15)
 			(drill 0.8)
@@
 		)
 		(pad "2" thru_hole circle
-			(at -2.5 0)
+			(at -2.5 0 180)
 			(size 1.15 1.15)
 			(drill 0.8)
@@
 		)
 		(pad "3" thru_hole circle
-			(at -5 0)
+			(at -5 0 180)
 			(size 1.15 1.15)
 			(drill 0.8)
@@
 			(layer "F.Fab")
 		)
-		(fp_text user "Designator42"
+		(fp_text user "ADC"
 			(at -2.921 -3.0988 0)
 			(unlocked yes)
@@
 			)
 		)
-		(property "Value" "MCP6286T-E/OT"
+		(property "Value" "VoltageBuffer"
 			(at 0 0 0)
 			(unlocked yes)

Commit message: detangling the ratsnest
Parts:
- U5: value VoltageBuffer -> MCP6286T-E/OT
- moved C12 334.7 mm to (455.1, 137.8)
- moved C25 329.8 mm to (455.1, 147.8)
- moved TP2 298.4 mm to (-68.0, -66.5)
- moved TP42 289.5 mm to (464.6, 140.3)
- moved C4 278.6 mm to (-75.4, -49.5)
- moved TP17 267.3 mm to (-62.2, 0.00)
- moved TP18 267.3 mm to (-62.2, 3.05)
- moved TP3 261.0 mm to (-90.5, 74.5)
- moved TP15 259.8 mm to (-88.5, 88.0)
- moved TP19 255.5 mm to (-51.8, -7.30)
- moved TP22 255.5 mm to (-51.8, -4.25)
- moved TP9 254.8 mm to (-57.2, -1.25)
- moved TP66 247.4 mm to (5.00, -42.8)
- moved C21 246.8 mm to (-24.5, -65.5)
- moved C23 244.9 mm to (-79.5, -0.50)
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Other:
- board text added: "Voltage Divider"

Commit message: more changes
Parts:
- moved TP54 326.1 mm to (458.8, 232.2)
- moved TP45 319.1 mm to (23.8, 329.5)
- moved C18 300.0 mm to (418.2, 189.8)
- moved C1 296.5 mm to (401.5, 66.0)
- moved TP53 292.9 mm to (451.8, 232.8)
- moved TP67 289.4 mm to (382.8, 257.2)
- moved TP52 288.2 mm to (445.5, 232.8)
- moved C11 286.0 mm to (401.5, 71.0)
- moved C5 283.2 mm to (390.0, 201.5)
- moved TP26 261.4 mm to (13.2, 328.8)
- moved TP7 256.4 mm to (416.2, 76.2)
- moved TP6 255.7 mm to (414.7, 70.0)
- moved TP27 255.6 mm to (18.5, 328.5)
- moved TP51 251.2 mm to (385.2, 264.0)
- moved TP55 250.1 mm to (428.5, 189.2)
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
Commit message: finished grouping
Parts:
- moved TP36 469.4 mm to (640.5, 133.8)
- moved TP29 468.5 mm to (635.2, 132.5)
- moved TP28 462.9 mm to (626.8, 140.8)
- moved TP30 462.4 mm to (634.8, 127.2)
- moved TP37 453.0 mm to (628.2, 127.4)
- moved TP38 453.0 mm to (628.2, 130.4)
- moved TP39 453.0 mm to (628.2, 133.5)
- moved TP41 452.0 mm to (621.8, 133.8)
- moved TP40 446.1 mm to (621.5, 127.2)
- moved C6 372.8 mm to (452.5, 0.25)
- moved C7 369.0 mm to (459.3, 2.00)
- moved C8 369.0 mm to (459.3, 5.01)
- moved C15 367.7 mm to (464.5, 6.75)
- moved C9 356.6 mm to (459.3, 10.4)
- moved C13 351.9 mm to (471.2, 101.5)
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
Commit message: layout starts
Parts:
- moved TP15 835.5 mm to (239.2, -680.5)
- moved C24 833.7 mm to (249.8, -685.0)
- moved TP8 819.8 mm to (208.2, -466.2)
- moved TP26 819.7 mm to (213.0, -466.2)
- moved TP27 812.7 mm to (206.2, -462.2)
- moved TP45 808.7 mm to (209.8, -457.5)
- moved C3 802.8 mm to (213.0, -463.2), turned to 90 degrees
- moved C22 798.4 mm to (264.7, -659.8)
- moved J2 798.4 mm to (244.6, -667.2)
- moved TP3 798.4 mm to (235.7, -654.2)
- moved U5 795.8 mm to (209.6, -463.3)
- moved C2 777.0 mm to (118.5, -482.8), turned to -90 degrees
- moved C16 764.7 mm to (111.5, -478.0), turned to 180 degrees
- moved C17 760.7 mm to (121.5, -478.0)
- moved U8 755.6 mm to (116.5, -479.0)
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Connections:
- C10 pad 3: (no net) -> Net-(U9-BYP)
- C10 pad 4: (no net) -> GND
- C22 pad 3: (no net) -> GND
- C22 pad 4: (no net) -> GND
- C4 pad 3: (no net) -> GND
- C4 pad 4: (no net) -> GND
Routing:
- net /CAN_H: track 0.00 -> 23.3 mm
- net +3.3V: track 0.00 -> 23.3 mm
- net /CAN_L: track 0.00 -> 19.7 mm
- net Net-(U9-BYP): track 0.00 -> 14.8 mm
- net Net-(U8-AIN1): track 0.00 -> 9.06 mm
- net +5V: track 0.00 -> 8.66 mm
- net Net-(U8-AIN0): track 0.00 -> 7.83 mm
- net GND: track 0.00 -> 6.55 mm
- net Net-(U8-AIN2): track 0.00 -> 6.32 mm
- net /STM32ChipSelectSignal: track 0.00 -> 5.35 mm
- net Net-(U8-DOUT_DRDY_N): track 0.00 -> 4.81 mm
- net /V_Sense: track 0.00 -> 3.38 mm
- net /SCK: track 0.00 -> 3.00 mm
- net /STM_MOSI: track 0.00 -> 2.74 mm

Commit message: layout
Parts:
- U4: footprint SMV_ICs:SOIC_DBVRQ1_TEX -> SMV_ICs:DVG0010A-MFG
- moved TP36 482.9 mm to (119.4, -615.1), turned to 180 degrees
- moved TP40 482.1 mm to (122.0, -606.5), turned to 180 degrees
- moved TP30 474.4 mm to (121.8, -618.9), turned to 180 degrees
- moved TP39 468.1 mm to (122.0, -613.5), turned to 180 degrees
- moved TP37 467.6 mm to (121.8, -616.7), turned to 180 degrees
- moved TP38 466.4 mm to (122.0, -608.9), turned to 180 degrees
- moved TP28 416.5 mm to (160.6, -485.2)
- moved TP29 416.5 mm to (169.1, -493.4)
- moved TP41 416.5 mm to (155.6, -492.2)
- moved U1 369.9 mm to (158.6, -610.0), turned to 180 degrees
- moved R7 338.9 mm to (118.6, -619.2), turned to 180 degrees
- moved R9 335.7 mm to (121.2, -611.3), turned to 180 degrees
- moved TP52 326.9 mm to (90.6, -617.6), turned to 180 degrees
- moved TP53 321.7 mm to (90.6, -612.6), turned to 180 degrees
- moved TP33 320.0 mm to (138.8, -464.8)
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Connections:
- net /CAN_H renamed /CAN_P
- net /CAN_L renamed /CAN_N
- C21 pad 1: GND -> Net-(J1-NEG)
- C22 pad 4: GND -> Net-(J2-NEG)
- C24 pad 1: GND -> Net-(J2-NEG)
- C4 pad 4: GND -> Net-(J1-NEG)
- J1 pad N: GND -> Net-(J1-NEG)
- J2 pad N: GND -> Net-(J2-NEG)
- TP14 pad 1: GND -> Net-(J1-NEG)
- TP15 pad 1: GND -> Net-(J2-NEG)
- U6 pad 12: (no net) -> 48V_OUT
- U6 pad 13: (no net) -> 48V_OUT
Routing:
- net +5V: track 8.66 -> 88.9 mm, vias 0 -> 2
- net +3.3V: track 23.3 -> 89.6 mm, vias 0 -> 2
- net /STM32ChipSelectSignal: track 5.35 -> 68.2 mm, vias 0 -> 2
- net 48V_OUT: track 0.00 -> 36.7 mm
- net Net-(J2-NEG): track 0.00 -> 23.3 mm
- net Net-(J1-NEG): track 0.00 -> 22.9 mm
- net /STM_CAN_RX_PIN: track 0.00 -> 18.9 mm
- net /CAN_N: track 19.7 -> 38.1 mm
- net 48V_IN: track 0.00 -> 18.3 mm
- net /V_Ref: track 0.00 -> 14.5 mm, vias 0 -> 2
- net /CAN_P: track 23.3 -> 37.7 mm
- net /VoltageDividerOut: track 0.00 -> 13.0 mm
- net Net-(U1-PA4): track 0.00 -> 11.3 mm
- net Net-(U1-PA7): track 0.00 -> 10.5 mm
- net Net-(U1-PA5): track 0.00 -> 10.4 mm
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Other:
- board size 771 x 448.5 mm -> 140.8 x 171.2 mm
- board text added: "ADC"

Commit message: more layout
Parts:
- removed TP20, TP21, TP24, TP25, TP28, TP29, TP31, TP32, TP33, TP41, TP44, TP47, TP54, TP62, TP63, TP67: TestPoint, TestPoint:TestPoint_Pad_4.0x4.0mm
- moved TP45 12.9 mm to (100.6, -640.0)
Connections:
- U6 pad 12: 48V_OUT -> (no net)
- U6 pad 13: 48V_OUT -> (no net)
Routing:
- net /SCK: track 3.00 -> 75.2 mm, vias 0 -> 2
- net /STM_MOSI: track 2.74 -> 71.9 mm, vias 0 -> 2
- net /STM_MISO: track 8.04 -> 68.4 mm, vias 0 -> 1
- net Net-(U1-PB0): track 2.40 -> 43.1 mm
- net /V_Sense: track 5.40 -> 24.8 mm, vias 0 -> 2
- net +3.3V: track 89.6 -> 104.1 mm
- net /STM_CAN_TX_PIN: track 7.37 -> 16.6 mm
- net GND: track 6.55 -> 14.1 mm
- net +5V: track 88.9 -> 87.3 mm
- added copper zone on F.Cu, net +3.3V
- added copper zone on In1.Cu, net GND
Other:
- board size 140.8 x 171.2 mm -> 119.2 x 118.6 mm
- board text removed: "Voltage Divider"

Commit message: fixed connection issues
Parts:
- moved TP45 13.6 mm to (96.6, -653.0)
- moved TP58 2.58 mm to (150.8, -656.6)
- moved C19 0.66 mm to (148.2, -657.6)
- moved TP60 0.40 mm to (146.0, -656.4)
- moved TP61 0.32 mm to (151.8, -658.8)
- moved C9 0.20 mm to (136.2, -675.6)
Routing:
- net GND: track 14.1 -> 148.0 mm, vias 0 -> 16
- net 48V_OUT: track 36.7 -> 38.7 mm
- net Net-(U8-AIN1): track 9.06 -> 7.11 mm
- net /VoltageDividerOut: track 13.0 -> 11.5 mm
- net +5V: track 87.3 -> 86.2 mm, vias 2 -> 5
- net +3.3V: track 104.1 -> 105.1 mm, vias 2 -> 4
- net /V_Sense: track 24.8 -> 25.6 mm
- added copper zone on In2.Cu, net +3.3V
- added copper zone on F.Cu, net +5V
- added copper zone on In2.Cu, net +5V
- added copper zone on F.Cu, net 48V_IN
- added copper zone on F.Cu, net 48V_OUT
