File: VDJoulemeter/HighPowerJoulemeter/HighPowerJoulemeter.kicad_pcb (KiCad board)
At the start: 4 copper layers, 119.2 x 118.6 mm, 97 parts, among them J1 XT60-M, J2 XT60-M, J3 22035035, J4 22035035, U3 MCP2562, U4 TMCS1126B6AQDVGRQ1, U5 MCP6286T-E/OT, U6 PTPSM365R6V5RDNR, U8 ADS1118QDGSRQ1, U9 MIC5219-3.3YM5-TR

Commit message: fixes for everything except LED layout placements and ADC shift
Parts:
- moved C17 720.1 mm to (163.9, 59.2)
- moved C1 720.1 mm to (151.8, 44.0)
- moved C10 720.1 mm to (167.5, 47.4)
- moved C11 720.1 mm to (157.8, 44.2)
- moved C12 720.1 mm to (204.3, 116.6)
- moved C13 720.1 mm to (205.3, 103.1)
- moved C14 720.1 mm to (205.5, 98.9)
- moved C15 720.1 mm to (140.7, 50.8)
- moved C16 720.1 mm to (153.7, 59.2)
- moved C18 720.1 mm to (110.4, 100.2)
- moved C19 720.1 mm to (156.9, 62.4)
- moved C2 720.1 mm to (160.7, 54.5)
- moved C21 720.1 mm to (116.9, 41.4)
- moved C22 720.1 mm to (125.5, 58.5)
- moved C23 720.1 mm to (149.3, 60.0)
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Routing:
- net GND: track 148.0 -> 125.5 mm, vias 16 -> 15
- net /STM_MISO: track 68.4 -> 68.9 mm
