File: JouleMeter/Joule Meter.kicad_sch (KiCad schematic)
At the start: 37 parts, among them J1 XT60-M, J2 22035035, U1 ADS1118IDGS-Q1, U4 MCP2551-I-P

Commit message: 9-18-2025
Parts:
- 0.1μF: value C7 -> C11
- renumbered BLM21PG221SN1D to BLM18AG102SN1D, C8 to C1, C4 to C10, C5 to C12, C7 to C14, C9 to C2, C1 to C3, C12 to C4, C10 to C5, C2 to C6, C11 to C7, C6 to C8, C3 to C9, R7 to R1, R4 to R10, R5 to R11, R6 to R12, R10 to R2, R1 to R3, R2 to R4, R12 to R5, R13 to R6, R8 to R7, R9 to R8, R3 to R9
Changed lines of the file:
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@@
 		(company "Sergio Gonzalez")
 		(comment 1 "Last edit: 9/17/2025")
+		(comment 2 "To do:")
+		(comment 3 "Verify correct values for the RC filter")
 	)
 	(rectangle
@@
 		(dnp no)
 		(fields_autoplaced yes)
-		(property "Reference" "C9"
+		(property "Reference" "C2"
 			(at 300.99 29.2099 0)
 			(effects
@@
 			(project ""
 				(path "/3c05686f-5554-4d70-b348-db94545e7981"
-					(reference "C9")
+					(reference "C2")
 					(unit 1)
 				)
@@
 		(dnp no)
 		(fields_autoplaced yes)
-		(property "Reference" "C10"
+		(property "Reference" "C5"
 			(at 55.88 64.7699 0)
 			(effects
@@
 			(project ""
 				(path "/3c05686f-5554-4d70-b348-db94545e7981"
-					(reference "C10")
+					(reference "C5")
 					(unit 1)
 				)
@@
 		(dnp no)
 		(fields_autoplaced yes)
-		(property "Reference" "R9"
+		(property "Reference" "R8"
 			(at 104.14 179.0699 0)
 			(effects
@@
 			(project "Joule Meter"
 				(path "/3c05686f-5554-4d70-b348-db94545e7981"
-					(reference "R9")
+					(reference "R8")
 					(unit 1)
 				)
@@
 		(on_board yes)
 		(dnp no)
-		(property "Reference" "R13"
+		(property "Reference" "R6"
 			(at 119.634 134.874 0)
 			(effects
@@
 			(project "Joule Meter"
 				(path "/3c05686f-5554-4d70-b348-db94545e7981"
-					(reference "R13")
+					(reference "R6")
 					(unit 1)
 				)
@@
 		(dnp no)
 		(fields_autoplaced yes)
-		(property "Reference" "C12"
+		(property "Reference" "C4"
 			(at 77.47 35.5599 0)
 			(effects
@@
 			(project ""
 				(path "/3c05686f-5554-4d70-b348-db94545e7981"
-					(reference "C12")
+					(reference "C4")
 					(unit 1)
 				)
@@
 		(on_board yes)
 		(dnp no)
-		(property "Reference" "R1"
+		(property "Reference" "R3"
 			(at 269.748 26.67 0)
 			(effects
@@
 			(project ""
 				(path "/3c05686f-5554-4d70-b348-db94545e7981"
-					(reference "R1")
+					(reference "R3")
 					(unit 1)
 				)
@@
 			)
 		)
-		(property "Value" "C7"
+		(property "Value" "C11"
 			(at 151.638 147.3201 0)
 			(effects
@@
 		(dnp no)
 		(fields_autoplaced yes)
-		(property "Reference" "R6"
+		(property "Reference" "R12"
 			(at 172.72 168.91 90)
 			(effects
@@
 			(project "Joule Meter"
 				(path "/3c05686f-5554-4d70-b348-db94545e7981"
-					(reference "R6")
+					(reference "R12")
 					(unit 1)
 				)
@@
 		(dnp no)
 		(fields_autoplaced yes)
-		(property "Reference" "R8"
+		(property "Reference" "R7"
 			(at 104.14 166.3699 0)
 			(effects
@@
 			(project "Joule Meter"
 				(path "/3c05686f-5554-4d70-b348-db94545e7981"
-					(reference "R8")
+					(reference "R7")
 					(unit 1)
 				)
@@
 		(dnp no)
 		(fields_autoplaced yes)
-		(property "Reference" "C4"
+		(property "Reference" "C10"
 			(at 261.62 49.5299 0)
 			(effects
@@
 			(project ""
 				(path "/3c05686f-5554-4d70-b348-db94545e7981"
-					(reference "C4")
+					(reference "C10")
 					(unit 1)
 				)
@@
 		(on_board yes)
 		(dnp no)
-		(property "Reference" "BLM21PG221SN1D"
+		(property "Reference" "BLM18AG102SN1D"
 			(at 251.714 161.29 90)
 			(effects
@@
 			(project ""
 				(path "/3c05686f-5554-4d70-b348-db94545e7981"
-					(reference "BLM21PG221SN1D")
+					(reference "BLM18AG102SN1D")
 					(unit 1)
 				)
@@
 		(on_board yes)
 		(dnp no)
-		(property "Reference" "R4"
+		(property "Reference" "R10"
 			(at 160.02 163.83 90)
 			(effects
@@
 			(project "Joule Meter"
 				(path "/3c05686f-5554-4d70-b348-db94545e7981"
-					(reference "R4")
+					(reference "R10")
 					(unit 1)
 				)
@@
 		(dnp no)
 		(fields_autoplaced yes)
-		(property "Reference" "R3"
+		(property "Reference" "R9"
 			(at 153.67 161.29 90)
 			(effects
@@
 			(project "Joule Meter"
 				(path "/3c05686f-5554-4d70-b348-db94545e7981"
-					(reference "R3")
+					(reference "R9")
 					(unit 1)
 				)
@@
 		(on_board yes)
 		(dnp no)
-		(property "Reference" "C3"
+		(property "Reference" "C9"
 			(at 189.23 45.7199 0)
 			(effects
@@
 			(project "Joule Meter"
 				(path "/3c05686f-5554-4d70-b348-db94545e7981"
-					(reference "C3")
+					(reference "C9")
 					(unit 1)
 				)
@@
 		(on_board yes)
 		(dnp no)
-		(property "Reference" "R5"
+		(property "Reference" "R11"
 			(at 166.37 166.116 90)
 			(effects
@@
 			(project "Joule Meter"
 				(path "/3c05686f-5554-4d70-b348-db94545e7981"
-					(reference "R5")
+					(reference "R11")
 					(unit 1)
 				)
@@
 		(dnp no)
 		(fields_autoplaced yes)
-		(property "Reference" "C1"
+		(property "Reference" "C3"
 			(at 64.77 35.5599 0)
 			(effects
@@
 			(project ""
 				(path "/3c05686f-5554-4d70-b348-db94545e7981"
-					(reference "C1")
+					(reference "C3")
 					(unit 1)
 				)
@@
 		(dnp no)
 		(fields_autoplaced yes)
-		(property "Reference" "R2"
+		(property "Reference" "R4"
 			(at 270.51 41.9099 0)
 			(effects
@@
 			(project ""
 				(path "/3c05686f-5554-4d70-b348-db94545e7981"
-					(reference "R2")
+					(reference "R4")
 					(unit 1)
 				)
@@
 		(on_board yes)
 		(dnp no)
-		(property "Reference" "C6"
+		(property "Reference" "C8"
 			(at 29.718 108.204 0)
 			(effects
@@
 			(project ""
 				(path "/3c05686f-5554-4d70-b348-db94545e7981"
-					(reference "C6")
+					(reference "C8")
 					(unit 1)
 				)
@@
 		(on_board yes)
 		(dnp no)
-		(property "Reference" "C7"
+		(property "Reference" "C14"
 			(at 115.57 86.3599 0)
 			(effects
@@
 			(project ""
 				(path "/3c05686f-5554-4d70-b348-db94545e7981"
-					(reference "C7")
+					(reference "C14")
 					(unit 1)
 				)
@@
 		(on_board yes)
 		(dnp no)
-		(property "Reference" "C8"
+		(property "Reference" "C1"
 			(at 283.21 29.2099 90)
 			(effects
@@
 			(project ""
 				(path "/3c05686f-5554-4d70-b348-db94545e7981"
-					(reference "C8")
+					(reference "C1")
 					(unit 1)
 				)
@@
 		(on_board yes)
 		(dnp no)
-		(property "Reference" "C5"
+		(property "Reference" "C12"
 			(at 104.14 147.32 90)
 			(effects
@@
 			(project ""
 				(path "/3c05686f-5554-4d70-b348-db94545e7981"
-					(reference "C5")
+					(reference "C12")
 					(unit 1)
 				)
@@
 		(dnp no)
 		(fields_autoplaced yes)
-		(property "Reference" "C11"
+		(property "Reference" "C7"
 			(at 91.44 107.9499 0)
 			(effects
@@
 			(project ""
 				(path "/3c05686f-5554-4d70-b348-db94545e7981"
-					(reference "C11")
+					(reference "C7")
 					(unit 1)
 				)
@@
 		(on_board yes)
 		(dnp no)
-		(property "Reference" "R12"
+		(property "Reference" "R5"
 			(at 102.616 134.62 0)
 			(effects
@@
 			(project "Joule Meter"
 				(path "/3c05686f-5554-4d70-b348-db94545e7981"
-					(reference "R12")
+					(reference "R5")
 					(unit 1)
 				)
@@
 		(dnp no)
 		(fields_autoplaced yes)
-		(property "Reference" "R7"
+		(property "Reference" "R1"
 			(at 35.56 80.01 90)
 			(effects
@@
 			(project ""
 				(path "/3c05686f-5554-4d70-b348-db94545e7981"
-					(reference "R7")
+					(reference "R1")
 					(unit 1)
 				)
@@
 		(dnp no)
 		(fields_autoplaced yes)
-		(property "Reference" "C2"
+		(property "Reference" "C6"
 			(at 74.93 107.9499 0)
 			(effects
@@
 			(project ""
 				(path "/3c05686f-5554-4d70-b348-db94545e7981"
-					(reference "C2")
+					(reference "C6")
 					(unit 1)
 				)
@@
 		(dnp no)
 		(fields_autoplaced yes)
-		(property "Reference" "R10"
+		(property "Reference" "R2"
 			(at 48.26 80.01 90)
 			(effects
@@
 			(project ""
 				(path "/3c05686f-5554-4d70-b348-db94545e7981"
-					(reference "R10")
+					(reference "R2")
 					(unit 1)
 				)

Commit message: 9-28-2025
Parts:
- removed LMR51610DCBuck1: U1, symbol Joule Meter:LMR51610_DC_Buck
- removed MCP6286T-E/OT1: ~, symbol Joule Meter:MCP6286T-E/OT
- removed TMCS1: ~, symbol Joule Meter:TMCS1107
- removed U4: MCP2551-I-P, Package_DIP:DIP-8_W7.62mm, symbol Interface_CAN_LIN:MCP2551-I-P
- added C11, C15, C18: 0.1μF, symbol Device:C
- added C16, C17: 10μF, symbol Device:C
- added J3: XT60-M, SMV_Connectors:AMASS_XT60-M, symbol Stm 32:XT60-M
- added J4: 22035035, SMV_Connectors:3pin_CON_22035035_MOL, symbol Stm 32:3-pin Mini Molex Spox
- added MCP2562: ~, symbol Joule Meter:MCP2562
- added R13: R_Shunt_US, symbol Device:R_Shunt_US
- added R14: 100kΩ, symbol Device:R_US
- added R15: R_US, symbol Device:R_US
- added TP1, TP10, TP11, TP12, TP13, TP14, TP15, TP16, TP17, TP18, TP19, TP2, TP3, TP4, TP5, TP6, TP7, TP8, TP9: TestPoint, symbol Connector:TestPoint
- added U2: INA240A1PW, Package_SO:TSSOP-8_4.4x3mm_P0.65mm, symbol Amplifier_Current:INA240A1PW
- added U5: MCP6286T-E/OT1, Package_TO_SOT_SMD:SOT-23-5, symbol Amplifier_Operational:MCP6001R
- added U6: LMR36510ADDA, Package_SO:Texas_HTSOP-8-1EP_3.9x4.9mm_P1.27mm_EP2.95x4.9mm_Mask2.4x3.1mm_ThermalVias, symbol Regulator_Switching:LMR36510ADDA
- C14: value 0.1μF -> 8.2pF
- C3: value 4.8μF -> 0.22μF
- C4: value 0.1μF -> 4.7μF
- C5: value 0.1μF -> 1μF
- R1: value 7.2kΩ -> 100kΩ
- R2: value 100kΩ -> 9.09kΩ
- R7: value 660Ω -> 500Ω
- R8: value 622Ω -> 500Ω
- renumbered 0.1μF to 0.1μF1, BLM18AG102SN1D to BLM18AG102SN1D1, Nucleo_F44RE to Nucleo_F44RE1
Connections:
- net +3.3V is gone; now on net +3V3: 0.1μF1.1, BLM18AG102SN1D1.2, C9.1, R7.1, U1.8 (VDD)
- net 3.3V is gone; now on net +3V3: C10.1
- net +5V: now also C15.1, TP4.1; no longer C14.1
- net CS: now also Nucleo_F44RE1.55 (PB6), R15.2, TP15.1; no longer Nucleo_F44RE1.32 (PA4)
- net OUT-Voltage Follower: now also TP8.1, U5.1, U5.4 (-)
- net RXD: now also MCP2562.4 (Rxd)
- net SCLK: now also TP12.1
- net TXD: now also MCP2562.1 (Txd)
- net +3V3: now reaches C5.1
- net +3V3: now also 0.1μF1.2, C1.1, C10.2, C12.2, C13.1, C2.2, C3.1, C4.1, C6.2, C7.2, C8.2, C9.2, J1.N (NEG), J2.2, Nucleo_F44RE1.19 (GND), R2.1, R4.2, R8.2, U1.3 (GND), U3.2 (COMMON), U3.4 (COMMON), C15.2, C16.1, C17.2, C18.1, C18.2, J3.N (NEG), J4.2, MCP2562.2 (Vss), MCP2562.3 (Vdd), MCP2562.5 (VIO), R15.1, TP16.1, TP5.1, TP6.1, U2.1 (GND), U2.4 (GND), U2.5 (V+), U2.6 (REF2), U2.7 (REF1), U5.2 (V+), U5.5 (V-), U6.1 (PGND)
- net at L1.1: now also C14.2, C11.2, U6.8 (SW); no longer C5.2
- net at R7.2, R8.1, U1.6 (AIN2): now also TP11.1
- net at C13.2, R6.2, U1.4 (AIN0): now also TP10.1
- net at J2.3: now also MCP2562.6 (CANL)
- net at J2.1: now also MCP2562.7 (CANH)
- net at R3.2, R4.1: now also TP7.1, U5.3 (+)
- net at C12.1, R5.2, U1.5 (AIN1): now also TP9.1
- net PG: now reaches C6.1, C7.1, L1.2, U3.1 (INPUT)
- net PG: now also R1.2, C16.2, C17.1, R14.1, TP3.1; no longer R2.2
- net DIN renamed DIN (MOSI)
- net DIN (MOSI): now also Nucleo_F44RE1.53 (PA7), TP13.1; no longer Nucleo_F44RE1.51 (PA6)
- net DOUT renamed DOUT (MISO)
- net DOUT (MISO): now also Nucleo_F44RE1.51 (PA6), TP14.1; no longer Nucleo_F44RE1.53 (PA7)
- removed net GND: 0.1μF1.2, C1.1, C10.2, C12.2, C13.1, C14.2, C2.2, C3.2, C4.2, C6.2, C7.2, C8.2, C9.2, J1.N (NEG), J2.2, Nucleo_F44RE1.19 (GND), R1.1, R4.2, R8.2, U1.3 (GND), U3.2 (COMMON), U3.4 (COMMON)
- net Main Power Line- Out: no longer names the net of C1.2, C2.1, J1.P (POS), R3.1
- net Main Power Line- Out: now also R13.1, TP1.1; no longer C3.1, C4.1
- net OUT-Hall Sensor renamed OUT-Current Sense
- net OUT-Current Sense: now also TP19.1, U2.8
- new net: C3.2, C4.2, J3.P (POS), R13.4, TP2.1, U6.2 (VIN), U6.3 (EN)
- new net: C14.1, R1.1, R2.2, U6.5 (FB)
- new net: C11.1, U6.7 (BOOT)
- new net: R14.2, U6.4 (PG)
- new net: R13.2, TP18.1, U2.2 (+)
- new net: R13.3, TP17.1, U2.3 (-)
- new net: C5.2, U6.6 (VCC)
- new net CANN: J4.3
- new net CANP: J4.1
- new net STBY: MCP2562.8 (Stby)
- no-connect marks 70 -> 69
Other:
- moved on the sheet: 0.1μF1, BLM18AG102SN1D1, C12, C13, C6, C7, C8, J2, Nucleo_F44RE1, R10, R11, R12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

Commit message: 9-29-2025
Parts:
- removed C11: 0.1μF, symbol Device:C
- removed C14: 8.2pF, symbol Device:C
- removed C16, C17: 10μF, symbol Device:C
- removed R1, R14: 100kΩ, symbol Device:R_US
- removed TP16, TP17, TP18, TP19: TestPoint, symbol Connector:TestPoint
- added C6: 0.1uF, symbol Device:C
- added C7, C8: 22uF, symbol Device:C
- added R3: 25K, symbol Device:R_US
- 0.1uF: renamed from 0.1μF1; value C11 -> C14
- BLM18AG102SN1D1: value FerriteBead -> FB
- C10: renamed from C7; value 22 μF -> 22 uF
- C11: renamed from C8; value 0.1μF -> 0.1uF
- C12: renamed from C9; value 0.1μF -> 0.1uF
- C15: renamed from C12; value 2.2μF -> 0.1uF
- C16: renamed from C13; value 2.2μF -> 0.1uF
- C18: renamed from C15; value 0.1μF -> 0.1uF
- C3: value 0.22μF -> 2.2uF
- C4: value 4.7μF -> 220nF
- C5: value 1μF -> 0.1uF
- C9: renamed from C6; value 0.33μF -> 0.33uF
- J2, J4: footprint SMV_Connectors:3pin_CON_22035035_MOL -> 3 Pin SMV
- L1: value 68μH -> 100uH
- R10: renamed from R11; value 50Ω -> 50
- R11: renamed from R12; value 50Ω -> 50
- R12: renamed from R15; value R_US -> 5k
- R2: value 9.09kΩ -> 100K
- R4: renamed from R5; value 1000Ω -> 1K
- R5: renamed from R6; value 1000Ω -> 1K
- R6: renamed from R7; value 500Ω -> 500
- R7: renamed from R8; value 500Ω -> 500
- R8: renamed from R9; value 50Ω -> 50
- R9: renamed from R10; value 50Ω -> 50
- renumbered C18 to C13, C10 to C17, J3 to J2, R13 to R1, R3 to R13, R4 to R14, U6 to U1
Connections:
- net CANN is gone; now on net CAN_N: J4.3
- net CANP is gone; now on net CAN_H: J4.1
- net +3V3: now also BLM18AG102SN1D1.1, Nucleo_F44RE1.16 (+3V3), TP7.1; no longer 0.1uF.1, C1.1, C10.2, C11.2, C12.2, C13.2, C15.2, C16.1, C17.2, C18.2, C2.2, C3.1, C4.1, C5.1, C9.2, J1.N (NEG), J2.2, J2.N (NEG), J4.2, MCP2562.2 (Vss), Nucleo_F44RE1.19 (GND), R14.2, R2.1, R7.2, TP5.1, TP6.1, U1.1 (PGND), U1.3 (GND), U2.1 (GND), U2.4 (GND), U2.6 (REF2), U2.7 (REF1), U3.2 (COMMON), U3.4 (COMMON), U5.5 (V-)
- net +5V: now also TP6.1; no longer TP4.1
- net DIN (MOSI): no longer TP13.1
- net DOUT (MISO): no longer TP14.1
- net OUT-Current Sense: now also TP8.1
- net OUT-Voltage Follower: no longer TP8.1
- net RXD: now also TP10.1
- net SCLK: now also TP14.1; no longer TP12.1
- net STBY: now also Nucleo_F44RE1.71 (PA10)
- net TXD: now also TP9.1
- net at C1.2, C2.1, J1.P (POS)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: now also TP2.1
- net at C16.2, R5.2, U1.4 (AIN0): no longer TP10.1
- net at J2.P (POS), R1.4, U1.2 (VIN)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: now also C3.1, C4.1, TP3.1, TP4.1; no longer C3.2, C4.2, TP2.1
- net at R13.2, R14.1, U5.3 (+): now also TP12.1; no longer TP7.1
- net at C15.1, R4.2, U1.5 (AIN1): no longer TP9.1
- net at U1.5 (FB): now also R2.1, R3.1; no longer R2.2
- net at L1.1, U1.8 (SW): now also R2.2, C6.2
- net at U1.7 (BOOT): now also C6.1
- net CAN_H: now reaches J2.1, MCP2562.7 (CANH)
- net CAN_N: now reaches J2.3, MCP2562.6 (CANL)
- net GND: now reaches Nucleo_F44RE1.22 (GND)
- net GND: now also 0.1uF.1, C1.1, C10.2, C11.2, C12.2, C13.2, C15.2, C16.1, C17.2, C18.2, C2.2, C3.2, C4.2, C5.1, C9.2, J1.N (NEG), J2.2, J2.N (NEG), J4.2, MCP2562.2 (Vss), Nucleo_F44RE1.19 (GND), Nucleo_F44RE1.47 (GND), Nucleo_F44RE1.58 (GND), Nucleo_F44RE1.8 (GND), R14.2, R7.2, TP13.1, U1.1 (PGND), U1.3 (GND), U2.1 (GND), U2.4 (GND), U2.6 (REF2), U2.7 (REF1), U3.2 (COMMON), U3.4 (COMMON), U5.5 (V-), C7.2, C8.2, R3.2
- net PG: no longer names the net of C10.1, C9.1, L1.2, U3.1 (INPUT)
- net PG: now also TP5.1, C7.1, C8.1; no longer TP3.1
- no-connect marks 69 -> 64
Other:
- company: Sergio Gonzalez -> by Sergio Gonzalez
- moved on the sheet: 0.1uF, C1, C10, C11, C12, C13, C15, C16, C17, C18, C2, C9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

Commit message: 10-6-2025
Parts:
- added C14: 0.333uF, symbol Device:C
- added TP16: Buck Converter Input, symbol Connector:TestPoint
- added TP17: DOUT (MISO), symbol Connector:TestPoint
- added TP18: DIN (MOSI), symbol Connector:TestPoint
- added TP19: Power - Digital 3V3, symbol Connector:TestPoint
- added TP20: Power-Analog 3V3, symbol Connector:TestPoint
- TP1: value TestPoint -> 48V Main - In
- TP10: value TestPoint -> RXD-Line
- TP11: value TestPoint -> Input - ADC 3V3
- TP12: value TestPoint -> Input - Voltage Follower
- TP13: value TestPoint -> Ground
- TP14: value TestPoint -> OUT-SCLK
- TP15: value TestPoint -> OUT-CS
- TP2: value TestPoint -> 48V Main - Before Shunt
- TP3: value TestPoint -> 48V Main - After Shunt
- TP4: value TestPoint -> 48V Main - Out
- TP5: value TestPoint -> Buck Converter - Output
- TP6: value TestPoint -> LDO-Output
- TP7: value TestPoint -> OUT-Voltage Follower
- TP8: value TestPoint -> O- Current Sense
- TP9: value TestPoint -> TXD Line
- U1: value LMR36510ADDA -> LMR36510
Connections:
- net +3V3: now also TP19.1, TP20.1; no longer TP7.1
- net DIN (MOSI): now also TP18.1
- net DOUT (MISO): now also TP17.1
- net GND: now also Nucleo_F44RE1.20 (GND), Nucleo_F44RE1.70 (AGND), C14.2
- net OUT-Voltage Follower: now also TP7.1
- net at C10.1, C7.1, C8.1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: now also C14.1
- net at C3.1, C4.1, J2.P (POS)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: now also TP16.1
- net CAN_H renamed CANH
- net CAN_N renamed CANL
- no-connect marks 64 -> 62
Other:
- moved on the sheet: C18, C7, C8, TP1, TP12, TP13, TP4, TP8

Commit message: 10-17-2025
Parts:
- removed BLM18AG102SN1D1: FB, symbol Device:FerriteBead
- removed C17: 0.1μF, symbol Device:C
- removed C18: 0.1uF, symbol Device:C
- removed C3: 2.2uF, symbol Device:C
- removed Nucleo_F44RE1: ~, symbol SMV_Custom:STM32_Nucleo_F446RE
- removed R1: R_Shunt_US, symbol Device:R_Shunt_US
- removed R13: 500k, symbol Device:R_US
- removed R14: 20k, symbol Device:R_US
- removed TP10: RXD-Line, symbol Connector:TestPoint
- removed TP11: Input - ADC 3V3, symbol Connector:TestPoint
- removed TP12: Input - Voltage Follower, symbol Connector:TestPoint
- removed TP13: Ground, symbol Connector:TestPoint
- removed TP14: OUT-SCLK, symbol Connector:TestPoint
- removed TP15: OUT-CS, symbol Connector:TestPoint
- removed TP16: Buck Converter Input, symbol Connector:TestPoint
- removed TP17: DOUT (MISO), symbol Connector:TestPoint
- removed TP18: DIN (MOSI), symbol Connector:TestPoint
- removed TP19: Power - Digital 3V3, symbol Connector:TestPoint
- removed TP20: Power-Analog 3V3, symbol Connector:TestPoint
- removed TP3: 48V Main - After Shunt, symbol Connector:TestPoint
- removed TP4: 48V Main - Out, symbol Connector:TestPoint
- removed TP5: Buck Converter - Output, symbol Connector:TestPoint
- removed TP6: LDO-Output, symbol Connector:TestPoint
- removed TP7: OUT-Voltage Follower, symbol Connector:TestPoint
- removed TP8: O- Current Sense, symbol Connector:TestPoint
- removed TP9: TXD Line, symbol Connector:TestPoint
- removed U2: INA240A1PW, Package_SO:TSSOP-8_4.4x3mm_P0.65mm, symbol Amplifier_Current:INA240A1PW
- removed U3: ~, symbol SMV_Custom:UA78M05-Q1
- added C13: 0.33uF, symbol Device:C
- added C15: 0.1uF, symbol Device:C
- added C16: 0.1μF, symbol Device:C
- added C3: 470uF, 63V, SMV_Passives:Big_Chunky_Cap, symbol SMV_Custom:Big_Chunky_Cap2
- added D1: Power_LED, symbol Device:LED
- added FB1: FerriteBead, symbol Device:FerriteBead
- added R0: R_Shunt_US, symbol Device:R_Shunt_US
- added R1: 100K, symbol Device:R_US
- added R4: 20k, symbol Device:R_US
- added U2: ~, symbol SMV_Custom:UA78M05-Q1
- added U3: INA240A1PW, Package_SO:TSSOP-8_4.4x3mm_P0.65mm, symbol Amplifier_Current:INA240A1PW
- 0.1uF: value C14 -> C19
- C10: value 22 uF -> 22uF
- C11: value 0.1uF -> 22uF
- C14: value 0.333uF -> 22 uF
- C4: value 220nF -> 10μF
- C5: value 0.1uF -> 220nF
- C6: value 0.1uF -> 2.2uF
- C7, C8: value 22uF -> 0.1uF
- C9: value 0.33uF -> 0.333uF
- R2: value 100K -> 16K
- R3: value 25K -> 500k
- R5: renamed from R4; value 1K -> 500
- R6: renamed from R5; value 1K -> 500
- R7: renamed from R6; value 500 -> 2k
- R8: renamed from R7; value 500 -> 2k
- TP1: value 48V Main - In -> Ground
- TP2: value 48V Main - Before Shunt -> TestPoint
- renumbered C15 to C17, C16 to C18, J2 to J4, U1 to U4
Connections:
- net STBY is gone; now on net GND: MCP2562.8 (STBY)
- net +3V3: no longer 0.1uF.2, C12.1, MCP2562.3 (Vdd), R12.1, R7.1, U4.8 (VDD), U5.2 (V+)
- net +5V: now also C12.1, D1.2 (A), FB1.1, U2.3 (OUTPUT); no longer C11.1
- net GND: now also C6.1, C7.1, R2.2, TP1.1, C13.2, C15.2, C16.2, C3.1, D1.1 (K), R4.2, U2.2 (COMMON), U2.4 (COMMON), U3.1 (GND), U3.4 (GND), U3.6 (REF2), U3.7 (REF1); no longer C7.2, C8.2, R3.2
- net at C1.2, C2.1, J1.P (POS): now also R3.1, R0.1; no longer TP1.1, TP2.1
- net +7V: now reaches C10.1, C14.1, C9.1, L1.2
- net +7V: now also C11.1, C13.1, R1.2, U2.1 (INPUT); no longer C7.1, C8.1
- net at C4.1, J2.P (POS), U1.2 (VIN)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: now also C5.2, C6.2, C3.2, R0.4
- net FB: now reaches R2.1, U1.5 (FB)
- net FB: now also R1.1; no longer R3.1
- net at L1.1, U1.8 (SW): now also C8.2; no longer C6.2, R2.2
- net at U5.3 (+): now also R3.2, R4.1
- net at U1.7 (BOOT): now also C8.1; no longer C6.1
- net at U1.6 (VCC): now also C7.2; no longer C5.2
- net at U1.4 (PG): now also TP2.1
- net CANH renamed CAN_H
- net CANL renamed CAN_L
- net DIN (MOSI) renamed MOSI
- net DOUT (MISO) renamed MISO
- net OUT-Current Sense renamed Current_Sense
- net Current_Sense: now also U3.8
- net OUT-Voltage Follower renamed Voltage Follower
- net Voltage Follower: no longer R5.1
- net RXD renamed CAN_RXD
- net TXD renamed CAN-TXD
- new net: R0.2, U3.2 (+)
- new net: R0.3, U3.3 (-)
- new net: FB1.2, MCP2562.3 (VDD)
- new net +3V3A: 0.1uF.2, C15.1, C16.1, R7.1, U3.5 (V+), U4.8 (VDD), U5.2 (V+)
- new net +3V3D: R12.1
- new net Voltage_Follower: R5.1
- no-connect marks 62 -> 2
Other:
- added sheet Nucleo_F446RE (Nucleo_F446RE_sch.kicad_sch)
- note added: "Buck Converter - 48V to 7V"
- title: Joule Meter for SMV -> Joule Meter (w/ Currennt Sensor)
- moved on the sheet: C13, C17, C18, J4, MCP2562, R12, R5, R6, R7, R8, U4
