File: smv_lv_fcb/smv_lv_fcb.kicad_sch (KiCad schematic)
At the start: 0 parts

Commit message: adding components
Parts:
- added J1, J5, J6: 430450200, SMV_Connectors:CONN_SD-43045-001_02_MOL, symbol SMV_Custom:430450200
- added J2, J3: 22035035, SMV_Connectors:3pin_CON_22035035_MOL, symbol SMV_Custom:3-pin Mini Molex Spox
- added J4: Molex Micro-Fit 4 Pin, SMV_Connectors:4_pin0430450401, symbol SMV_Custom:Molex Micro-Fit 4 Pin
- added U1: ~, symbol SMV_Custom:STM32_Nucleo_F446RE
