File: Rear_Control_Board_Jason_Liu/Rear_Control_Board_Jason_Liu.kicad_sch (KiCad schematic)
At the start: 85 parts, among them J1 430450200, J10 Front-Control Board, J11 M22-7130442, J2 Molex Micro-Fit 4 Pin, J3 22035035, J4 Low-Power Jouelmeter, J5 430450200, J6 430450200, J7 430450200, J8 430450200, J9 430450200, Q1 PSMN1R8-40YLC_115, Q2 PSMN1R8-40YLC_115, Q3 PSMN1R8-40YLC_115, Q4 PSMN1R8-40YLC_115, U1 UA78M05QDCYRG4Q1, U3 ADS1118QDGSRQ1, U4 MCP2562-E/P, U5 MCP6286T-E/OT, U6 MCP6286T-E/OT, U7 MCP6286T-E/OT, U8 ASM330LHHTR

Commit message: Implemented feedback 1
Parts:
- TP7: value GND1 -> AIN3
Connections:
- net PB5 is gone; now on net CAN_RX: J11.A3, TP15.1, U4.4 (RXD)
- net PB6 is gone; now on net CAN_TX: J11.A4, TP14.1, U4.1 (TXD)
- net +3.3V: now also TP7.1, U2.45 (AVDD), U2.5 (VDD), U3.7 (AIN3)
- net +5V: now also U2.6 (E5V); no longer U2.24 (VIN)
- net GND: now also U2.70 (AGND); no longer TP7.1, U3.7 (AIN3)
- net CAN_RX: now reaches U2.57 (PC7)
- net CAN_TX: now reaches U2.59 (PA9)
- no-connect marks 53 -> 50

Commit message: added parts respository
Parts:
- added J12: 430450200, SMV_Connectors:CONN_SD-43045-001_02_MOL, symbol SMV_Custom:430450200
- added R26, R27, R28, R29, R30, R31, R7: 0 Ohm, SMV_Passives:0805RESC2012X60N, symbol SMV_Custom:CRGCQ0402F47K
- C13: value C0603C103K5RACTU, 10nF -> 10nF; footprint CAPC17595_87N_KEM -> SMV_Passives:Cap0805
- J11: footprint M22-7130442_TYC -> SMV_Connectors:M22-7130442_TYC
- Q1, Q2, Q3, Q4: footprint LFPAK56_SOT669_NEX -> SMV_ICs:LFPAK56_SOT669_NEX
- R1, R15, R17, R3: value CRCW06031K00FKEA, 1KΩ -> 1KΩ
- R10, R6: value CRCW060312K1FKEAC, 12.1k Ohms -> 12.1k Ohms; footprint CRCW060312K1FKEAC:RESC1608X55N -> SMV_Passives:0805RESC2012X60N
- R11, R14, R21, R8: value CRCW020149R9FNED, 50Ω -> 50Ω
- R5, R9: value CRGCQ0402F47K, 47k Ohms -> 47k Ohms; footprint CRGCQ0402F47K:RESC1005X40N -> SMV_Passives:0805RESC2012X60N
- TP1, TP10, TP11, TP12, TP13, TP14, TP15, TP16, TP17, TP18, TP19, TP2, TP20, TP21, TP22, TP23, TP3, TP4, TP5, TP6, TP7, TP8, TP9: footprint (none) -> TestPoint:TestPoint_Pad_D1.0mm
- U2: footprint (none) -> SMV_ICs:MODULE_NUCLEO-F446RE
- U3: footprint DGS0010A_N -> SMV_ICs:DGS0010A_N
- U4: footprint PDIP8_300MC_MCH -> SMV_ICs:PDIP8_300MC_MCH
- U8: footprint LGA-14L_2P5X3X0P83_STM -> SMV_ICs:LGA-14L_2P5X3X0P83_STM
Connections:
- net +3V3 is gone; now on net +3.3V: R19.2, R20.2
- net +12V: now also J12.1
- net +3.3V: now also U2.CN10_7 (AVDD), U2.CN7_16 (+3V3), U2.CN7_5 (VDD), R26.2, R27.2, R28.2, R30.2, R31.1, R7.2; no longer C13.2, C14.2, C3.2, U2.16 (+3V3), U2.45 (AVDD), U2.5 (VDD), U3.8 (VDD), U5.5 (VDD), U6.5 (VDD), U7.5 (VDD), U8.2 (RES), U8.3 (RES), U8.5 (VDD_IO), U8.8 (VDD)
- net +5V: now also U2.CN7_6 (E5V), R29.2; no longer C6.2, U2.6 (E5V), U4.3 (VDD)
- net BL_MOSFET: now also U2.CN7_25 (PC14); no longer U2.37 (PC3)
- net CAN_RX: now also U2.CN10_19 (PC7); no longer U2.57 (PC7)
- net CAN_TX: now also U2.CN10_21 (PA9); no longer U2.59 (PA9)
- net CS_ADC: now also U2.CN10_16 (PB12); no longer U2.32 (PA4)
- net CS_Acc: now also U2.CN7_17 (PA15); no longer U2.17 (PA15)
- net GND: now also U2.CN10_20 (GND), U2.CN10_32 (AGND), U2.CN10_9 (GND), U2.CN7_19 (GND), U2.CN7_20 (GND), U2.CN7_22 (GND), U2.CN7_8 (GND); no longer U2.19 (GND), U2.20 (GND), U2.22 (GND), U2.47 (GND), U2.58 (GND), U2.70 (AGND), U2.8 (GND)
- net TL_MOSFET: now also U2.CN7_29 (PH0); no longer U2.38 (PC0)
- net TSL_MOSFET: now also U2.CN7_13 (PA13); no longer U2.36 (PC1)
- net TSR_MOSFET: now also U2.CN7_15 (PA14); no longer U2.35 (PC2)
- net at J7.2, Q2.5: now also J12.2
- net CAN_N: now reaches J10.3, J4.3, TP12.1, U4.6 (CANL)
- net at R22.2: now also U2.CN10_28 (PB14); no longer U2.51 (PA6)
- net CAN_P: now reaches J10.1, J4.1, TP13.1, U4.7 (CANH)
- net at R21.2: now also U2.CN10_30 (PB13); no longer U2.49 (PA5)
- net at R23.2: now also U2.CN10_26 (PB15); no longer U2.53 (PA7)
- new net: C14.2, R30.1, U8.2 (RES), U8.3 (RES), U8.5 (VDD_IO)
- new net: C6.2, R29.1, U4.3 (VDD)
- new net: C13.2, C3.2, R31.2, U8.8 (VDD)
- new net: R7.1, U3.8 (VDD)
- new net: R27.1, U6.5 (VDD)
- new net: R28.1, U7.5 (VDD)
- new net: R26.1, U5.5 (VDD)
- no-connect marks 50 -> 52
Other:
- moved on the sheet: C11, C7, C9, J11, J7, R21, R22, R23, TP20, TP21, TP22
