File: Rear_Control_Board_Jason_Liu/Rear_Control_Board_Jason_Liu.kicad_sch (KiCad schematic)
At the start: 89 parts, among them J1 430450200, J10 Front-Control Board, J11 M22-7130442, J12 430450200, J2 Molex Micro-Fit 4 Pin, J3 22035035, J4 Low-Power Jouelmeter, J5 430450200, J6 430450200, J7 430450200, J8 430450200, J9 430450200, Q1 PSMN1R8-40YLC_115, Q2 PSMN1R8-40YLC_115, Q3 PSMN1R8-40YLC_115, Q4 PSMN1R8-40YLC_115, U1 UA78M05QDCYRG4Q1, U3 ADS1118QDGSRQ1, U4 MCP2562-E/P, U5 MCP6286T-E/OT, U6 MCP6286T-E/OT, U7 MCP6286T-E/OT, U8 ASM330LHHTR

Commit message: Layout Draft 2
Connections:
- net CAN_RX: now also J11.3; no longer J11.A3
- net CAN_TX: now also J11.4; no longer J11.A4
- net MISO: no longer TP21.1
- net MOSI: no longer TP22.1
- net SCLK: no longer TP20.1
- net at R22.2, U2.CN10_28 (PB14): now also TP21.1
- net at R21.2, U2.CN10_30 (PB13): now also TP20.1
- net at R23.2, U2.CN10_26 (PB15): now also TP22.1
Other:
- moved on the sheet: TP20, TP21, TP22
Changed lines of the file:
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@@
 	)
 	(junction
+		(at 165.1 111.76)
+		(diameter 0)
+		(color 0 0 0 0)
+	)
+	(junction
 		(at 328.93 130.81)
 		(diameter 0)
@@
 	)
 	(junction
+		(at 165.1 106.68)
+		(diameter 0)
+		(color 0 0 0 0)
+	)
+	(junction
 		(at 265.43 72.39)
 		(diameter 0)
@@
 	)
 	(junction
+		(at 165.1 116.84)
+		(diameter 0)
+		(color 0 0 0 0)
+	)
+	(junction
 		(at 46.99 143.51)
 		(diameter 0)
@@
 	(wire
 		(pts
+			(xy 165.1 111.76) (xy 166.37 111.76)
+		)
+		(stroke
+			(width 0)
+			(type default)
+		)
+	)
+	(wire
+		(pts
 			(xy 39.37 41.91) (xy 39.37 46.99)
 		)
@@
 	(wire
 		(pts
+			(xy 165.1 106.68) (xy 166.37 106.68)
+		)
+		(stroke
+			(width 0)
+			(type default)
+		)
+	)
+	(wire
+		(pts
 			(xy 295.91 72.39) (xy 309.88 72.39)
 		)
@@
 	(wire
 		(pts
-			(xy 160.02 106.68) (xy 166.37 106.68)
+			(xy 160.02 106.68) (xy 165.1 106.68)
 		)
 		(stroke
@@
 	(wire
 		(pts
-			(xy 160.02 111.76) (xy 166.37 111.76)
+			(xy 165.1 116.84) (xy 166.37 116.84)
+		)
+		(stroke
+			(width 0)
+			(type default)
+		)
+	)
+	(wire
+		(pts
+			(xy 160.02 111.76) (xy 165.1 111.76)
 		)
 		(stroke
@@
 	(wire
 		(pts
-			(xy 160.02 116.84) (xy 166.37 116.84)
+			(xy 160.02 116.84) (xy 165.1 116.84)
 		)
 		(stroke
@@
 			)
 		)
-		(pin "A1"
+		(pin "4"
 		)
-		(pin "A2"
+		(pin "2"
 		)
-		(pin "A3"
+		(pin "1"
 		)
-		(pin "A4"
+		(pin "3"
 		)
 		(instances
@@
 	(symbol
 		(lib_id "Connector:TestPoint")
-		(at 184.15 111.76 270)
+		(at 165.1 111.76 0)
 		(unit 1)
 		(exclude_from_sim no)
@@
 		(dnp no)
 		(property "Reference" "TP21"
-			(at 185.674 109.982 90)
+			(at 163.322 110.236 90)
 			(effects
 				(font
@@
 		)
 		(property "Value" "MISO"
-			(at 185.42 113.284 90)
+			(at 166.624 110.49 90)
 			(effects
 				(font
@@
 		)
 		(property "Footprint" "TestPoint:TestPoint_Pad_D1.0mm"
-			(at 184.15 116.84 0)
+			(at 170.18 111.76 0)
 			(effects
 				(font
@@
 		)
 		(property "Datasheet" "~"
-			(at 184.15 116.84 0)
+			(at 170.18 111.76 0)
 			(effects
 				(font
@@
 		)
 		(property "Description" "test point"
-			(at 184.15 111.76 0)
+			(at 165.1 111.76 0)
 			(effects
 				(font
@@
 	(symbol
 		(lib_id "Connector:TestPoint")
-		(at 184.15 106.68 270)
+		(at 165.1 106.68 0)
 		(unit 1)
 		(exclude_from_sim no)
@@
 		(fields_autoplaced yes)
 		(property "Reference" "TP22"
-			(at 189.23 105.4099 90)
+			(at 167.64 102.1079 0)
 			(effects
 				(font
@@
 		)
 		(property "Value" "MOSI"
-			(at 189.23 107.9499 90)
+			(at 167.64 104.6479 0)
 			(effects
 				(font
@@
 		)
 		(property "Footprint" "TestPoint:TestPoint_Pad_D1.0mm"
-			(at 184.15 111.76 0)
+			(at 170.18 106.68 0)
 			(effects
 				(font
@@
 		)
 		(property "Datasheet" "~"
-			(at 184.15 111.76 0)
+			(at 170.18 106.68 0)
 			(effects
 				(font
@@
 		)
 		(property "Description" "test point"
-			(at 184.15 106.68 0)
+			(at 165.1 106.68 0)
 			(effects
 				(font
@@
 	(symbol
 		(lib_id "Connector:TestPoint")
-		(at 184.15 116.84 270)
+		(at 165.1 116.84 180)
 		(unit 1)
 		(exclude_from_sim no)
@@
 		(dnp no)
 		(property "Reference" "TP20"
-			(at 185.42 115.57 90)
+			(at 166.37 118.11 90)
 			(effects
 				(font
@@
 		)
 		(property "Value" "SCLK"
-			(at 184.912 119.126 90)
+			(at 162.814 117.602 90)
 			(effects
 				(font
@@
 		)
 		(property "Footprint" "TestPoint:TestPoint_Pad_D1.0mm"
-			(at 184.15 121.92 0)
+			(at 160.02 116.84 0)
 			(effects
 				(font
@@
 		)
 		(property "Datasheet" "~"
-			(at 184.15 121.92 0)
+			(at 160.02 116.84 0)
 			(effects
 				(font
@@
 		)
 		(property "Description" "test point"
-			(at 184.15 116.84 0)
+			(at 165.1 116.84 0)
 			(effects
 				(font

Commit message: Implemented feedbacks from 1/5
Parts:
- removed TP12: CAN_N, TestPoint:TestPoint_Pad_D1.0mm, symbol Connector:TestPoint
- removed TP13: CAN_P, TestPoint:TestPoint_Pad_D1.0mm, symbol Connector:TestPoint
- added D1, D2, D3, D4, D5, D6, D7: WL-SMCW_0603, SMV_Passives:WL-SMCW_0603(diode), symbol SMV_Custom:WL-SMCW_0603
- added R32, R33, R34: 10kohms, 0.125W, SMV_Passives:0805RESC2012X60N, symbol SMV_Custom:CRCW080510K0FKEAC
Connections:
- net +12V: now also R32.2
- net +3.3V: now also R34.2
- net +5V: now also R33.1; no longer U2.CN7_18 (+5V)
- net GND: now also D1.1, D2.1, D3.1, D4.1, D5.1, D6.1, D7.1
- net at Q3.4, R15.2, R16.1: now also D7.2
- net at Q2.4, R3.2, R4.1: now also D5.2
- net at Q4.4, R17.2, R18.1: now also D6.2
- net at Q1.4, R1.2, R2.1: now also D4.2
- new net: D2.2, R33.2
- new net: D1.2, R32.1
- new net: D3.2, R34.1
- no-connect marks 52 -> 50

Commit message: 1/13 Update
Parts:
- U4: footprint SMV_ICs:PDIP8_300MC_MCH -> MCP2562-E/MF:SOIC127P600X175-8N
Changed lines of the file:
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@@
 	(wire
 		(pts
-			(xy 326.39 133.35) (xy 326.39 146.05)
-		)
-		(stroke
-			(width 0)
-			(type default)
-		)
-	)
-	(wire
-		(pts
 			(xy 113.03 172.72) (xy 118.11 172.72)
 		)
@@
 	(wire
 		(pts
+			(xy 326.39 133.35) (xy 326.39 146.05)
+		)
+		(stroke
+			(width 0)
+			(type default)
+		)
+	)
+	(wire
+		(pts
 			(xy 105.41 96.52) (xy 109.22 96.52)
 		)
@@
 	)
 	(symbol
+		(lib_id "SMV_Custom:MCP2562-E_P")
+		(at 265.43 125.73 0)
+		(unit 1)
+		(exclude_from_sim no)
+		(in_bom yes)
+		(on_board yes)
+		(dnp no)
+		(fields_autoplaced yes)
+		(property "Reference" "U4"
+			(at 295.91 115.57 0)
+			(effects
+				(font
+					(size 1.524 1.524)
+				)
+			)
+		)
+		(property "Value" "MCP2562-E/P"
+			(at 295.91 118.11 0)
+			(effects
+				(font
+					(size 1.524 1.524)
+				)
+			)
+		)
+		(property "Footprint" "MCP2562-E/MF:SOIC127P600X175-8N"
+			(at 265.43 125.73 0)
+			(effects
+				(font
+					(size 1.27 1.27)
+					(italic yes)
+				)
+				(hide yes)
+			)
+		)
+		(property "Datasheet" "MCP2562-E/P"
+			(at 265.43 125.73 0)
+			(effects
+				(font
+					(size 1.27 1.27)
+					(italic yes)
+				)
+				(hide yes)
+			)
+		)
+		(property "Description" ""
+			(at 265.43 125.73 0)
+			(effects
+				(font
+					(size 1.27 1.27)
+				)
+				(hide yes)
+			)
+		)
+		(pin "2"
+		)
+		(pin "3"
+		)
+		(pin "6"
+		)
+		(pin "8"
+		)
+		(pin "4"
+		)
+		(pin "5"
+		)
+		(pin "7"
+		)
+		(pin "1"
+		)
+		(instances
+			(project ""
+				(path "/866fd9fd-9057-4f06-b5ac-cc23ee87995f"
+					(reference "U4")
+					(unit 1)
+				)
+			)
+		)
+	)
+	(symbol
 		(lib_id "power:GND")
 		(at 95.25 38.1 180)
@@
 					(unit 1)
 				)
-			)
-		)
-	)
-	(symbol
-		(lib_id "SMV_Custom:MCP2562-E_P")
-		(at 265.43 125.73 0)
-		(unit 1)
-		(exclude_from_sim no)
-		(in_bom yes)
-		(on_board yes)
-		(dnp no)
-		(fields_autoplaced yes)
-		(property "Reference" "U4"
-			(at 295.91 115.57 0)
-			(effects
-				(font
-					(size 1.524 1.524)
-				)
-			)
-		)
-		(property "Value" "MCP2562-E/P"
-			(at 295.91 118.11 0)
-			(effects
-				(font
-					(size 1.524 1.524)
-				)
-			)
-		)
-		(property "Footprint" "SMV_ICs:PDIP8_300MC_MCH"
-			(at 265.43 125.73 0)
-			(effects
-				(font
-					(size 1.27 1.27)
-					(italic yes)
-				)
-				(hide yes)
-			)
-		)
-		(property "Datasheet" "MCP2562-E/P"
-			(at 265.43 125.73 0)
-			(effects
-				(font
-					(size 1.27 1.27)
-					(italic yes)
-				)
-				(hide yes)
-			)
-		)
-		(property "Description" ""
-			(at 265.43 125.73 0)
-			(effects
-				(font
-					(size 1.27 1.27)
-				)
-				(hide yes)
-			)
-		)
-		(pin "3"
-		)
-		(pin "5"
-		)
-		(pin "6"
-		)
-		(pin "2"
-		)
-		(pin "4"
-		)
-		(pin "8"
-		)
-		(pin "7"
-		)
-		(pin "1"
-		)
-		(instances
-			(project ""
-				(path "/866fd9fd-9057-4f06-b5ac-cc23ee87995f"
-					(reference "U4")
-					(unit 1)
-				)
