File: Rear_Control_Board_Jason_Liu/Rear_Control_Board_Jason_Liu.kicad_pcb (KiCad board)
At the start: 2 copper layers, 252.5 x 141 mm, 85 parts, among them J1 430450200, J10 Front-Control Board, J11 M22-7130442, J2 Molex Micro-Fit 4 Pin, J3 22035035, J4 Low-Power Jouelmeter, J5 430450200, J6 430450200, J7 430450200, J8 430450200, J9 430450200, Q1 PSMN1R8-40YLC_115, Q2 PSMN1R8-40YLC_115, Q3 PSMN1R8-40YLC_115, Q4 PSMN1R8-40YLC_115, U1 UA78M05QDCYRG4Q1, U3 ADS1118QDGSRQ1, U4 MCP2562-E/P, U5 MCP6286T-E/OT, U6 MCP6286T-E/OT, U7 MCP6286T-E/OT, U8 ASM330LHHTR

Commit message: PCB first draft
Parts:
- removed TP11: P_ADC, TestPoint:TestPoint_Pad_D1.0mm
- removed TP17: T_N_ADC, TestPoint:TestPoint_Pad_D1.0mm
- removed TP18: T_P_ADC, TestPoint:TestPoint_Pad_D1.0mm
- removed TP7: AIN3, TestPoint:TestPoint_Pad_D1.0mm
- added J12: 430450200, SMV_Connectors:CONN_SD-43045-001_02_MOL, F.Cu at (105.1, 94.6)
- added R26: 0 Ohm, SMV_Passives:0805RESC2012X60N, F.Cu at (211.8, 58.8)
- added R27: 0 Ohm, SMV_Passives:0805RESC2012X60N, F.Cu at (196.5, 59.2)
- added R28: 0 Ohm, SMV_Passives:0805RESC2012X60N, F.Cu at (200.3, 89.0)
- added R29: 0 Ohm, SMV_Passives:0805RESC2012X60N, F.Cu at (137.4, 113.7)
- added R30: 0 Ohm, SMV_Passives:0805RESC2012X60N, F.Cu at (202.2, 74.2)
- added R31: 0 Ohm, SMV_Passives:0805RESC2012X60N, F.Cu at (217.2, 73.1)
- added R7: 0 Ohm, SMV_Passives:0805RESC2012X60N, F.Cu at (197.2, 67.8)
- moved TP1 290.8 mm to (103.2, 47.6)
- moved TP13 284.0 mm to (128.7, 134.4)
- moved TP4 282.1 mm to (113.9, 93.4)
- moved TP5 282.0 mm to (112.0, 63.5)
- moved TP6 281.2 mm to (113.0, 77.3)
- moved TP3 281.1 mm to (117.6, 108.4)
- moved TP12 275.7 mm to (128.7, 129.3)
- moved TP15 248.0 mm to (157.9, 110.4)
- moved TP14 234.2 mm to (172.6, 109.5)
- moved TP8 221.0 mm to (184.6, 114.9)
- moved TP20 212.1 mm to (192.2, 76.1)
- moved TP21 211.9 mm to (191.7, 70.2)
- moved TP22 211.4 mm to (192.1, 72.7)
- moved TP10 207.9 mm to (192.1, 94.7)
- moved TP19 204.4 mm to (200.7, 78.8)
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Connections:
- net Net-(U4-CANH) renamed /CAN_P
- net Net-(U4-CANL) renamed /CAN_N
- C13 pad 2: +3.3V -> Net-(U8-VDD)
- C14 pad 2: +3.3V -> Net-(U8-VDD_IO)
- C3 pad 2: +3.3V -> Net-(U8-VDD)
- C6 pad 2: +5V -> Net-(U4-VDD)
- J11 pad 1: (no net) -> unconnected-(J11-Pad1)
- J11 pad 2: (no net) -> unconnected-(J11-Pad2)
- J11 pad 3: (no net) -> /CAN_RX
- J11 pad 4: (no net) -> /CAN_TX
- R19 pad 2: +3V3 -> +3.3V
- R20 pad 2: +3V3 -> +3.3V
- R21 pad 2: Net-(U2-PA5) -> Net-(U2-PB13)
- R22 pad 2: Net-(U2-PA6) -> Net-(U2-PB14)
- R23 pad 2: Net-(U2-PA7) -> Net-(U2-PB15)
- U1 pad 1: +5V -> +12V
- U1 pad 3: +12V -> +5V
- U2 pad CN10_11: Net-(U2-PA5) -> unconnected-(U2-PA5-PadCN10_11)
- U2 pad CN10_13: Net-(U2-PA6) -> unconnected-(U2-PA6-PadCN10_13)
- U2 pad CN10_15: Net-(U2-PA7) -> unconnected-(U2-PA7-PadCN10_15)
- U2 pad CN10_16: unconnected-(U2-PB12-PadCN10_16) -> /CS_ADC
- U2 pad CN10_19: /CAN_RX -> unconnected-(U2-PC7-PadCN10_19)
- U2 pad CN10_21: /CAN_TX -> unconnected-(U2-PA9-PadCN10_21)
- U2 pad CN10_26: unconnected-(U2-PB15-PadCN10_26) -> Net-(U2-PB15)
- U2 pad CN10_28: unconnected-(U2-PB14-PadCN10_28) -> Net-(U2-PB14)
- U2 pad CN10_30: unconnected-(U2-PB13-PadCN10_30) -> Net-(U2-PB13)
- U2 pad CN10_35: unconnected-(U2-PA2-PadCN10_35) -> /CAN_TX
- U2 pad CN10_37: unconnected-(U2-PA3-PadCN10_37) -> /CAN_RX
- U2 pad CN10_5: unconnected-(U2-PB9-PadCN10_5) -> /CS_Acc
- U2 pad CN7_17: /CS_Acc -> unconnected-(U2-PA15-PadCN7_17)
- U2 pad CN7_18: unconnected-(U2-+5V-PadCN7_18) -> +5V
- U2 pad CN7_32: /CS_ADC -> unconnected-(U2-PA4-PadCN7_32)
- U3 pad 8: +3.3V -> Net-(U3-VDD)
- U4 pad 3: +5V -> Net-(U4-VDD)
- U5 pad 5: +3.3V -> Net-(U5-VDD)
- U6 pad 5: +3.3V -> Net-(U6-VDD)
- U7 pad 5: +3.3V -> Net-(U7-VDD)
- U8 pad 2: +3.3V -> Net-(U8-VDD_IO)
- U8 pad 3: +3.3V -> Net-(U8-VDD_IO)
- U8 pad 5: +3.3V -> Net-(U8-VDD_IO)
- U8 pad 8: +3.3V -> Net-(U8-VDD)
Routing:
- net +3.3V: track 126.8 -> 298.2 mm, vias 2 -> 3
- net +5V: track 37.9 -> 181.6 mm
- net GND: track 0.00 -> 100.3 mm, vias 0 -> 32
- net /CAN_RX: track 0.00 -> 64.5 mm
- net /CAN_P: track 0.00 -> 48.7 mm
- net /CAN_N: track 0.00 -> 48.6 mm
- net /CAN_TX: track 0.00 -> 38.1 mm
- net /CS_Acc: track 0.00 -> 29.4 mm, vias 0 -> 1
- net Net-(U2-PB14): track 0.00 -> 26.2 mm
- net Net-(U2-PB15): track 0.00 -> 26.1 mm
- net Net-(U2-PB13): track 0.00 -> 26.1 mm
- net /P_Sensor_ADC: track 2.52 -> 25.2 mm, vias 0 -> 2
- net /T_Sensor_ADC_N: track 34.0 -> 16.6 mm
- net /MOSI: track 5.80 -> 23.0 mm, vias 0 -> 2
- net /P_Sensor: track 0.00 -> 16.8 mm
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- added copper zone on B.Cu, net GND
- added copper zone on F.Cu, net GND
Other:
- board size 252.5 x 141 mm -> 135 x 120 mm
- board text added: "*"

Commit message: Layout Draft 2
Parts:
- moved TP20 11.6 mm to (189.4, 87.4)
- moved TP22 10.5 mm to (189.3, 82.8)
- moved TP2 6.07 mm to (189.1, 70.2)
- moved R21 5.71 mm to (194.2, 74.8), turned to 180 degrees
- moved R23 5.31 mm to (194.2, 72.7), turned to 180 degrees
- moved R22 5.26 mm to (194.2, 70.6), turned to 180 degrees
- moved TP21 5.25 mm to (189.0, 74.7)
- moved TP12 0.10 mm to (128.7, 129.4)
Connections:
- TP20 pad 1: /SCLK -> Net-(U2-PB13)
- TP21 pad 1: /MISO -> Net-(U2-PB14)
- TP22 pad 1: /MOSI -> Net-(U2-PB15)
Routing:
- net +3.3V: track 298.2 -> 270.3 mm, vias 3 -> 6
- net GND: track 100.3 -> 111.3 mm, vias 32 -> 31
- net /MOSI: track 23.0 -> 15.6 mm, vias 2 -> 0
- net /SCLK: track 24.6 -> 31.2 mm, vias 2 -> 0
- net Net-(U2-PB14): track 26.2 -> 28.7 mm
- net /CAN_N: track 48.6 -> 51.1 mm
- net Net-(U2-PB15): track 26.1 -> 28.5 mm
- net Net-(U2-PB13): track 26.1 -> 28.3 mm
- net /CAN_P: track 48.7 -> 50.8 mm
- net /T_Sensor_ADC_N: track 16.6 -> 18.4 mm, vias 0 -> 2
- net /MISO: track 22.7 -> 21.4 mm, vias 2 -> 0
- net /T_Sensor_ADC_P: track 24.8 -> 24.9 mm, vias 0 -> 2
- net /CS_ADC: vias 0 -> 1
- added copper zone on B.Cu, net +3.3V

Commit message: Implemented feedbacks from 1/5
Parts:
- removed TP12: CAN_N, TestPoint:TestPoint_Pad_D1.0mm
- removed TP13: CAN_P, TestPoint:TestPoint_Pad_D1.0mm
- added D1: WL-SMCW_0603, SMV_Passives:WL-SMCW_0603(diode), F.Cu at (95.9, 35.0)
- added D2: WL-SMCW_0603, SMV_Passives:WL-SMCW_0603(diode), F.Cu at (105.1, 50.2)
- added D3: WL-SMCW_0603, SMV_Passives:WL-SMCW_0603(diode), F.Cu at (115.6, 40.8)
- added D4: WL-SMCW_0603, SMV_Passives:WL-SMCW_0603(diode), F.Cu at (112.4, 117.7)
- added D5: WL-SMCW_0603, SMV_Passives:WL-SMCW_0603(diode), F.Cu at (111.9, 93.0)
- added D6: WL-SMCW_0603, SMV_Passives:WL-SMCW_0603(diode), F.Cu at (109.2, 63.4)
- added D7: WL-SMCW_0603, SMV_Passives:WL-SMCW_0603(diode), F.Cu at (109.9, 77.1)
- added R32: 10kohms, 0.125W, SMV_Passives:0805RESC2012X60N, F.Cu at (99.6, 35.0)
- added R33: 10kohms, 0.125W, SMV_Passives:0805RESC2012X60N, F.Cu at (105.2, 48.3)
- added R34: 10kohms, 0.125W, SMV_Passives:0805RESC2012X60N, F.Cu at (115.4, 45.9)
- moved R12 5.62 mm to (192.0, 92.3), turned to -90 degrees
- moved TP1 3.59 mm to (102.4, 44.1)
- moved R13 2.13 mm to (194.2, 92.3)
- moved TP19 1.78 mm to (199.3, 79.9)
- moved TP5 1.61 mm to (113.4, 64.3)
- moved R2 1.20 mm to (112.4, 113.9), turned to 90 degrees
- moved TP10 1.20 mm to (192.2, 95.9)
- moved TP6 1.20 mm to (112.1, 78.1)
- moved R4 1.20 mm to (112.3, 89.5), turned to 90 degrees
- moved R18 1.03 mm to (112.0, 61.5), turned to 90 degrees
- moved R16 1.03 mm to (112.1, 75.3), turned to 90 degrees
- moved R3 0.94 mm to (115.3, 89.5), turned to 90 degrees
- moved R15 0.93 mm to (115.0, 75.3), turned to 90 degrees
- moved R17 0.90 mm to (115.0, 61.5), turned to 90 degrees
- moved R1 0.81 mm to (115.1, 113.9), turned to 90 degrees
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Connections:
- U2 pad CN7_18: +5V -> unconnected-(U2-+5V-PadCN7_18)
Routing:
- net /CS_ADC: track 12.3 -> 56.5 mm, vias 1 -> 0
- net GND: track 111.3 -> 68.7 mm, vias 31 -> 84
- net /T_Sensor_ADC_N: track 18.4 -> 50.8 mm, vias 2 -> 0
- net /T_Sensor_ADC_P: track 24.9 -> 40.8 mm, vias 2 -> 0
- net /CS_Acc: track 29.4 -> 44.2 mm, vias 1 -> 0
- net /P_Sensor: track 16.8 -> 9.04 mm
- net /CAN_N: track 51.1 -> 43.6 mm
- net +3.3V: track 270.3 -> 277.8 mm, vias 6 -> 8
- net /CAN_P: track 50.8 -> 43.7 mm
- net Net-(J9-Pad2): track 5.42 -> 0.00 mm
- net Net-(J8-Pad2): track 5.37 -> 0.00 mm
- net Net-(J6-Pad2): track 5.12 -> 0.00 mm
- net Net-(J12-Pad2): track 16.9 -> 12.0 mm
- net Net-(D6-Pad2): track 4.17 -> 8.89 mm
- net /TSL_MOSFET: track 19.0 -> 14.6 mm
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- added copper zone on F.Cu, net (none)
Other:
- board text added: "+"
- board text removed: "*"

Commit message: 1/13 Update
Parts:
- U4: footprint SMV_ICs:PDIP8_300MC_MCH -> MCP2562-E/MF:SOIC127P600X175-8N
- moved U4 4.64 mm to (149.1, 116.6)
- moved TP14 4.53 mm to (172.1, 114.0)
- moved J4 0.28 mm to (162.1, 134.3)
Routing:
- net /CAN_RX: track 64.5 -> 40.2 mm
- net +12V: track 188.1 -> 195.1 mm
- net /CAN_TX: track 38.1 -> 44.1 mm
- net +3.3V: track 277.8 -> 280.5 mm
- net /CAN_P: track 43.7 -> 45.3 mm
- net /CAN_N: track 43.6 -> 45.2 mm
- net Net-(U4-VDD): track 10.4 -> 11.9 mm
- net GND: vias 84 -> 83

Commit message: Final Board Draft (I think)
Parts:
- added GND: 5V1, TestPoint:TestPoint_Pad_D1.0mm, F.Cu at (197.4, 113.4)
- added REF**: SEM_logo, SMV_Logo:SEM_logo, F.Cu at (209.9, 34.8)
- moved J10 87.0 mm to (219.5, 109.7), turned to 0 degrees
- moved C4 79.5 mm to (218.5, 103.4)
- moved J4 73.7 mm to (219.5, 88.2), turned to 0 degrees
- moved C6 72.0 mm to (212.2, 103.4), turned to 180 degrees
- moved R29 71.4 mm to (208.3, 104.9), turned to -90 degrees
- moved U4 68.1 mm to (214.9, 98.9), turned to 0 degrees
- moved J11 62.9 mm to (208.3, 101.8), turned to 90 degrees
- moved CAN_RX 49.6 mm to (205.8, 97.6)
- moved CAN_TX 25.7 mm to (189.2, 94.8)
- moved 5V 23.6 mm to (204.5, 102.2)
- moved D1 23.5 mm to (116.8, 24.3), turned to 90 degrees
- moved R32 16.7 mm to (112.6, 24.5), turned to 180 degrees
- moved D4 3.72 mm to (109.4, 115.5), turned to 0 degrees
- renumbered TP1 to 12V, TP8 to 5V, TP4 to BL_MOSFET, TP15 to CAN_RX, TP14 to CAN_TX, TP19 to CS_ADC, TP10 to P_Sensor, TP3 to TL_MOSFET, TP6 to TSR_M, TP9 to TS_N, TP16 to TS_P
Routing:
- net +12V: track 195.1 -> 0.00 mm
- net +3.3V: track 280.5 -> 238.4 mm
- net +5V: track 182.6 -> 155.1 mm
- net /CAN_P: track 45.3 -> 26.7 mm
- net /CAN_N: track 45.2 -> 26.8 mm
- net /CAN_TX: track 44.1 -> 37.7 mm
- net /CAN_RX: track 40.2 -> 34.7 mm
- net GND: track 68.7 -> 71.7 mm, vias 83 -> 65
- net Net-(U4-VDD): track 11.9 -> 10.4 mm
- added copper zone on F.Cu, net +12V
Other:
- board size 135 x 120 mm -> 130 x 97 mm
- board text added: "Jason Liu 1/18/26 Rear Control Board"
- board text added: "MISO"
- board text added: "MOSI"
- board text added: "SCLK"
