File: Safety_Board_Kavish_Shah/Safety_Board_Kavish_Shah.kicad_sch (KiCad schematic)
At the start: 0 parts

Commit message: Complted schematic design
Parts:
- added C1: 22uF, symbol Device:C_US
- added C2: 0.33uF, symbol Device:C_US
- added C3: 0.1uF, symbol Device:C_US
- added C4: 0.1uF, symbol Device:C_Small
- added C5: 0.1uF, symbol Device:C
- added C6: C, symbol Device:C
- added D1: 1N4148WT, Diode_SMD:D_SOD-523, symbol Diode:1N4148WT
- added J1, J4: XT60-M, SMV_Connectors:AMASS_XT60-M, symbol SMV_Custom:XT60-M
- added J2: 430450200, SMV_Connectors:CONN_SD-43045-001_02_MOL, symbol SMV_Custom:430450200
- added J3: TGS2611-C00, TGS2611-C00:TO180P920X780-4P, symbol TGS2611-C00:TGS2611-C00
- added K1: Fujitsu_FTR-LYAA005x, Relay_THT:Relay_SPST-NO_Fujitsu_FTR-LYAA005x_FormA_Vertical, symbol Relay:Fujitsu_FTR-LYAA005x
- added L1, L2: L, symbol Device:L
- added Q1: MOSFET, IRLML6344TRPBF:TRANS_IRLML6344TRPBF, symbol SMV_Custom:MOSFET
- added R1, R2: 1.2k, symbol Device:R
- added R3: 10k, symbol Device:R
- added R4, R6: 100k, symbol Device:R
- added R5: 5.23k, symbol Device:R
- added R7: 15.4k, symbol Device:R
- added U1: ~, symbol SMV_Custom:STM32_Nucleo_F446RE
- added U2: MCP2562-E/P, PDIP8_300MC_MCH, symbol SMV_Custom:CAN Transceiver
- added U3: MCP6286T-E/OT, SMV_ICs:SOT-23-5_MC_MCH, symbol SMV_Custom:MCP6286T-E_OT
- added U4: 74LVC1G08, symbol 74xGxx:74LVC1G08
- added U5, U6: AP66200FVBW-13, U-QFN4040-16/SWP_UXB_DIO, symbol Buck_Converter:AP66200FVBW-13
- added U7: SN78MCDCYR, DCY0004A_N, symbol 2025-12-26_21-13-59:SN78MCDCYR
Connections:
- new net: R4.1, R5.1, U6.15 (FB)
- new net: U1.50 (PA12), U2.1 (TXD)
- new net: U1.52 (PA11), U2.4 (RXD)
- new net: C5.1, U5.5 (BST)
- new net: C5.2, L2.1, U5.6 (SW)
- new net: J3.3 (VC+), R2.1, U3.4 (VIN-)
- new net: L2.2, R6.2
- new net: J1.P (POS), U5.3 (VIN), U5.4 (VIN)
- new net: D1.2 (A), K1.A2, Q1.3
- new net: L1.2, R4.2
- new net: R6.1, R7.1, U5.15 (FB)
- new net: C4.1, U6.5 (BST)
- new net: C4.2, L1.1, U6.6 (SW)
- new net: R3.1, U4.2
- new net +12V: C1.1, D1.1 (K), K1.A1, U6.3 (VIN), U6.4 (VIN)
- new net +3.3V: C3.2, J2.1, J3.1 (VH@1), J3.4 (VH@2), R1.1, U3.3 (VIN+), U3.5 (VDD), U4.5 (VCC), U7.3 (OUTPUT)
- new net +55V: J4.P (POS), K1.14
- new net +5V: C2.1, U2.3 (VDD), U5.7 (SW), U7.1 (INPUT)
- new net GND: C1.2, C2.2, C3.1, C6.2, J1.N (NEG), J4.N (NEG), Q1.2, R1.2, R2.2, R3.2, R5.2, R7.2, U3.2 (VSS), U4.3 (GND), U5.16 (GND), U5.9 (PGND), U6.16 (GND), U6.9 (PGND), U7.2 (COMMON), U7.4 (COMMON)
