File: 1-5-26/UIBoard PHONE&DONLD.kicad_sch (KiCad schematic)
At the start: 84 parts, among them J1 XT60-M, J2 XT60-M, J5 M22-7130442, J7 22035035, Q1 2N3904, Q2 2N3904, Q3 2N3904, Q4 2N3904, SW1 A8L-11-12N1, U1 UA78M05-Q1, U2 MCP2562-E-P, U3 CD4511BPWR, U5 7 Segment Display, U6 STM32 Nucleo F446RE, U7 PCF8574AP

Commit message: Fixed nets for STM32 and 7 Segment Display
Parts:
- RV2: footprint SMV_Passives:0805RESC2012X60N -> Potentiometer_SMD:Potentiometer_ACP_CA6-VSMD_Vertical
Changed lines of the file:
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@@
 			)
 		)
-		(property "Footprint" "SMV_Passives:0805RESC2012X60N"
+		(property "Footprint" "Potentiometer_SMD:Potentiometer_ACP_CA6-VSMD_Vertical"
 			(at 236.22 105.41 0)
 			(effects
