File: UI_Board_Evan_Matsunaga/UI_Board_Evan_Matsunaga/Untitled/Untitled.kicad_sch (KiCad schematic)
At the start: 36 parts, among them J1 22035035, J2 XT60-M, Q1 Q_NPN, Q2 Q_NPN, Q3 Q_NPN, Q4 Q_NPN, SW1 A8L-11-12N1, U2 MCP2562-E-P, U4 NHD-0420H1Z, U7 UA78M05QDCYRQ1

Commit message: edits
Parts:
- removed B1: ~, SMV_Misc:Twidec Button, symbol SMV_Custom:Twidec_Button
- removed D1, D2: 0.1µF, symbol Device:D_Capacitance
- removed Q1, Q2, Q3, Q4: Q_NPN, symbol Device:Q_NPN
- removed R1: 18Ω, symbol Device:R
- removed R10, R11, R8, R9: 220Ω, symbol Device:R
- removed R12, R13, R14, R15: 10kΩ, symbol Device:R
- removed R2: 100kΩ, symbol Device:R
- removed R3: 33kΩ, symbol Device:R
- added Button_Extra: ~, SMV_Misc:Twidec Button, symbol SMV_Custom:Twidec_Button
- added C1, C3, C4: 0.1µF, symbol Device:C
- added C2: 1µF, symbol Device:C
- added Q4, Q6, Q7, Q8: MMBT3904, Package_TO_SOT_SMD:SOT-23, symbol Transistor_BJT:MMBT3904
- added R16, R17, R18, R19, R20, R21, R22, R23, R24, R25, R26, R27, R35: 10k, symbol Device:R
- added R27, R28, R29, R30, R31, R32, R33, R34: 220Ω, symbol Device:R
- added RV1: 10k, symbol Device:R_Potentiometer
- added Switch_Extra, Switch_Signal, Switch_Wipers: ~, SMV_Misc:TAISS 3 Pin Switch, symbol SMV_Custom:TAISS_3_Pin_Switch
- R4, R5, R6: value 220Ω -> 10k
- R7: value 220Ω -> 120Ω
- renumbered B3 to Button_Hazards, B2 to Button_Horn, SW1 to SW_Ignition, S1 to Switch_Lights
Connections:
- net BAT+ is gone; now on net GND: SW_Ignition.1
- net VIN_SW is gone; now on net SW_IGNITION: SW_Ignition.2
- net +3.3V: now also A1.2 (3V3), C1.1, C4.1, R16.2, R17.2, R18.2, R19.2, R20.2, R21.2, R22.2, R23.2, R24.2, R25.2, R26.2, R27.2; no longer U4.15 (A)
- net +5V: now also U1.6 (E5V), C3.2; no longer A1.26 (USB), J2.P (POS)
- net DIG1_CTRL: now also R35.2
- net DIG2_CTRL: now also R4.2
- net DIG3_CTRL: now also R5.2
- net DIG4_CTRL: now also R6.2
- net GND: now also U1.22 (GND), U1.47 (GND), U1.70 (AGND), U1.8 (GND), Button_Extra.1, C2.1, C3.1, C4.2, Q4.2 (E), Q6.2 (E), Q7.2 (E), Q8.2 (E), Switch_Extra.2 (Center), Switch_Signal.2 (Center), Switch_Wipers.2 (Center); no longer U4.3 (VO)
- net LIGHT_HI: now also R19.1
- net SEG_A_DRV: now also R27.1; no longer R4.1
- net SEG_B_DRV: now also R28.1; no longer R7.2
- net SEG_C_DRV: now also R29.1
- net SEG_DP_DRV: now also R34.1
- net SEG_D_DRV: now also R30.1
- net SEG_E_DRV: now also R31.1
- net SEG_F_DRV: now also R32.2; no longer R5.1
- net SEG_G_DRV: now also R33.2; no longer R6.1
- net at U5.1 (E): now also R31.2
- net at U5.10 (F): now also R32.1; no longer R5.2
- net at U5.11 (G): now also R33.1; no longer R6.2
- net at U5.12 (DIGIT_1): now also Q6.3 (C)
- net at U5.2 (D): now also R30.2
- net at U5.3 (DIGIT_4): now also Q4.3 (C)
- net at U5.4 (C): now also R29.2
- net at U5.5 (DP): now also R34.2
- net at U5.6 (B): now also R28.2; no longer R7.1
- net at U5.7 (DIGIT_3): now also Q8.3 (C)
- net at U5.8 (DIGIT_2): now also Q7.3 (C)
- net at U5.9 (A): now also R27.2; no longer R4.2
- net WIPER_LOW: now reaches U1.49 (PA5)
- net WIPER_LOW: now also R22.1, Switch_Wipers.1 (Top)
- net SIGNAL_L: now reaches U1.50 (PA12)
- net SIGNAL_L: now also R21.1, Switch_Signal.3 (Bottom)
- net WIPER_HI: now reaches U1.51 (PA6)
- net WIPER_HI: now also R23.1, Switch_Wipers.3 (Bottom)
- net SIGNAL_R: now reaches U1.52 (PA11)
- net SIGNAL_R: now also R20.1, Switch_Signal.1 (Top)
- net at J1.3, U2.6 (CANL): now also R7.2
- net at J1.1, U2.7 (CANH): now also R7.1
- net BTN_MENU renamed BTN_HORN
- net BTN_HORN: now also R16.1
- net BTN_SELECT renamed BTN_HAZARD
- net BTN_HAZARD: now also R17.1
- net IGN_SENSE renamed SW_IGNITION
- net SW_IGNITION: now also R27.1
- net LIGHT_LO renamed LIGHT_LOW
- net LIGHT_LOW: now also R18.1
- new net: Q8.1 (B), R5.1
- new net: R25.1, Switch_Extra.1 (Top)
- new net: R26.1, Switch_Extra.3 (Bottom)
- new net: C2.2, RV1.1
- new net: Button_Extra.2, R24.1
- new net: Q7.1 (B), R4.1
- new net: RV1.2, U4.3 (VO)
- new net: C1.2, RV1.3
- new net: Q4.1 (B), R6.1
- new net: Q6.1 (B), R35.1
- new net +12V: J2.P (POS)
- new net +3.0V: U4.15 (A)
- no-connect marks 5 -> 57
Other:
- note added: "CAN Connector"
- note added: "CAN Transceiver"
- note added: "ESP32"
- note added: "LCD Display"
- note added: "LDO"
- note added: "Power In/Out"
- note added: "STM32"
- note added: "Seven-Segment Display"
- note removed: "12V?"
- moved on the sheet: A1, Button_Hazards, Button_Horn, Cin, Cout, J1, J2, SW_Ignition, Switch_Lights, U2, U4, U7
