File: Front_Control_Board_Duc_Dang/Front_Control_Board_Duc_Dang.kicad_sch (KiCad schematic)
At the start: 0 parts

Commit message: this is my updated version of the board
Parts:
- added C1, C4, C5: C, symbol Device:C
- added C10, C7: 22 p, symbol Device:C
- added C11, C2, C3, C8: 100 nF, symbol Device:C
- added D1, D2, D3, D4, D5, D6, D7: 1N4148WT, Diode_SMD:D_SOD-523, symbol Diode:1N4148WT
- added J1(pressuresensor), J11(throttlesensor), J12(brakesensor), J13(CANin), J14(CANout), J4(hallsensor): 22035035, SMV_Connectors:3pin_CON_22035035_MOL, symbol SMV_Custom:3-pin Mini Molex Spox
- added J10(leftblinker), J5(horn), J6(rightblinker), J7(powerin/out), J8(leftlight), J9(rightlight): 430450200, SMV_Connectors:CONN_SD-43045-001_02_MOL, symbol SMV_Custom:430450200
- added J2: M22-7130442 (jumper pins), SMV_Connectors:M22-7130442_TYC, symbol SMV_Custom:M22-7130442
- added J3(wiper): Molex Micro-Fit 4 Pin, SMV_Connectors:4_pin0430450401, symbol SMV_Custom:Molex Micro-Fit 4 Pin
- added Q1: PSMN1R8-40YLC_115 (MOSFET) (horn), SMV_ICs:LFPAK56_SOT669_NEX, symbol SMV_Custom:PSMN1R8-40YLC_115
- added Q2: PSMN1R8-40YLC_115 (MOSFET) (RBLINK), SMV_ICs:LFPAK56_SOT669_NEX, symbol SMV_Custom:PSMN1R8-40YLC_115
- added Q3: PSMN1R8-40YLC_115 (MOSFET) (LBLINK), SMV_ICs:LFPAK56_SOT669_NEX, symbol SMV_Custom:PSMN1R8-40YLC_115
- added Q4: PSMN1R8-40YLC_115 (MOSFET) (WIPER), SMV_ICs:LFPAK56_SOT669_NEX, symbol SMV_Custom:PSMN1R8-40YLC_115
- added Q5: PSMN1R8-40YLC_115 (MOSFET) (HEADLIGHTS), SMV_ICs:LFPAK56_SOT669_NEX, symbol SMV_Custom:PSMN1R8-40YLC_115
- added R1: 0R, symbol Device:R_US
- added R10, R3, R4, R5, R6, R7, R8, R9: R_US, symbol Device:R_US
- added R11, R12, R13, R14, R16: 100, symbol Device:R_US
- added R15, R17, R18, R2: 10k, symbol Device:R_US
- added SW1: SW_Push, symbol Switch:SW_Push
- added U1: ~, symbol SMV_Custom:STM32_Nucleo_F446RE
- added U2: MCP2562-E/P (CAN TRANSCIVER), SMV_ICs:PDIP8_300MC_MCH, symbol SMV_Custom:MCP2562-E_P
- added U3: MCP6286T-E/OT (OP-AMP) (PS), SMV_ICs:SOT-23-5_MC_MCH, symbol SMV_Custom:MCP6286T-E_OT
- added U4: ADS1118IDGSR (ADC), SMV_ICs:DGS0010A_M, symbol SMV_Custom:ADS1118IDGSR
- added U5: ASM330LHHXTR, SMV_ICs:QFN_LHHXTR_STM-M, symbol SMV_Custom:ASM330LHHXTR
- added U6: SN78MCDCYR (LDO), DCY0004A_N, symbol SMV_Custom:SN78MCDCYR
- added U7: MCP6286T-E/OT (OP-AMP) (BS), SMV_ICs:SOT-23-5_MC_MCH, symbol SMV_Custom:MCP6286T-E_OT
- added U8: MCP6286T-E/OT (OP-AMP) (TS), SMV_ICs:SOT-23-5_MC_MCH, symbol SMV_Custom:MCP6286T-E_OT
- added U9: MCP6286T-E/OT (OP-AMP) (HS), SMV_ICs:SOT-23-5_MC_MCH, symbol SMV_Custom:MCP6286T-E_OT
Connections:
- new net: C2.1, R2.2, SW1.1, U1.14 (RESET)
- new net: R5.2, R6.1, U3.4 (VIN-)
- new net: Q5.4, R16.2
- new net: R10.1, R9.2, U8.4 (VIN-)
- new net: Q4.4, R14.2
- new net: Q3.4, R13.2
- new net: Q1.4, R11.2
- new net: Q2.4, R12.2
- new net: R7.2, R8.1, U7.4 (VIN-)
- new net: R3.1, R4.2, U9.4 (VIN-)
- new net: C7.2, U1.29 (PH0)
- new net: C10.2, U1.31 (PH1)
- new net +12V: C5.2, D2.1 (K), J7(powerin/out).1, U6.1 (INPUT)
- new net 12C_CLOCK: R17.2, U1.61 (PA8), U5.13 (SCL)
- new net 12C_DATA: R18.2, U1.13 (PA13), U5.14 (SDA)
- new net ADC_CS_N: U1.67 (PB5), U4.2 (CS_N)
- new net ADC_DIN: U1.69 (PB3), U4.10 (DIN)
- new net ADC_DOUT: U1.68 (PB13), U4.9 (DOUT_DRDY_N)
- new net ADC_SCLK: U1.66 (PB14), U4.1 (SCLK)
- new net BS OUT: U7.3 (VIN+)
- new net BSOoa: R7.1, U4.6 (AIN2), U7.1 (VOUT)
- new net CAN_H: J13(CANin).1, J14(CANout).1, U2.7 (CANH)
- new net CAN_L: J13(CANin).2, J14(CANout).2, U2.6 (CANL)
- new net CAN_RX: J2.A2, U2.4 (RXD)
- new net CAN_TX: J2.A1, U2.1 (TXD)
- new net CS: U1.16 (+3V3), U5.12 (CS)
- new net GND: C1.2, C10.1, C11.1, C2.2, C3.1, C4.2, C5.1, C7.1, C8.2, D2.2 (A), J1(pressuresensor).2, J11(throttlesensor).2, J12(brakesensor).2, J13(CANin).3, J14(CANout).3, J4(hallsensor).2, J7(powerin/out).2, Q1.1, Q1.2, Q1.3, Q2.1, Q2.2, Q2.3, Q3.1, Q3.2, Q3.3, Q4.1, Q4.2, Q4.3, Q5.1, Q5.2, Q5.3, R1.2, R10.2, R3.2, R6.2, R8.2, SW1.2, U1.19 (GND), U1.20 (GND), U1.22 (GND), U1.47 (GND), U1.8 (GND), U2.2 (VSS), U2.8 (STBY), U3.2 (VSS), U4.3 (GND), U5.7 (GND), U6.2 (COMMON), U6.4 (COMMON), U7.2 (VSS), U8.2 (VSS), U9.2 (VSS)
- new net GNDA: R1.1, U1.70 (AGND)
- new net HORN DRAIN: D1.2 (A), J5(horn).2, Q1.5
- new net HORN M_OUT: R11.1, U1.21 (PB7)
- new net HS OUT: J4(hallsensor).3, U9.3 (VIN+)
- new net HSOoa: R4.1, U4.4 (AIN0), U9.1 (VOUT)
- new net INT1: U1.39 (PC9), U5.4 (INT1)
- new net INT2: U1.40 (PC8), U5.9 (INT2)
- new net JP_RX: J2.A3, U1.52 (PA11)
- new net JP_TX: J2.A4, U1.51 (PA6)
- new net LBLINK DRAIN: D4.2 (A), J10(leftblinker).2, Q3.5
- new net LBLINK M_OUT: R13.1, U1.54 (PB12)
- new net LIGHT DRAIN: D6.2 (A), D7.2 (A), J8(leftlight).2, J9(rightlight).2, Q5.5
- new net LIGHT M_OUT: R16.1, U1.57 (PC7)
- new net PARK SENSE: J3(wiper).3, R15.2, U1.65 (PB4)
- new net PS OUT: J1(pressuresensor).3, U3.3 (VIN+)
- new net PSOoa: R5.1, U3.1 (VOUT), U4.5 (AIN1)
- new net RBLINK DRAIN: D3.2 (A), J6(rightblinker).2, Q2.5
- new net RBLINK M_OUT: R12.1, U1.53 (PA7)
- new net SDO: U1.58 (GND), U5.1 (SDO/SA0)
- new net TS OUT: J11(throttlesensor).3, U8.3 (VIN+)
- new net TSOoa: R9.1, U4.7 (AIN3), U8.1 (VOUT)
- new net VCC: C1.1, C3.2, C4.1, D1.1 (K), D3.1 (K), D4.1 (K), D5.1 (K), D5.2 (A), D6.1 (K), D7.1 (K), J10(leftblinker).1, J11(throttlesensor).1, J12(brakesensor).1, J3(wiper).1, J3(wiper).2, J4(hallsensor).1, J5(horn).1, J6(rightblinker).1, J8(leftlight).1, J9(rightlight).1, Q4.5, R15.1, R17.1, R18.1, U1.24 (VIN), U2.3 (VDD), U3.5 (VDD), U4.8 (VDD), U6.3 (OUTPUT), U7.5 (VDD), U8.5 (VDD), U9.5 (VDD)
- new net VCC 3.3V: C11.2, C8.1, R2.1, U1.45 (AVDD), U1.5 (VDD), U5.5 (Vdd_IO), U5.8 (Vdd)
- new net VCC 5V: J1(pressuresensor).1
- new net WIPER M_OUT: R14.1, U1.55 (PB6)
- no-connect marks 0 -> 42

Commit message: sorry edwin here is the board
Parts:
- removed C3: 100 nF, symbol Device:C
- removed R4, R5, R7, R9: R_US, symbol Device:R_US
- removed U2: MCP2562-E/P (CAN TRANSCIVER), SMV_ICs:PDIP8_300MC_MCH, symbol SMV_Custom:MCP2562-E_P
- added C6: 100 nF, symbol Device:C
- added D8: 1N4148WT, Diode_SMD:D_SOD-523, symbol Diode:1N4148WT
- added J7(powerin/out)1: 430450200, SMV_Connectors:CONN_SD-43045-001_02_MOL, symbol SMV_Custom:430450200
- added U10: MCP2562FD-E/SN (CAN TRANSCIEVER), SMV_ICs:SOIC8-N_MC_MCH-M, symbol SMV_Custom:MCP2562FD-E_SN
- C4, C5: value C -> 10µ
- R10, R3, R6, R8: value R_US -> 10k
Connections:
- net +12V: now also D8.1 (K), J7(powerin/out)1.1
- net BS OUT: now also J12(brakesensor).3
- net CAN_H: now also U10.7 (CANH)
- net CAN_L: now also J13(CANin).3, J14(CANout).3, U10.6 (CANL); no longer J13(CANin).2, J14(CANout).2
- net CAN_RX: now also U10.4 (RXD)
- net CAN_TX: now also U10.1 (TXD)
- net GND: now also J13(CANin).2, J14(CANout).2, C6.1, D8.2 (A), J7(powerin/out)1.2, U10.2 (VSS), U10.8 (STBY); no longer J13(CANin).3, J14(CANout).3
- net VCC: now also C6.2, U10.3 (VDD)
- net 12C_CLOCK renamed SPI_SCK
- net 12C_DATA renamed SPI_MOSI
- net VCC 3.3V renamed +3v3
- net VCC 5V renamed 5v
Other:
- moved on the sheet: C1, C10, C11, C2, C4, C5, C7, C8, D1, D2, D3, D4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
