File: Rear_Control_Board_Levi_Lichtmaher/Rear_Control_Board_Levi_Lichtmaher.kicad_sch (KiCad schematic)
At the start: 90 parts, among them J1 430450200, J10 Molex Micro-Fit 4 Pin, J11 22035035, J12 22035035, J2 430450200, J3 430450200, J4 430450200, J5 430450200, J6 430450200, J7 430450200, J8 430450200, J9 22035035, Q1 PSMN1R8-40YLC_115, Q2 PSMN1R8-40YLC_115, Q3 PSMN1R8-40YLC_115, Q4 PSMN1R8-40YLC_115, U11 MCP6286T-E/OT, U12 MCP6286T-E/OT, U2 ADS1118QDGSRQ1, U3 MCP2562-E/P, U4 UA78M05QDCYRG4Q1, U5 ASM330LHHTR, U6 MCP6286T-E/OT

Commit message: implemented feedback
Parts:
- added R22: 2K, Resistor_SMD:R_0805_2012Metric, symbol Device:R
- added R23: 1K, Resistor_SMD:R_0805_2012Metric, symbol Device:R
- TP35: value 2V5 -> 2V2
Connections:
- net +12V: now also U4.1 (INPUT); no longer U4.3 (INPUT)
- net +3V3: now also R23.2
- net +5V: now also U4.3 (OUTPUT); no longer U4.1 (OUTPUT)
- net GND: now also R22.2
- net +2V5: no longer names the net of TP35.1, U2.7 (AIN3)
- net +2V5: now also R22.1, R23.1
Other:
- moved on the sheet: TP35

Commit message: Implemented Feedback
Parts:
- removed TP36: 12V, TestPoint:TestPoint_Pad_D1.0mm, symbol Connector:TestPoint
- removed TP43, TP44: GND, TestPoint:TestPoint_Pad_D1.0mm, symbol Connector:TestPoint
- added D2, D3, D4: LED, SMV_Passives:WL-SMCW_0603(diode), symbol Device:LED
- added J13, J14: Conn_01x01_Socket, Connector_PinSocket_2.54mm:PinSocket_1x01_P2.54mm_Vertical, symbol Connector:Conn_01x01_Socket
- added LED1, LED2, LED3, LED4: LTST-C170GKT, Green LED:LED_LTST-C170GKT_LTO, symbol Green LED:LTST-C170GKT
- added R24: 1k, Resistor_SMD:R_0805_2012Metric, symbol Device:R
- added R25: 300, Resistor_SMD:R_0805_2012Metric, symbol Device:R
- added R26: 220, Resistor_SMD:R_0805_2012Metric, symbol Device:R
- added R27: 0, Resistor_SMD:R_0805_2012Metric, symbol Device:R
- added TP1: 3.3V, TestPoint:TestPoint_Pad_D1.0mm, symbol Connector:TestPoint
- added TP10: 3V3, TestPoint:TestPoint_Plated_Hole_D2.0mm, symbol Connector:TestPoint
- added TP11: GND, TestPoint:TestPoint_Plated_Hole_D2.0mm, symbol Connector:TestPoint
- added TP13, TP17, TP23: NC, TestPoint:TestPoint_Pad_D1.0mm, symbol Connector:TestPoint
- added TP19: CS2, TestPoint:TestPoint_Pad_D1.0mm, symbol Connector:TestPoint
- added TP20: MOSI, TestPoint:TestPoint_Pad_D1.0mm, symbol Connector:TestPoint
- added TP22: SCK, TestPoint:TestPoint_Pad_D1.0mm, symbol Connector:TestPoint
- added TP3: MISO, TestPoint:TestPoint_Pad_D1.0mm, symbol Connector:TestPoint
- added TP4: Mosfet #4, TestPoint:TestPoint_Pad_D1.0mm, symbol Connector:TestPoint
- added TP5: Mosfet #3, TestPoint:TestPoint_Pad_D1.0mm, symbol Connector:TestPoint
- added TP6: Mosfet #2, TestPoint:TestPoint_Pad_D1.0mm, symbol Connector:TestPoint
- added TP8: Mosfet #1, TestPoint:TestPoint_Pad_D1.0mm, symbol Connector:TestPoint
- added TP9: 12V, TestPoint:TestPoint_Plated_Hole_D2.0mm, symbol Connector:TestPoint
- TP7: footprint TestPoint:TestPoint_Pad_D1.0mm -> TestPoint:TestPoint_Plated_Hole_D2.0mm
- renumbered Q3 to Q2, Q4 to Q3, Q2 to Q4
Connections:
- net +12V: now also R24.1, TP9.1
- net +3V3: now also R26.1, R27.1, R27.2, TP1.1, TP10.1
- net +5V: now also U7.CN7_6 (E5V), R25.1
- net CS2: now also TP19.1
- net GND: now also D2.1 (K), D3.1 (K), D4.1 (K), LED1.1, LED2.1, LED3.1, LED4.1, TP11.1
- net MISO: now also TP3.1
- net MOSI: now also TP20.1
- net RX: now also J14.1 (Pin_1)
- net SCK: now also TP22.1
- net TX: now also J13.1 (Pin_1)
- net at U5.11 (NC): now also TP13.1
- net at U5.4 (INT1): now also TP23.1
- net at U5.9 (INT2): now also TP17.1
- net at Q2.4 (Gate), R5.1, R6.1: now also LED2.2, TP6.1
- net at Q1.4 (Gate), R1.1, R2.1: now also LED4.2, TP8.1
- net at Q4.4 (Gate), R3.1, R4.1: now also LED1.2, TP4.1
- net at Q3.4 (Gate), R7.1, R8.1: now also LED3.2, TP5.1
- new net: D2.2 (A), R24.2
- new net: D4.2 (A), R26.2
- new net: D3.2 (A), R25.2
Other:
- note added: "Mosfet #1"
- note added: "Mosfet #2"
- note added: "Mosfet #3"
- note added: "Mosfet #4"
- note removed: "Mosfet"
- moved on the sheet: J6, R2, R4, R6, R8, TP7
