File: Front_CB_ML/Front_CB_ML.kicad_sch (KiCad schematic)
At the start: 0 parts

Commit message: update
Parts:
- added J1, J10, J2, J3: 22035035, SMV_Connectors:3pin_CON_22035035_MOL, symbol SMV_Custom:3-pin Mini Molex Spox
- added J4: Molex Micro-Fit 4 Pin, SMV_Connectors:4_pin0430450401, symbol SMV_Custom:Molex Micro-Fit 4 Pin
- added J5, J6, J7, J8, J9: 430450200, SMV_Connectors:CONN_SD-43045-001_02_MOL, symbol SMV_Custom:430450200
- added Q1: PSMN1R8-40YLC_115, LFPAK56_SOT669_NEX, symbol SMV_Custom:PSMN1R8-40YLC_115
- added U1: ~, symbol SMV_Custom:STM32_Nucleo_F446RE
- added U2: ADS1118QDGSRQ1, DGS0010A_N, symbol SMV_Custom:ADS1118QDGSRQ1
- added U3: MCP6286T-E/OT, SMV_ICs:SOT-23-5_MC_MCH, symbol SMV_Custom:MCP6286T-E_OT
- added U4: MCP2562-E-P, Package_DIP:DIP-8_W7.62mm, symbol Interface_CAN_LIN:MCP2562-E-P
Connections:
- new net: J10.3, U4.6 (CANL)
- new net: J10.1, U4.7 (CANH)
- new net +12V: J5.1, J6.1, J7.1, J8.1, J9.1
- new net +5V: J1.1, J2.1, J3.1, U4.3 (VDD)
- new net GND: J1.3, J10.2, J2.3, J3.3, U4.2 (VSS), U4.8 (STBY)
Other:
- note added: "Brake Sensor"
- note added: "Pressure Sensor"
- note added: "Throttle Sensor"
- note added: "U1_PB8"
- note added: "U1_PB9"
- note added: "U4_RXD"
- note added: "U4_TXD"
- note added: "Wipers"

Commit message: update
Parts:
- added C1, C10, C11, C12, C13, C14, C15, C2, C3, C4, C5, C6, C7, C8, C9: 0.1uF, SMV_Passives:Cap0805, symbol SMV_Custom:C0805C104K5RACTU
- added Q2, Q3, Q4, Q5: PSMN1R8-40YLC_115, LFPAK56_SOT669_NEX, symbol SMV_Custom:PSMN1R8-40YLC_115
- added R1: 10k, symbol Device:R
- added R10, R11, R12, R13, R14, R15, R16, R2, R3, R4, R5, R6, R7, R8, R9: 100k, symbol Device:R
- added U5, U6: MCP6286T-E/OT, SMV_ICs:SOT-23-5_MC_MCH, symbol SMV_Custom:MCP6286T-E_OT
- added U7: UA78M05QDCYRG4Q1, SMV_ICs:DCY4_TEX, symbol SMV_Custom:UA78M05QDCYRG4Q1
Connections:
- net +12V: now also J4.3, C10.1, C15.1, U7.3 (INPUT)
- net +5V: now also U1.6 (E5V), U2.8 (VDD), C14.2, C2.1, C3.1, C4.1, C5.1, C9.2, U7.1 (OUTPUT)
- net GND: now also Q1.1, Q1.2, Q1.3, U2.3 (GND), U3.1 (VOUT), U3.2 (VSS), U3.4 (VIN-), C1.2, C10.2, C11.2, C12.1, C12.2, C13.2, C14.1, C2.2, C3.2, C4.2, C5.2, C6.2, C7.2, C8.2, C9.1, Q2.1, Q2.2, Q2.3, Q3.1, Q3.2, Q3.3, Q4.1, Q4.2, Q4.3, Q5.1, Q5.2, Q5.3, R1.2, R13.2, R16.1, R3.2, R5.2, R7.2, R9.2, U5.2 (VSS), U6.2 (VSS), U7.2 (GND), U7.4 (GND); no longer U4.8 (STBY)
- net at J1.2: now also R10.2
- net at J3.2: now also R11.2
- net at J2.2: now also U6.3 (VIN+)
- net ADC_SCLK: now reaches U1.49 (PA5)
- net Headlight_L_Mosfet_4: now reaches U1.55 (PB6)
- net Headlight_R_Mosfet_4: now reaches U1.57 (PC7)
- net Turn_Signal_L_Mosfet_4: now reaches U1.59 (PA9)
- net Turn_Signal_R_Mosfet_4: now reaches U1.61 (PA8)
- net ADC_DIN: now reaches U1.64 (PB15)
- net ADC_CS_N: now reaches U1.65 (PB4)
- net ADC_DOUT_DRDY_N: now reaches U1.66 (PB14)
- net STM32_PB8: now reaches U4.1 (TXD)
- net STM32_PB9: now reaches U4.4 (RXD)
- net at U4.5 (Vio): now also C1.1
- net at J7.2: now also J9.2, Q1.5
- net at U3.3 (VIN+): now also R10.1
- net +3.3V: now reaches U3.5 (VDD)
- net +3.3V: now also C6.1, C7.1, C8.1, U5.5 (VDD), U6.5 (VDD)
- net at J5.2: now also Q3.5
- net at J6.2: now also Q2.5
- net STM32_PA_5: now reaches U2.1 (SCLK)
- net STM32_SPI_MOSI: now reaches U2.10 (DIN)
- net STM32_PB4: now reaches U2.2 (CS_N)
- net Throttle Sensor VOUT: now reaches U2.4 (AIN0)
- net Brake Sensor VOUT: now reaches U2.5 (AIN1)
- net Pressure Sensor VOUT: now reaches U2.6 (AIN2)
- net STM32_SPI_MISO: now reaches U2.9 (DOUT_DRDY_N)
- net at Q1.4: now also R2.2, R3.1
- net at J8.2: now also Q4.5
- net at J4.2: now also Q5.4, R15.1, R16.2
- net at J4.4: now also C15.2, Q5.5
- new net: Q3.4, R6.2, R7.1
- new net: C13.1, R14.2, U6.1 (VOUT), U6.4 (VIN-)
- new net: Q4.4, R8.2, R9.1
- new net: R1.1, U4.8 (STBY)
- new net: R11.1, U5.3 (VIN+)
- new net: Q2.4, R4.2, R5.1
- new net: C11.1, R12.2, U5.1 (VOUT), U5.4 (VIN-)
- new net ADC_AIN0: R13.1
- new net ADC_AIN1: R12.1
- new net ADC_AIN2: R14.1
- new net PA_8: R2.1
- new net PA_9: R4.1
- new net PC_7: R6.1
- no-connect marks 0 -> 2
Other:
- note added: "Headlight_Left"
- note added: "Headlight_Right"
- note added: "Horn"
- note added: "Turn_Signal_Left"
- note added: "Turn_Signal_Right"
- note removed: "U1_PB8"
- note removed: "U1_PB9"
- note removed: "Wipers"
- moved on the sheet: J1, J10, J2, J3, J4, J5, J6, J7, J8, J9, Q1, U1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

Commit message: some tweaks?
Connections:
- net +12V: now also C10.2; no longer C10.1
- net +3.3V: now also U1.16 (+3V3)
- net GND: now also C10.1, U1.19 (GND), U1.20 (GND), U1.22 (GND); no longer C10.2
- net PA10_D2: now reaches R1.1, U4.8 (STBY)
- net U4_CAN_TXD: now reaches U1.41 (PB8)
- net U4_CAN_RXD: now reaches U1.43 (PB9)
- net PA10_D2_Standby: now reaches U1.71 (PA10)
- no-connect marks 2 -> 53
Other:
- note removed: "U4_RXD"
- note removed: "U4_TXD"
- moved on the sheet: C10
