File: Wilson_Wu_William_Yang_Safety_Board/_autosave-Wilson_Wu_William_Yang_Safety_Board.kicad_pcb (KiCad board)
At the start: 2 copper layers, 259 x 142 mm, 49 parts, among them J1 22035035, J2 XT60-M, J3 XT60-M, J4 M22-7130442, J5 Molex Micro-Fit 4 Pin, J6 430450200, J7 430450200, Q1 IRLML6344TRPBF, U1 STM32, U10 10kohm, U2 MCP2562-E_P, U3 MCP6286T-E/OT, U4 CD4002BE, U5 100 ohm, U6 J115F11AH12VDCS61.5U, U7 LM1117IDTX-3.3/NOPB, U8 LM1117IDTX-3.3/NOPB, U9 MCP6286T-E/OT

Commit message: Layout Changes
Parts:
- U1: footprint stm32nucleoflr:LQFP100-14x14mm -> SMV_ICs:MODULE_NUCLEO-F446RE
- moved C1 169.0 mm to (251.0, 63.0)
- moved C2 169.0 mm to (259.1, 56.5)
- moved U7 169.0 mm to (259.4, 63.0)
- moved C11 155.5 mm to (249.4, 54.6)
- moved C6 155.5 mm to (253.9, 38.1)
- moved C7 155.5 mm to (268.4, 38.1)
- moved J5 155.5 mm to (240.4, 29.1)
- moved R6 155.5 mm to (255.9, 49.0)
- moved R7 155.5 mm to (250.7, 49.0)
- moved R80 155.5 mm to (250.0, 30.0)
- moved R9 155.5 mm to (265.3, 49.0)
- moved U10 155.5 mm to (264.9, 26.0)
- moved U5 155.5 mm to (241.6, 36.5)
- moved R4 155.5 mm to (270.4, 29.0)
- moved R8 155.5 mm to (242.8, 42.5)
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Connections:
- D1 pad 1: GND -> Net-(D1-K)
- D1 pad 2: Net-(D1-A) -> GND
- R2 pad 1: Net-(D1-A) -> Net-(D1-K)

Commit message: Layout changes
Parts:
- U1: footprint SMV_ICs:MODULE_NUCLEO-F446RE -> SMV_ICs:MODULE_NUCLEO-F446RE_NEW
- moved C8 176.0 mm to (211.2, 111.9), turned to 90 degrees
- moved C1 166.4 mm to (104.6, 142.2)
- moved C11 166.4 mm to (103.0, 133.8)
- moved C2 166.4 mm to (112.7, 135.8)
- moved C6 166.4 mm to (107.5, 117.3)
- moved C7 166.4 mm to (122.0, 117.3)
- moved J5 166.4 mm to (94.0, 108.3)
- moved R6 166.4 mm to (109.5, 128.2)
- moved R7 166.4 mm to (104.3, 128.2)
- moved R80 166.4 mm to (103.6, 109.3)
- moved R81 166.4 mm to (81.8, 107.9)
- moved R9 166.4 mm to (118.9, 128.2)
- moved U10 166.4 mm to (118.5, 105.3)
- moved U5 166.4 mm to (95.2, 115.8)
- moved U7 166.4 mm to (113.0, 142.3)
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