File: Wilson_Wu_William_Yang_Safety_Board/_autosave-Wilson_Wu_William_Yang_Safety_Board.kicad_pcb (KiCad board)
At the start: 2 copper layers, 110 parts, among them J1 22035035, J18 XT60-M, J2 22035035, J3 430450200, J4 M22-7130442, J5 430450200, J6 XT60-M, J7 XT60-M, J8 430450200, J9 Molex Micro-Fit 4 Pin, Q1 IRLML6344TRPBF, Q2 IRLML6344TRPBF, Q3 NTBLS0D8N08XTXG, Q4 NTBLS0D8N08XTXG, U1 STM32, U10 LTC4364HS, U11 LMV331IDBVR, U12 J115F11AH12VDCS61.5U, U15 INA826AID, U16 J115F11AH12VDCS61.5U, U2 MCP2562-E_P, U3 10kohm, U4 SN74HCS21QPWRQ1, U5 J115F11AH12VDCS61.5U, U6 J115F11AH12VDCS61.5U, U7 LM1117IDTX-5.0/NOPB, U8 LM1117IMPX-ADJ/NOPB, U9 100 ohm

Commit message: layout
Parts:
- moved C2 12.0 mm to (140.5, 59.1)
- moved TP17 12.0 mm to (137.3, 59.1)
- moved U7 12.0 mm to (141.7, 54.5)
- moved C1 8.85 mm to (151.8, 53.1)
- moved TP12 4.65 mm to (112.0, 64.5)
Changed lines of the file:
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@@
 	(footprint "TestPoint:TestPoint_Pad_D1.0mm"
 		(layer "F.Cu")
-		(at 149.160001 57.154999 180)
+		(at 137.32 59.054999 180)
 		(descr "SMD pad as test Point, diameter 1.0mm")
 		(tags "test point SMD pad")
@@
 	(footprint "ul_LM1117IDTX-3-3-NOPB:NDP0003B"
 		(layer "F.Cu")
-		(at 153.540001 52.6 180)
+		(at 141.7 54.5 180)
 		(tags "LM1117IDTX-3.3/NOPB ")
 		(property "Reference" "U7"
@@
 	(footprint "TestPoint:TestPoint_Loop_D2.54mm_Drill1.5mm_Beaded"
 		(layer "F.Cu")
-		(at 111.85 69.15)
+		(at 112 64.5)
 		(descr "wire loop with bead as test point, loop diameter2.548mm, hole diameter 1.5mm")
 		(tags "test point wire loop bead")
@@
 	(footprint "Capacitor_SMD:C_0805_2012Metric"
 		(layer "F.Cu")
-		(at 160.6 52.2 -90)
+		(at 151.8 53.15 -90)
 		(descr "Capacitor SMD 0805 (2012 Metric), square (rectangular) end terminal, IPC-7351 nominal, (Body size source: IPC-SM-782 page 76, https://www.pcb-3d.com/wordpress/wp-content/uploads/ipc-sm-782a_amendment_1_and_2.pdf, https://docs.google.com/spreadsheets/d/1BsfQQcO9C6DZCsRaXUlFlo91Tg2WpOkGARC1WS5S8t0/edit?usp=sharing), generated with kicad-footprint-generator")
 		(tags "capacitor")
@@
 	(footprint "Capacitor_SMD:C_0805_2012Metric"
 		(layer "F.Cu")
-		(at 152.360001 57.154999 180)
+		(at 140.52 59.054999 180)
 		(descr "Capacitor SMD 0805 (2012 Metric), square (rectangular) end terminal, IPC-7351 nominal, (Body size source: IPC-SM-782 page 76, https://www.pcb-3d.com/wordpress/wp-content/uploads/ipc-sm-782a_amendment_1_and_2.pdf, https://docs.google.com/spreadsheets/d/1BsfQQcO9C6DZCsRaXUlFlo91Tg2WpOkGARC1WS5S8t0/edit?usp=sharing), generated with kicad-footprint-generator")
 		(tags "capacitor")
@@
 	)
 	(via
-		(at 154.423333 57.098916)
+		(at 142.583332 58.998916)
 		(size 0.6)
 		(drill 0.3)
