File: Wilson_Wu_William_Yang_Safety_Board/_autosave-hydrogen_sensors.kicad_sch (KiCad schematic)
At the start: 11 parts, among them J5 Molex Micro-Fit 4 Pin, J9 Molex Micro-Fit 4 Pin, U15 INA826AID, U9 100 ohm

Commit message: sch changes
Parts:
- added C6: 0.1 uF, symbol Device:C
- added R14: 100 ohm, Resistor_SMD:R_0805_2012Metric, symbol Device:R_US
Connections:
- net hydrogen_out is gone; now on net h_out: J9.3, J9.4, TP3.1
- net hydrogen_ref is gone; now on net h_ref: TP16.1, U9.3
- net +3V0: now also U15.8 (VS+), C6.2
- net GND: now also U15.5 (VS-), C6.1
- net h_out: now reaches U15.1 (IN-)
- net at U15.2 (RG): now also R14.2
- net at U15.3 (RG): now also R14.1
- net h_ref: now reaches U15.4 (IN+)
- net ina_output: now reaches U15.7 (VOUT)
- no-connect marks 1 -> 2
