File: Wilson_Wu_William_Yang_Safety_Board/inverter.kicad_sch (KiCad schematic)
At the start: 1 part, among them U14 SN74AHCT14QPWRQ1

Commit message: sch update
Parts:
- added C19: 0.1uF, symbol Device:C
Connections:
- net +3.3V: now also C19.1
- net GND: now also C19.2
- net INVERT_1: now reaches U14.10 (5Y)
- net INVERT_1: now also U14.12 (6Y), U14.8 (4Y)
- net h_sensor_2: now reaches U14.11 (5A)
- net h_sensor_1: now reaches U14.13 (6A)
- net h_sensor_3: now reaches U14.9 (4A)

Commit message: sch changes
Parts:
- C19: footprint (none) -> Capacitor_SMD:C_0805_2012Metric
Connections:
- net INVERT_1: no longer U14.10 (5Y), U14.8 (4Y)
- net h_sensor_3: no longer names the net of U14.9 (4A)
- new net INVERT_2: U14.10 (5Y)
- no-connect marks 3 -> 5
Changed lines of the file:
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@@
+	)
+	(no_connect
+		(at 99.06 48.26)
+	)
+	(no_connect
+		(at 99.06 45.72)
 	)
 	(no_connect
@@
 		(pts
 			(xy 40.64 38.1) (xy 43.18 38.1)
-		)
-		(stroke
-			(width 0)
-			(type default)
-		)
-	)
-	(wire
-		(pts
-			(xy 99.06 45.72) (xy 115.57 45.72)
-		)
-		(stroke
-			(width 0)
-			(type default)
-		)
-	)
-	(wire
-		(pts
-			(xy 99.06 48.26) (xy 100.33 48.26)
 		)
 		(stroke
@@
 		)
 	)
-	(label "INVERT_1"
+	(label "INVERT_2"
 		(at 100.33 43.18 0)
 		(effects
@@
 		)
 	)
-	(label "INVERT_1"
-		(at 100.33 48.26 0)
+	(global_label "h_sensor_1"
+		(shape input)
+		(at 115.57 35.56 0)
+		(fields_autoplaced yes)
 		(effects
 			(font
 				(size 1.27 1.27)
 			)
-			(justify left bottom)
-		)
-	)
-	(global_label "h_sensor_1"
-		(shape input)
-		(at 115.57 35.56 0)
-		(fields_autoplaced yes)
-		(effects
-			(font
-				(size 1.27 1.27)
-			)
 			(justify left)
 		)
 		(property "Intersheetrefs" "${INTERSHEET_REFS}"
 			(at 129.0779 35.56 0)
-			(effects
-				(font
-					(size 1.27 1.27)
-				)
-				(justify left)
-				(hide yes)
-			)
-		)
-	)
-	(global_label "h_sensor_3"
-		(shape input)
-		(at 115.57 45.72 0)
-		(fields_autoplaced yes)
-		(effects
-			(font
-				(size 1.27 1.27)
-			)
-			(justify left)
-		)
-		(property "Intersheetrefs" "${INTERSHEET_REFS}"
-			(at 129.0779 45.72 0)
 			(effects
 				(font
@@
 			)
 		)
-		(property "Footprint" ""
+		(property "Footprint" "Capacitor_SMD:C_0805_2012Metric"
 			(at 99.3648 22.86 0)
 			(effects
