File: Wilson_Wu_William_Yang_Safety_Board/_autosave-untitled.kicad_sch (KiCad schematic)
At the start: 50 parts, among them J10 XT60-M, J11 XT60-M, J6 430450200, J7 430450200, Q2 IRLML6344TRPBF, Q3 IRLML6344TRPBF, Q4 IRLML6344TRPBF, U10 J115F11AH12VDCS61.5U, U12 J115F11AH12VDCS61.5U, U13 TS5A23157QDGSRQ1, U14 J115F11AH12VDCS61.5U, U5 J115F11AH12VDCS61.5U, U6 TS5A23157QDGSRQ1

Commit message: bruh
Connections:
- net A Relay is gone; now on net MOSFET Connection: U13.4 (NO2), U6.4 (NO2)
- net at R20.2: now also U13.6 (COM2); no longer U13.5 (IN2)
- no-connect marks 2 -> 5
Changed lines of the file:
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@@
 	)
 	(junction
+		(at 54.61 35.56)
+		(diameter 0)
+		(color 0 0 0 0)
+	)
+	(junction
 		(at 187.96 110.49)
 		(diameter 0)
@@
 	)
 	(junction
-		(at 187.96 27.94)
+		(at 49.53 35.56)
 		(diameter 0)
 		(color 0 0 0 0)
 	)
 	(junction
-		(at 157.48 88.9)
+		(at 187.96 27.94)
 		(diameter 0)
 		(color 0 0 0 0)
 	)
 	(junction
-		(at 49.53 35.56)
+		(at 157.48 88.9)
 		(diameter 0)
 		(color 0 0 0 0)
@@
 	)
 	(no_connect
+		(at 120.65 82.55)
+	)
+	(no_connect
 		(at 120.65 135.89)
 	)
 	(no_connect
-		(at 120.65 125.73)
+		(at 120.65 92.71)
 	)
-	(wire
-		(pts
-			(xy 157.48 81.28) (xy 157.48 88.9)
-		)
-		(stroke
-			(width 0)
-			(type default)
-		)
+	(no_connect
+		(at 120.65 120.65)
+	)
+	(no_connect
+		(at 120.65 130.81)
 	)
 	(wire
 		(pts
-			(xy 73.66 118.11) (xy 73.66 116.84)
+			(xy 157.48 81.28) (xy 157.48 88.9)
 		)
 		(stroke
@@
 	(wire
 		(pts
-			(xy 120.65 140.97) (xy 124.46 140.97)
+			(xy 120.65 140.97) (xy 127 140.97)
 		)
 		(stroke
@@
 	(wire
 		(pts
-			(xy 73.66 118.11) (xy 74.93 118.11)
+			(xy 63.5 118.11) (xy 74.93 118.11)
 		)
 		(stroke
@@
 	(wire
 		(pts
-			(xy 129.54 118.11) (xy 129.54 120.65)
-		)
-		(stroke
-			(width 0)
-			(type default)
-		)
-	)
-	(wire
-		(pts
 			(xy 62.23 100.33) (xy 74.93 100.33)
 		)
@@
 	(wire
 		(pts
-			(xy 54.61 30.48) (xy 54.61 40.64)
+			(xy 54.61 30.48) (xy 54.61 35.56)
 		)
 		(stroke
@@
 	(wire
 		(pts
+			(xy 54.61 35.56) (xy 59.69 35.56)
+		)
+		(stroke
+			(width 0)
+			(type default)
+		)
+	)
+	(wire
+		(pts
 			(xy 46.99 45.72) (xy 49.53 45.72)
 		)
@@
 	(wire
 		(pts
-			(xy 49.53 35.56) (xy 59.69 35.56)
+			(xy 201.93 19.05) (xy 208.28 19.05)
 		)
 		(stroke
@@
 	(wire
 		(pts
-			(xy 201.93 19.05) (xy 208.28 19.05)
+			(xy 157.48 27.94) (xy 187.96 27.94)
 		)
 		(stroke
@@
 	(wire
 		(pts
-			(xy 157.48 27.94) (xy 187.96 27.94)
+			(xy 187.96 147.32) (xy 194.31 147.32)
 		)
 		(stroke
@@
 	(wire
 		(pts
-			(xy 187.96 147.32) (xy 194.31 147.32)
+			(xy 233.68 41.91) (xy 233.68 40.64)
 		)
 		(stroke
@@
 	(wire
 		(pts
-			(xy 233.68 41.91) (xy 233.68 40.64)
+			(xy 177.8 73.66) (xy 190.5 73.66)
 		)
 		(stroke
@@
 	(wire
 		(pts
-			(xy 177.8 73.66) (xy 190.5 73.66)
+			(xy 158.75 128.27) (xy 158.75 134.62)
 		)
 		(stroke
@@
 	(wire
 		(pts
-			(xy 158.75 128.27) (xy 158.75 134.62)
+			(xy 208.28 27.94) (xy 219.71 27.94)
 		)
 		(stroke
@@
 	(wire
 		(pts
-			(xy 208.28 27.94) (xy 219.71 27.94)
+			(xy 129.54 118.11) (xy 129.54 125.73)
 		)
 		(stroke
@@
 	(wire
 		(pts
-			(xy 148.59 35.56) (xy 148.59 45.72)
+			(xy 49.53 35.56) (xy 54.61 35.56)
 		)
 		(stroke
@@
 	(wire
 		(pts
-			(xy 208.28 91.44) (xy 215.9 91.44)
+			(xy 148.59 35.56) (xy 148.59 45.72)
 		)
 		(stroke
@@
 	(wire
 		(pts
-			(xy 129.54 120.65) (xy 120.65 120.65)
+			(xy 208.28 91.44) (xy 215.9 91.44)
 		)
 		(stroke
@@
 	(wire
 		(pts
+			(xy 129.54 125.73) (xy 120.65 125.73)
+		)
+		(stroke
+			(width 0)
+			(type default)
+		)
+	)
+	(wire
+		(pts
 			(xy 201.93 62.23) (xy 208.28 62.23)
 		)
@@
 	(wire
 		(pts
-			(xy 120.65 102.87) (xy 123.19 102.87)
+			(xy 120.65 102.87) (xy 133.35 102.87)
 		)
 		(stroke
@@
 	(wire
 		(pts
+			(xy 54.61 35.56) (xy 54.61 40.64)
+		)
+		(stroke
+			(width 0)
+			(type default)
+		)
+	)
+	(wire
+		(pts
 			(xy 187.96 19.05) (xy 194.31 19.05)
 		)
@@
 	(symbol
 		(lib_id "power:+3V3")
-		(at 123.19 102.87 0)
+		(at 133.35 102.87 0)
 		(unit 1)
 		(exclude_from_sim no)
@@
 		(fields_autoplaced yes)
 		(property "Reference" "#PWR09"
-			(at 123.19 106.68 0)
+			(at 133.35 106.68 0)
 			(effects
 				(font
@@
 		)
 		(property "Value" "+3V3"
-			(at 123.19 97.79 0)
+			(at 133.35 97.79 0)
 			(effects
 				(font
@@
 		)
 		(property "Footprint" ""
-			(at 123.19 102.87 0)
+			(at 133.35 102.87 0)
 			(effects
 				(font
@@
 		)
 		(property "Datasheet" ""
-			(at 123.19 102.87 0)
+			(at 133.35 102.87 0)
 			(effects
 				(font
@@
 		)
 		(property "Description" "Power symbol creates a global label with name \"+3V3\""
-			(at 123.19 102.87 0)
+			(at 133.35 102.87 0)
 			(effects
 				(font
@@
 	(symbol
 		(lib_id "power:+3V3")
-		(at 124.46 140.97 0)
+		(at 127 140.97 0)
 		(unit 1)
 		(exclude_from_sim no)
@@
 		(fields_autoplaced yes)
 		(property "Reference" "#PWR011"
-			(at 124.46 144.78 0)
+			(at 127 144.78 0)
 			(effects
 				(font
@@
 		)
 		(property "Value" "+3V3"
-			(at 124.46 135.89 0)
+			(at 127 135.89 0)
 			(effects
 				(font
@@
 		)
 		(property "Footprint" ""
-			(at 124.46 140.97 0)
+			(at 127 140.97 0)
 			(effects
 				(font
@@
 		)
 		(property "Datasheet" ""
-			(at 124.46 140.97 0)
+			(at 127 140.97 0)
 			(effects
 				(font
@@
 		)
 		(property "Description" "Power symbol creates a global label with name \"+3V3\""
-			(at 124.46 140.97 0)
+			(at 127 140.97 0)
 			(effects
 				(font
@@
 	(symbol
 		(lib_id "power:GND")
-		(at 73.66 116.84 180)
+		(at 63.5 118.11 0)
 		(unit 1)
 		(exclude_from_sim no)
@@
 		(fields_autoplaced yes)
 		(property "Reference" "#PWR050"
-			(at 73.66 110.49 0)
+			(at 63.5 124.46 0)
 			(effects
 				(font
@@
 		)
 		(property "Value" "GND"
-			(at 73.66 111.76 0)
+			(at 63.5 123.19 0)
 			(effects
 				(font
@@
 		)
 		(property "Footprint" ""
-			(at 73.66 116.84 0)
+			(at 63.5 118.11 0)
 			(effects
 				(font
@@
 		)
 		(property "Datasheet" ""
-			(at 73.66 116.84 0)
+			(at 63.5 118.11 0)
 			(effects
 				(font
@@
 		)
 		(property "Description" "Power symbol creates a global label with name \"GND\" , ground"
-			(at 73.66 116.84 0)
+			(at 63.5 118.11 0)
 			(effects
 				(font
