File: Wilson_Wu_William_Yang_Safety_Board/_autosave-load_switch.kicad_sch (KiCad schematic)
At the start: 20 parts, among them Q3 NTBLS0D8N08XTXG, Q4 NTBLS0D8N08XTXG, U10 LTC4364HS

Commit message: grouped components together
Parts:
- Q3, Q4: footprint H-PSOF8L_100CU_ONS_OSI -> load switch mosfet:H-PSOF8L_100CU_ONS_OSI
Changed lines of the file:
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@@
 			)
 		)
-		(property "Footprint" "H-PSOF8L_100CU_ONS_OSI"
+		(property "Footprint" "load switch mosfet:H-PSOF8L_100CU_ONS_OSI"
 			(at 162.56 60.96 0)
 			(effects
@@
 			)
 		)
-		(property "Footprint" "H-PSOF8L_100CU_ONS_OSI"
+		(property "Footprint" "load switch mosfet:H-PSOF8L_100CU_ONS_OSI"
 			(at 152.4 60.96 0)
 			(effects
