File: VDJoulemeter/HighPowerJoulemeter.kicad_pcb (KiCad board)
At the start: 4 copper layers, 119.2 x 118.6 mm, 92 parts, among them J1 XT60-M, J2 XT60-M, J3 22035035, J4 22035035, U3 MCP2562, U4 TMCS1126B6AQDVGRQ1, U5 MCP6286T-E/OT, U6 PTPSM365R6V5RDNR, U8 ADS1118QDGSRQ1, U9 MIC5219-3.3YM5-TR

Commit message: changes
Parts:
- removed TP15: TestPoint, TestPoint:TestPoint_Pad_4.0x4.0mm
- added D1: LED (Green), Resistor_SMD:R_0201_0603Metric, F.Cu at (149.2, -679.5)
- added D2: LED (Blue), Resistor_SMD:R_0201_0603Metric, F.Cu at (142.2, -679.0)
- added D3: LED, Resistor_SMD:R_0201_0603Metric, F.Cu at (152.0, -654.3)
- added D4: LED, Resistor_SMD:R_0201_0603Metric, F.Cu at (156.5, -654.5)
- added R10: 2.2k, Resistor_SMD:R_0805_2012Metric_Pad1.20x1.40mm_HandSolder, F.Cu at (149.7, -653.5)
- added R13: 2.2k, Resistor_SMD:R_0805_2012Metric_Pad1.20x1.40mm_HandSolder, F.Cu at (155.5, -653.0)
- added R14: 2.2k, Resistor_SMD:R_0805_2012Metric_Pad1.20x1.40mm_HandSolder, F.Cu at (152.0, -679.5)
- added R15: 2.2k, Resistor_SMD:R_0805_2012Metric_Pad1.20x1.40mm_HandSolder, F.Cu at (139.0, -679.5)
- U3: footprint SMV_ICs:PDIP8_300MC_MCH -> SMV_ICs:MCP2562-E_SN_SOIC8-N_MC_MCH-M
- moved TP45 98.0 mm to (193.0, -670.5)
- moved R11 27.1 mm to (196.5, -635.0), turned to 180 degrees
- moved TP43 24.7 mm to (195.5, -632.0)
- moved U3 8.80 mm to (104.5, -615.0)
- moved C22 6.50 mm to (110.0, -654.5)
- moved TP56 6.30 mm to (96.5, -609.5)
- moved TP57 5.54 mm to (96.5, -617.5)
- moved J3 4.02 mm to (92.0, -612.6)
- moved TP9 3.19 mm to (122.5, -667.0)
Connections:
- C11 pad 2: +3.3V -> Net-(U9-OUT)
- C8 pad 1: +5V -> Net-(U6-BIAS)
- C9 pad 1: +5V -> Net-(U6-BIAS)
- R11 pad 2: Net-(U1-PB0) -> Net-(U1-VBAT)
- TP43 pad 1: Net-(U1-PB0) -> Net-(U1-VBAT)
- TP5 pad 1: +5V -> Net-(U6-BIAS)
- TP7 pad 1: +3.3V -> Net-(U9-OUT)
- U1 pad 33: unconnected-(U1-VBAT-Pad33) -> Net-(U1-VBAT)
- U1 pad 34: Net-(U1-PB0) -> unconnected-(U1-PB0-Pad34)
- U1 pad 65: unconnected-(U1-PB4-Pad65) -> Net-(U1-PB4)
- U1 pad 67: unconnected-(U1-PB5-Pad67) -> Net-(U1-PB5)
- U6 pad 4: +5V -> Net-(U6-BIAS)
- U6 pad 9: +5V -> Net-(U6-BIAS)
- U9 pad 5: +3.3V -> Net-(U9-OUT)
Routing:
- net GND: track 158.2 -> 102.7 mm, vias 60 -> 58
- net Net-(U1-PB0): track 43.1 -> 0.00 mm
- net Net-(U1-PB5): track 0.00 -> 39.4 mm
- net Net-(U1-PB4): track 0.00 -> 29.1 mm
- net +3.3V: track 104.5 -> 93.1 mm, vias 4 -> 5
- net Net-(U1-VBAT): track 0.00 -> 11.3 mm, vias 0 -> 1
- net /STM_CAN_TX_PIN: track 16.6 -> 22.7 mm
- net Net-(U6-BIAS): track 0.00 -> 4.65 mm
- net /STM_CAN_RX_PIN: track 18.9 -> 23.6 mm
- net /CAN_P: track 28.1 -> 31.9 mm
- net /CAN_N: track 28.6 -> 31.9 mm
- net 48V_IN: track 27.5 -> 24.4 mm
- net Net-(D2-A): track 0.00 -> 2.04 mm
- net +5V: track 87.9 -> 89.8 mm
- net Net-(D4-A): track 0.00 -> 1.63 mm
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- added copper zone on B.Cu, net GND

Commit message: hall sensor fix
Parts:
- removed TP14, TP19, TP2, TP22, TP26, TP27, TP60, TP66: TestPoint, TestPoint:TestPoint_Pad_1.0x1.0mm
- TP23, TP45: footprint TestPoint:TestPoint_Pad_4.0x4.0mm -> TestPoint:TestPoint_Pad_1.0x1.0mm
- moved TP9 13.0 mm to (117.5, -679.0)
- moved R1 12.7 mm to (140.5, -651.0)
- moved R2 10.3 mm to (145.0, -653.5)
- moved TP1 8.01 mm to (139.5, -653.0)
- moved U5 3.92 mm to (140.7, -656.0)
- moved C3 3.87 mm to (145.0, -655.5), turned to 180 degrees
- moved TP3 3.47 mm to (120.0, -653.5)
- moved TP8 3.04 mm to (137.5, -658.0)
- moved U4 2.50 mm to (130.0, -662.5)
- moved TP23 0.98 mm to (141.0, -669.5)
Routing:
- net 48V_OUT: track 31.1 -> 7.34 mm
- net 48V_IN: track 24.4 -> 16.5 mm
- net GND: track 102.7 -> 96.4 mm, vias 58 -> 56
- net +3.3V: track 93.1 -> 89.0 mm
- net /VoltageDividerOut: track 11.5 -> 8.54 mm
- net Net-(U9-OUT): track 0.00 -> 2.91 mm
- net Net-(U6-BIAS): track 4.65 -> 7.27 mm
- net Net-(U8-AIN1): track 7.06 -> 4.76 mm
- net /I_Sense: track 6.23 -> 8.53 mm
- net /V_Ref: track 14.5 -> 16.8 mm
- net /V_Sense: track 25.6 -> 23.8 mm
- net Net-(D1-A): track 0.00 -> 1.53 mm
- net Net-(U6-VCC): track 6.52 -> 5.46 mm
