File: VDJoulemeter/HighPowerJoulemeter.kicad_sch (KiCad schematic)
At the start: 98 parts, among them J1 XT60-M, J2 XT60-M, J3 22035035, J4 22035035, U3 MCP2562, U4 TMCS1126B6AQDVGRQ1, U5 MCP6286T-E/OT, U6 PTPSM365R6V5RDNR, U8 ADS1118QDGSRQ1, U9 MIC5219-3.3YM5-TR

Commit message: changes
Parts:
- U3: footprint SMV_ICs:PDIP8_300MC_MCH -> SMV_ICs:MCP2562-E_SN_SOIC8-N_MC_MCH-M
Connections:
- net at R11.2, TP43.1: now also U1.33 (VBAT); no longer U1.34 (PB0)
Other:
- note added: "48V to 5V DCDC Converter"
- note removed: "48Vto5V DCDC Converter"
- moved on the sheet: TP43
Changed lines of the file:
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@@
 		)
 	)
-	(text "48Vto5V DCDC Converter"
+	(text "48V to 5V DCDC Converter"
 		(exclude_from_sim no)
 		(at 257.048 40.64 0)
@@
 	)
 	(junction
-		(at 386.08 212.09)
+		(at 403.86 138.43)
 		(diameter 0)
 		(color 0 0 0 0)
 	)
 	(junction
-		(at 403.86 138.43)
+		(at 386.08 209.55)
 		(diameter 0)
 		(color 0 0 0 0)
@@
 	)
 	(no_connect
-		(at 416.56 209.55)
-	)
-	(no_connect
 		(at 257.81 76.2)
 	)
@@
 	)
 	(no_connect
+		(at 416.56 212.09)
+	)
+	(no_connect
 		(at 416.56 194.31)
 	)
@@
 	(wire
 		(pts
-			(xy 386.08 212.09) (xy 369.57 212.09)
+			(xy 386.08 209.55) (xy 369.57 209.55)
 		)
 		(stroke
@@
 	(wire
 		(pts
-			(xy 369.57 205.74) (xy 369.57 212.09)
+			(xy 369.57 205.74) (xy 369.57 209.55)
 		)
 		(stroke
@@
 	(wire
 		(pts
-			(xy 416.56 212.09) (xy 386.08 212.09)
+			(xy 416.56 209.55) (xy 386.08 209.55)
 		)
 		(stroke
@@
 			)
 		)
-		(property "Footprint" "SMV_ICs:PDIP8_300MC_MCH"
+		(property "Footprint" "SMV_ICs:MCP2562-E_SN_SOIC8-N_MC_MCH-M"
 			(at 344.17 302.26 0)
 			(effects
@@
 	(symbol
 		(lib_id "Connector:TestPoint")
-		(at 386.08 212.09 180)
+		(at 386.08 209.55 180)
 		(unit 1)
 		(exclude_from_sim no)
@@
 		(fields_autoplaced yes)
 		(property "Reference" "TP43"
-			(at 388.62 214.1219 0)
+			(at 388.62 211.5819 0)
 			(effects
 				(font
@@
 		)
 		(property "Value" "TestPoint"
-			(at 388.62 216.6619 0)
+			(at 388.62 214.1219 0)
 			(effects
 				(font
@@
 		)
 		(property "Footprint" "TestPoint:TestPoint_Pad_1.0x1.0mm"
-			(at 381 212.09 0)
+			(at 381 209.55 0)
 			(effects
 				(font
@@
 		)
 		(property "Datasheet" "~"
-			(at 381 212.09 0)
+			(at 381 209.55 0)
 			(effects
 				(font
@@
 		)
 		(property "Description" "test point"
-			(at 386.08 212.09 0)
+			(at 386.08 209.55 0)
 			(effects
 				(font

Commit message: hall sensor fix
Parts:
- removed TP14, TP19, TP2, TP22, TP26, TP66: TestPoint, TestPoint:TestPoint_Pad_1.0x1.0mm, symbol Connector:TestPoint
- TP23, TP45: footprint TestPoint:TestPoint_Pad_4.0x4.0mm -> TestPoint:TestPoint_Pad_1.0x1.0mm
