File: Safety_Board_Nirav_Michelsen/_autosave-Safety_Board_Nirav_Michelsen.kicad_sch (KiCad schematic)
At the start: 29 parts, among them J1 430450200, J2 Molex Micro-Fit 4 Pin, J3 XT60-M, J4 430450200, J5 22035035, J6 XT60-M, J7 430450200, K1 Fujitsu_FTR-LYAA005x, U1 MCP6286T-E/OT, U3 4068, U4 74AHC1G04, U5 MCP2562-E-P, U6 MCP1700x-330xxTT

Commit message: draft 4
Parts:
- removed U1: MCP6286T-E/OT, SMV_ICs:SOT-23-5_MC_MCH, symbol SMV_Custom:MCP6286T-E_OT
- added C8, C9: 0.1 uF, symbol Device:C
- added R6, R9: 10K Ohms, symbol Device:R_US
- added R7: 1M Ohms, symbol Device:R_US
- added R8: 10k Ohms, symbol Device:R_US
- added U7: 4068, symbol 4xxx_IEEE:4068
- added U8: LMV331, symbol Comparator:LMV331
Connections:
- net +3.3V: now also U7.10 (F), U7.11 (G), U7.12 (H), U7.9 (E)
- net +5V: now also J1.2, J7.2, R9.2, U7.14 (Vdd), U8.5 (V+); no longer R2.2, R5.2
- net GATEDR: now also C9.1, R7.2, R9.1, U7.2 (A), U8.4
- net GATE_E: now also U7.3 (B); no longer J7.1, R5.1
- net GND: now also R2.2, R5.2, C8.1, C9.2, U7.7 (Vss), U8.2 (V-); no longer J1.2, J7.2
- net PA4_STOP: now also U7.4 (C)
- net hs_ref: now also R8.2
- net mosfet switch: now also U7.1 (K)
- net hs_out_INV: now reaches U4.4
- net hs_out_INV: now also R6.2
- new net: C8.2, R8.1, U8.3 (-)
- new net: R6.1, R7.1, U8.1 (+)
- new net GATE_E2: J7.1, R5.1, U7.5 (D)
- no-connect marks 56 -> 57
Other:
- note added: "comparator"
- note removed: "op-amp"
