File: 1-23-26/UIBoard PHONE&DONLD.kicad_pcb (KiCad board)
At the start: 2 copper layers, 285.5 x 122.3 mm, 100 parts, among them J3 430450200, J4 430450200, J5 M22-7130442, J7 22035035, Q1 2N3904, Q2 2N3904, Q3 2N3904, Q4 2N3904, SW1 A8L-11-12N1, U1 UA78M05-Q1, U2 MCP2562-E-P, U3 CD4511BPWR, U4 UA78M05-Q1, U5 7 Segment Display, U6 STM32 Nucleo F446RE, U7 PCF8574AP

Commit message: made a few minor changes to layout
Routing:
- net /A: track 39.2 -> 39.9 mm
- net GND: vias 44 -> 57
