File: Front_Control_Board_Leo_Zhang/Front_Control_Board_Leo_Zhang.kicad_pcb (KiCad board)
At the start: 2 copper layers, 261 x 140 mm, 110 parts, among them J1 22035035, J10 430450200, J11 430450200, J12 430450200, J13 22035035, J14 M22-7130442, J2 Molex Micro-Fit 4 Pin, J3 430450200, J4 430450200, J5 430450200, J6 430450200, J7 22035035, J8 22035035, J9 22035035, Q1 PSMN5R2-60YL, Q2 PSMN5R2-60YL, Q3 PSMN5R2-60YL, Q4 PSMN5R2-60YL, Q5 PSMN5R2-60YL, Q6 PSMN5R2-60YL, U2 ADS1118IDGS, U3 MCP2562-E-P, U4 MCP6286T-E/OT, U5 UA78M05QDCYRG4Q1, U6 MCP6286T-E/OT, U7 MCP6286T-E/OT

Commit message: TODO: finish layout lol
Parts:
- moved U5 188.4 mm to (37.5, 136.5)
- moved C8 173.9 mm to (35.5, 142.0)
- moved C7 172.3 mm to (39.0, 142.0)
- moved J13 152.6 mm to (272.2, 128.9)
- moved J9 119.5 mm to (272.5, 69.5)
- moved J4 118.7 mm to (156.5, 30.5)
- moved J10 114.4 mm to (185.0, 30.0)
- moved J12 110.8 mm to (138.5, 31.0)
- moved J1 110.0 mm to (272.5, 29.5)
- moved J3 107.1 mm to (122.0, 30.2)
- moved J11 103.9 mm to (171.0, 30.0)
- moved R2 100.2 mm to (253.1, 30.5)
- moved J2 99.0 mm to (206.0, 30.2)
- moved J8 97.4 mm to (272.5, 49.0)
- moved R3 95.6 mm to (245.1, 31.0)
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Routing:
- added copper zone on B.Cu, net GND
Changed lines of the file:
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@@
 	(footprint "Package_DIP:DIP-8_W7.62mm"
 		(layer "F.Cu")
-		(at 212.695 55.19)
+		(at 236.88 94.88)
 		(descr "8-lead though-hole mounted DIP package, row spacing 7.62mm (300 mils)")
 		(tags "THT DIP DIL PDIP 2.54mm 7.62mm 300mil")
@@
 	(footprint "Resistor_SMD:R_0805_2012Metric"
 		(layer "F.Cu")
-		(at 173.414997 100.129998)
+		(at 245.0875 50.5)
 		(descr "Resistor SMD 0805 (2012 Metric), square (rectangular) end terminal, IPC-7351 nominal, (Body size source: IPC-SM-782 page 72, https://www.pcb-3d.com/wordpress/wp-content/uploads/ipc-sm-782a_amendment_1_and_2.pdf), generated with kicad-footprint-generator")
 		(tags "resistor")
@@
 	(footprint "SMV_Connectors:3pin_CON_22035035_MOL"
 		(layer "F.Cu")
-		(at 176 62)
+		(at 272.5 49)
 		(tags "22035035 ")
 		(property "Reference" "J8"
@@
 	(footprint "SMV_Connectors:3pin_CON_22035035_MOL"
 		(layer "F.Cu")
-		(at 138.74599 54.850002)
+		(at 272.24599 128.850002)
 		(tags "22035035 ")
 		(property "Reference" "J13"
@@
 	(footprint "Capacitor_SMD:C_0805_2012Metric"
 		(layer "F.Cu")
-		(at 187.504997 54.559998)
+		(at 39 142)
 		(descr "Capacitor SMD 0805 (2012 Metric), square (rectangular) end terminal, IPC-7351 nominal, (Body size source: IPC-SM-782 page 76, https://www.pcb-3d.com/wordpress/wp-content/uploads/ipc-sm-782a_amendment_1_and_2.pdf, https://docs.google.com/spreadsheets/d/1BsfQQcO9C6DZCsRaXUlFlo91Tg2WpOkGARC1WS5S8t0/edit?usp=sharing), generated with kicad-footprint-generator")
 		(tags "capacitor")
@@
 	(footprint "SMV_Connectors:4_pin0430450401"
 		(layer "F.Cu")
-		(at 205.5 129.18)
+		(at 206 30.18)
 		(descr "0430450401-5")
 		(tags "Connector")
@@
 	(footprint "SMV_Connectors:CONN_SD-43045-001_02_MOL"
 		(layer "F.Cu")
-		(at 113.5 141.179998)
+		(at 156.5 30.499999)
 		(tags "430450200 ")
 		(property "Reference" "J4"
@@
 	(footprint "SMV_Connectors:3pin_CON_22035035_MOL"
 		(layer "F.Cu")
-		(at 153 70.5)
+		(at 272.5 69.5)
 		(tags "22035035 ")
 		(property "Reference" "J9"
@@
 	(footprint "SMV_Connectors:3pin_CON_22035035_MOL"
 		(layer "F.Cu")
-		(at 174 78.5)
+		(at 272.5 29.5)
 		(tags "22035035 ")
 		(property "Reference" "J1"
@@
 	(footprint "SMV_Connectors:CONN_SD-43045-001_02_MOL"
 		(layer "F.Cu")
-		(at 128 129.179998)
+		(at 185 30)
 		(tags "430450200 ")
 		(property "Reference" "J10"
@@
 	(footprint "SMV_ICs:DCY4_TEX"
 		(layer "F.Cu")
-		(at 214.6886 72.38215)
+		(at 37.5 136.5)
 		(tags "UA78M05QDCYRG4Q1 ")
 		(property "Reference" "U5"
@@
 	(footprint "SMV_Connectors:CONN_SD-43045-001_02_MOL"
 		(layer "F.Cu")
-		(at 157.5 140.179998)
+		(at 138.5 31)
 		(tags "430450200 ")
 		(property "Reference" "J12"
@@
 	(footprint "SMV_Connectors:CONN_SD-43045-001_02_MOL"
 		(layer "F.Cu")
-		(at 58.5 147.679998)
+		(at 42.5 149.179998)
 		(tags "430450200 ")
 		(property "Reference" "J6"
@@
 	(footprint "Resistor_SMD:R_0805_2012Metric"
 		(layer "F.Cu")
-		(at 173.414997 94.229998)
+		(at 245.0875 31)
 		(descr "Resistor SMD 0805 (2012 Metric), square (rectangular) end terminal, IPC-7351 nominal, (Body size source: IPC-SM-782 page 72, https://www.pcb-3d.com/wordpress/wp-content/uploads/ipc-sm-782a_amendment_1_and_2.pdf), generated with kicad-footprint-generator")
 		(tags "resistor")
@@
 	(footprint "Capacitor_SMD:C_0805_2012Metric"
 		(layer "F.Cu")
-		(at 191.954997 48.539998)
+		(at 252.5 103)
 		(descr "Capacitor SMD 0805 (2012 Metric), square (rectangular) end terminal, IPC-7351 nominal, (Body size source: IPC-SM-782 page 76, https://www.pcb-3d.com/wordpress/wp-content/uploads/ipc-sm-782a_amendment_1_and_2.pdf, https://docs.google.com/spreadsheets/d/1BsfQQcO9C6DZCsRaXUlFlo91Tg2WpOkGARC1WS5S8t0/edit?usp=sharing), generated with kicad-footprint-generator")
 		(tags "capacitor")
@@
 	(footprint "SMV_Connectors:CONN_SD-43045-001_02_MOL"
 		(layer "F.Cu")
-		(at 143.5 130.179998)
+		(at 171 29.999999)
 		(tags "430450200 ")
 		(property "Reference" "J11"
@@
 	(footprint "Resistor_SMD:R_0805_2012Metric"
 		(layer "F.Cu")
-		(at 173.414997 88.329998)
+		(at 245.0875 109.5)
 		(descr "Resistor SMD 0805 (2012 Metric), square (rectangular) end terminal, IPC-7351 nominal, (Body size source: IPC-SM-782 page 72, https://www.pcb-3d.com/wordpress/wp-content/uploads/ipc-sm-782a_amendment_1_and_2.pdf), generated with kicad-footprint-generator")
 		(tags "resistor")
@@
 	(footprint "Resistor_SMD:R_0805_2012Metric"
 		(layer "F.Cu")
-		(at 177.824997 88.329998)
+		(at 243.5 71.5)
 		(descr "Resistor SMD 0805 (2012 Metric), square (rectangular) end terminal, IPC-7351 nominal, (Body size source: IPC-SM-782 page 72, https://www.pcb-3d.com/wordpress/wp-content/uploads/ipc-sm-782a_amendment_1_and_2.pdf), generated with kicad-footprint-generator")
 		(tags "resistor")
@@
 	(footprint "Resistor_SMD:R_0805_2012Metric"
 		(layer "F.Cu")
-		(at 173.414997 97.179998)
+		(at 251.4125 50)
 		(descr "Resistor SMD 0805 (2012 Metric), square (rectangular) end terminal, IPC-7351 nominal, (Body size source: IPC-SM-782 page 72, https://www.pcb-3d.com/wordpress/wp-content/uploads/ipc-sm-782a_amendment_1_and_2.pdf), generated with kicad-footprint-generator")
 		(tags "resistor")
@@
 	(footprint "SMV_Connectors:CONN_SD-43045-001_02_MOL"
 		(layer "F.Cu")
-		(at 101 135.179998)
+		(at 122 30.179998)
 		(tags "430450200 ")
 		(property "Reference" "J3"
@@
 	(footprint "Capacitor_SMD:C_0805_2012Metric"
 		(layer "F.Cu")
-		(at 191.954997 45.529998)
+		(at 252 97)
 		(descr "Capacitor SMD 0805 (2012 Metric), square (rectangular) end terminal, IPC-7351 nominal, (Body size source: IPC-SM-782 page 76, https://www.pcb-3d.com/wordpress/wp-content/uploads/ipc-sm-782a_amendment_1_and_2.pdf, https://docs.google.com/spreadsheets/d/1BsfQQcO9C6DZCsRaXUlFlo91Tg2WpOkGARC1WS5S8t0/edit?usp=sharing), generated with kicad-footprint-generator")
 		(tags "capacitor")
@@
 	(footprint "Capacitor_SMD:C_0805_2012Metric"
 		(layer "F.Cu")
-		(at 187.504997 57.569998)
+		(at 35.5 142)
 		(descr "Capacitor SMD 0805 (2012 Metric), square (rectangular) end terminal, IPC-7351 nominal, (Body size source: IPC-SM-782 page 76, https://www.pcb-3d.com/wordpress/wp-content/uploads/ipc-sm-782a_amendment_1_and_2.pdf, https://docs.google.com/spreadsheets/d/1BsfQQcO9C6DZCsRaXUlFlo91Tg2WpOkGARC1WS5S8t0/edit?usp=sharing), generated with kicad-footprint-generator")
 		(tags "capacitor")
@@
 	(footprint "Resistor_SMD:R_0805_2012Metric"
 		(layer "F.Cu")
-		(at 173.414997 91.279998)
+		(at 253.0875 30.5)
 		(descr "Resistor SMD 0805 (2012 Metric), square (rectangular) end terminal, IPC-7351 nominal, (Body size source: IPC-SM-782 page 72, https://www.pcb-3d.com/wordpress/wp-content/uploads/ipc-sm-782a_amendment_1_and_2.pdf), generated with kicad-footprint-generator")
 		(tags "resistor")
@@
 	(footprint "Resistor_SMD:R_0805_2012Metric"
 		(layer "F.Cu")
-		(at 173.414997 103.079998)
+		(at 250 71.5)
 		(descr "Resistor SMD 0805 (2012 Metric), square (rectangular) end terminal, IPC-7351 nominal, (Body size source: IPC-SM-782 page 72, https://www.pcb-3d.com/wordpress/wp-content/uploads/ipc-sm-782a_amendment_1_and_2.pdf), generated with kicad-footprint-generator")
 		(tags "resistor")
@@
 	(footprint "SMV_Connectors:CONN_SD-43045-001_02_MOL"
 		(layer "F.Cu")
-		(at 47.5 147.679998)
+		(at 29.5 149.179998)
 		(tags "430450200 ")
 		(property "Reference" "J5"
@@
 	(footprint "SMV_Connectors:3pin_CON_22035035_MOL"
 		(layer "F.Cu")
-		(at 201 78)
+		(at 273.5 100)
 		(tags "22035035 ")
 		(property "Reference" "J7"
@@
 		(layer "Edge.Cuts")
 	)
+	(zone
+		(net 1)
+		(net_name "GND")
+		(layer "B.Cu")
+		(hatch edge 0.5)
+		(connect_pads
+			(clearance 0.5)
+		)
+		(min_thickness 0.25)
+		(filled_areas_thickness no)
+		(fill yes
+			(thermal_gap 0.5)
+			(thermal_bridge_width 0.5)
+		)
+		(polygon
+			(pts
+				(xy 23 23.5) (xy 23 159.5) (xy 280 160) (xy 279 23)
+			)
+		)
+	)
 	(embedded_fonts no)

Commit message: placements should be good? 12V corner, 5v corner, analog side, CAN bottom. Get confirmation and start tracing
Parts:
- TP17: value Pressure -> Accelerator
- TP7: value Pressure -> Brake
- moved J6 257.2 mm to (268.5, 26.4)
- moved J1 240.6 mm to (34.1, 62.2), turned to 90 degrees
- moved J8 240.4 mm to (34.1, 80.2), turned to 90 degrees
- moved J9 240.2 mm to (34.0, 98.0), turned to 90 degrees
- moved R2 180.1 mm to (75.0, 57.8)
- moved R3 180.1 mm to (67.0, 58.3)
- moved R4 180.1 mm to (73.4, 77.3)
- moved R5 180.1 mm to (67.0, 77.8)
- moved R6 180.1 mm to (71.9, 98.8)
- moved R7 180.1 mm to (65.4, 98.8)
- moved TP1 164.5 mm to (34.9, 30.9)
- moved U7 152.4 mm to (54.6, 98.7)
- moved U4 151.6 mm to (56.6, 63.7)
- moved U6 150.7 mm to (56.6, 77.7)
- moved TP33 149.8 mm to (51.1, 75.2)
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Connections:
- U1 pad 1: unconnected-(U1-CN7_1-Pad1) -> /SPI1_SCLK
- U1 pad 2: unconnected-(U1-CN7_2-Pad2) -> /SPI1_MISO
- U1 pad 3: unconnected-(U1-CN7_3-Pad3) -> /SPI1_MOSI
- U1 pad 32: /SPI1_CS -> unconnected-(U1-PA4-Pad32)
- U1 pad 4: unconnected-(U1-CN7_4-Pad4) -> /SPI1_CS
- U1 pad 40: unconnected-(U1-CN10_2-Pad40) -> /PA8_D7_Standby
- U1 pad 49: /SPI1_SCLK -> unconnected-(U1-PA5-Pad49)
- U1 pad 51: /SPI1_MISO -> /Horn/STM32
- U1 pad 53: /SPI1_MOSI -> /HLL/STM32
- U1 pad 55: unconnected-(U1-CN10_17-Pad55) -> /HLR/STM32
- U1 pad 57: unconnected-(U1-CN10_19-Pad57) -> /BlinkRight/STM32
- U1 pad 59: unconnected-(U1-CN10_21-Pad59) -> /BlinkLeft/STM32
- U1 pad 61: /PA8_D7_Standby -> unconnected-(U1-PA8-Pad61)
Other:
- board size 261 x 140 mm -> 265.5 x 158 mm
- board text added: "ADC"
- board text added: "BlinkL"
- board text added: "BlinkR"
- board text added: "CANbus"
- board text added: "HLL"
- board text added: "HLR"
- board text added: "Horn"
- board text added: "Power (12V)"
- board text added: "Wiper"

Commit message: layout confirmed, just need to draw traces and pour
Parts:
- removed D2, D3: PTVS12VZ1USK, Diode_SMD:Nexperia_DSN1608-2_1.6x0.8mm
- added TP37: Horn, TestPoint:TestPoint_Pad_D1.0mm, F.Cu at (242.0, 66.5)
- added TP38: HLL, TestPoint:TestPoint_Pad_D1.0mm, F.Cu at (242.0, 69.5)
- added TP39: HLR, TestPoint:TestPoint_Pad_D1.0mm, F.Cu at (242.0, 72.6)
- added TP40: BlinkRight, TestPoint:TestPoint_Pad_D1.0mm, F.Cu at (242.0, 75.6)
- added TP41: BlinkLeft, TestPoint:TestPoint_Pad_D1.0mm, F.Cu at (242.0, 78.7)
- moved TP1 164.9 mm to (199.5, 21.0)
- moved J9 120.5 mm to (152.3, 121.1), turned to 180 degrees
- moved TP4 114.9 mm to (268.5, 41.2), turned to -90 degrees
- moved J3 113.4 mm to (274.0, 37.9), turned to 180 degrees
- moved D1 108.3 mm to (269.0, 35.8), turned to -90 degrees
- moved TP12 108.2 mm to (261.5, 32.7), turned to -90 degrees
- moved TP34 106.3 mm to (156.4, 92.0)
- moved R8 105.8 mm to (264.5, 32.7)
- moved TP33 105.3 mm to (156.1, 83.1)
- moved C14 102.4 mm to (156.2, 88.8), turned to -90 degrees
- moved R9 102.3 mm to (259.0, 35.2)
- moved Q1 102.2 mm to (263.6, 38.1), turned to -90 degrees
- moved TP10 101.8 mm to (268.5, 56.4), turned to -90 degrees
- moved C13 100.8 mm to (156.1, 80.1), turned to -90 degrees
- moved U3 100.5 mm to (205.6, 116.3), turned to -90 degrees
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Connections:
- J14 pad A3: /CAN_TX -> unconnected-(J14-PadA3)
- J14 pad A4: /CAN_RX -> unconnected-(J14-PadA4)
Routing:
- net Net-(Q1-G): track 0.00 -> 6.41 mm
- net GND: track 0.00 -> 4.94 mm, vias 0 -> 1
- added copper zone on F.Cu, net Net-(D1-A)
Other:
- board text removed: "ADC"
- board text removed: "Power (12V)"

Commit message: 12v pours done, finalize placements of some subsystems and then run traces, also place all my vias
Parts:
- added J15: M22-7130442, SMV_Connectors:M22-7130442_TYC, F.Cu at (241.4, 62.5)
- J14: footprint Jumperz:M22-7130442_TYC -> SMV_Connectors:M22-7130442_TYC
- moved J1 41.2 mm to (142.0, 134.5), turned to 180 degrees
- moved J8 36.8 mm to (156.0, 134.5), turned to 180 degrees
- moved R2 30.8 mm to (144.8, 127.6), turned to -90 degrees
- moved R5 28.9 mm to (158.8, 127.6), turned to 90 degrees
- moved R3 25.7 mm to (145.8, 124.1), turned to 0 degrees
- moved R4 25.2 mm to (159.8, 124.1), turned to 0 degrees
- moved TP6 22.4 mm to (144.8, 121.1), turned to 90 degrees
- moved J9 22.2 mm to (170.0, 134.5)
- moved R6 22.2 mm to (173.5, 125.0)
- moved R7 22.2 mm to (172.5, 128.0)
- moved TP17 22.2 mm to (172.5, 122.0)
- moved TP7 20.3 mm to (158.8, 120.6), turned to 90 degrees
- moved TP34 19.0 mm to (157.0, 73.0), turned to 180 degrees
- moved U7 18.6 mm to (160.5, 74.0), turned to 180 degrees
- moved TP5 18.6 mm to (149.5, 83.0), turned to 180 degrees
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Routing:
- net Net-(D5-A): track 0.00 -> 6.92 mm
- net Net-(Q1-G): track 6.41 -> 0.24 mm
- net Net-(Q2-D): track 0.00 -> 4.98 mm
- net Net-(D4-A): track 0.00 -> 4.87 mm
- net Net-(D6-A): track 0.00 -> 4.84 mm
- net Net-(Q3-D): track 0.00 -> 4.50 mm
- net GND: track 4.94 -> 0.94 mm, vias 1 -> 11
- net Net-(D1-A): track 0.00 -> 1.15 mm
- net Net-(Q4-G): track 0.00 -> 0.86 mm
- net Net-(Q6-G): track 0.00 -> 0.75 mm
- net Net-(Q2-G): track 0.00 -> 0.55 mm
- added copper zone on F.Cu, net +12V
- removed copper zone on F.Cu, net Net-(D1-A)

Commit message: vias placed?
Parts:
- moved J9 55.3 mm to (117.0, 118.6), turned to 90 degrees
- moved J1 50.5 mm to (117.0, 90.6), turned to 90 degrees
- moved R7 49.4 mm to (123.5, 121.1), turned to 0 degrees
- moved J8 49.1 mm to (117.0, 104.6), turned to 90 degrees
- moved R6 47.1 mm to (126.5, 122.1), turned to -90 degrees
- moved TP17 43.0 mm to (129.5, 121.1), turned to 0 degrees
- moved R5 40.3 mm to (123.9, 107.4), turned to 0 degrees
- moved R2 40.1 mm to (123.9, 93.4), turned to 180 degrees
- moved R4 36.0 mm to (127.4, 108.4), turned to -90 degrees
- moved R3 35.0 mm to (127.4, 94.4), turned to -90 degrees
- moved TP6 31.3 mm to (130.4, 93.4), turned to 0 degrees
- moved TP7 30.9 mm to (130.9, 107.4), turned to 0 degrees
- moved C14 25.5 mm to (131.7, 76.6)
- moved U7 25.1 mm to (135.4, 74.6)
- moved C1 24.5 mm to (147.7, 74.6)
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Routing:
- net GND: vias 11 -> 25
- added copper zone on F.Cu, net +5V

Commit message: Made edits before Edwin made his edits: replaced CANTran footprint, rerouted jumper for RX/TX, added LED for 3v3
Parts:
- removed J14: M22-7130442, SMV_Connectors:M22-7130442_TYC
- removed TP41: BlinkLeft, TestPoint:TestPoint_Pad_D1.0mm
- added LED1: LTST-C170GKT, SMV_Passives:LED_LTST-C170GKT_LTO, F.Cu at (199.0, 113.5)
- added LED2: LTST-C170GKT, SMV_Passives:LED_LTST-C170GKT_LTO, F.Cu at (170.5, 34.5)
- added LED3: LTST-C170GKT, SMV_Passives:LED_LTST-C170GKT_LTO, F.Cu at (170.6, 72.8)
- added R31: 200, Resistor_SMD:R_0805_2012Metric, F.Cu at (198.0, 110.0)
- added R32: 1K, Resistor_SMD:R_0805_2012Metric, F.Cu at (173.6, 37.0)
- added R33: 100, Resistor_SMD:R_0805_2012Metric, F.Cu at (170.6, 76.8)
- J15: footprint SMV_Connectors:M22-7130442_TYC -> Jumperz:M22-7130442_TYC
- TP1: value TestPoint -> BlinkLSig
- TP16: value BlinkR_MOS_G -> BlinkL_MOS_G
- TP37: value Horn -> BlinkRSig
- TP38: value HLL -> HLRSig
- TP39: value HLR -> HLLSig
- TP40: value BlinkRight -> HornSig
- U3: footprint Package_DIP:DIP-8_W7.62mm -> SMV_ICs:SOIC127P600X175-8N
- moved TP22 117.5 mm to (161.2, 86.6)
- moved J6 78.5 mm to (273.8, 105.4), turned to 0 degrees
- moved TP1 76.5 mm to (249.6, 78.8), turned to 180 degrees
- moved J1 66.4 mm to (179.5, 113.0), turned to 180 degrees
- moved R2 59.5 mm to (182.0, 106.3), turned to -90 degrees
- moved R3 56.2 mm to (183.0, 102.7), turned to 0 degrees
- moved TP6 55.0 mm to (184.0, 105.5), turned to 90 degrees
- moved J5 51.8 mm to (153.5, 27.3), turned to 180 degrees
- moved TP2 50.2 mm to (167.0, 35.0), turned to 0 degrees
- moved J8 49.2 mm to (165.5, 113.0), turned to 180 degrees
- moved C7 47.5 mm to (164.5, 36.5), turned to 90 degrees
- moved U5 44.8 mm to (159.0, 38.0), turned to 90 degrees
- moved R5 44.4 mm to (168.3, 106.1), turned to -90 degrees
- moved C8 42.6 mm to (164.5, 40.0), turned to 90 degrees
- moved C12 42.5 mm to (169.0, 39.8), turned to 180 degrees
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Connections:
- J15 pad 1: /CAN_TX -> unconnected-(J15-A1-Pad1)
- J15 pad 3: unconnected-(J15-A3-Pad3) -> /CAN_RX
- J15 pad 4: /CAN_RX -> /CAN_TX
- TP1 pad 1: unconnected-(TP1-Pad1) -> /BlinkLeft/STM32
- TP37 pad 1: /Horn/STM32 -> /BlinkRight/STM32
- TP38 pad 1: /HLL/STM32 -> /HLR/STM32
- TP39 pad 1: /HLR/STM32 -> /HLL/STM32
- TP40 pad 1: /BlinkRight/STM32 -> /Horn/STM32
- U1 pad 40: /PA8_D7_Standby -> unconnected-(U1-PC8-Pad40)
- U1 pad 41: /CAN_RX -> unconnected-(U1-PB8-Pad41)
- U1 pad 43: /CAN_TX -> unconnected-(U1-PB9-Pad43)
- U1 pad 67: unconnected-(U1-PB5-Pad67) -> /CAN_RX
- U1 pad 68: unconnected-(U1-PB13-Pad68) -> /CAN_TX
- U1 pad 71: unconnected-(U1-PA10-Pad71) -> /PA8_D7_Standby
- U3 pad 1: /CAN_TX/Jump -> /CAN_TX
- U3 pad 4: /CAN_RX/Jump -> /CAN_RX
Routing:
- net +3V3: track 0.00 -> 183.0 mm
- net /Pressure/VFin: track 0.00 -> 124.0 mm
- net /Brake(Hall)/VFin: track 0.00 -> 91.3 mm
- net GND: track 0.94 -> 83.3 mm, vias 25 -> 126
- net /Accelerator(Hall)/VFin: track 0.00 -> 60.7 mm
- net +5V: track 0.00 -> 52.8 mm
- net /CANL: track 0.00 -> 41.9 mm
- net /CAN_RX: track 0.00 -> 41.9 mm
- net /Horn/STM32: track 0.00 -> 39.9 mm
- net /CANH: track 0.00 -> 36.6 mm
- net /CAN_TX: track 0.00 -> 34.6 mm
- net /HLL/STM32: track 0.00 -> 32.5 mm
- net /Brake(Hall)/VFout: track 0.00 -> 30.9 mm
- net /Accelerator(Hall)/VFout: track 0.00 -> 29.8 mm
- net /SPI1_MISO: track 0.00 -> 27.5 mm
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- added copper zone on F.Cu, net GND
Other:
- board size 265.5 x 158 mm -> 135 x 102.5 mm
- board text removed: "CANbus"

Commit message: readded minor changes
Parts:
- LED1, LED2, LED3: footprint SMV_Passives:LED_LTST-C170GKT_LTO -> Personal:LED_LTST-C170GKT_LTO
- moved TP35 2.10 mm to (221.5, 111.5)
- moved TP39 0.46 mm to (248.9, 60.5)
- moved TP36 0.11 mm to (223.7, 115.5)
Connections:
- net /CANH renamed /CAN_P
- net /CANL renamed /CAN_N
Routing:
- net /CAN_P: track 36.6 -> 44.6 mm
- net GND: track 83.3 -> 88.0 mm, vias 126 -> 128
- net /CAN_N: track 41.9 -> 44.2 mm
- net /SPI1_MOSI: track 20.7 -> 21.2 mm
