File: Front_Control_Board_Leo_Zhang/_autosave-Front_Control_Board_Leo_Zhang.kicad_pcb (KiCad board)
At the start: 2 copper layers, 142.8 x 132 mm, 127 parts, among them J1 22035035, J10 430450200, J11 430450200, J12 430450200, J13 22035035, J15 M22-7130442, J16 XT60-M, J2 Molex Micro-Fit 4 Pin, J3 XT60-M, J4 430450200, J5 430450200, J6 430450200, J7 22035035, J8 22035035, J9 22035035, Q1 PSMN1R8-40YLC_115, Q2 PSMN1R8-40YLC_115, Q3 PSMN1R8-40YLC_115, Q4 PSMN1R8-40YLC_115, Q5 PSMN1R8-40YLC_115, Q6 PSMN1R8-40YLC_115, U2 ADS1118IDGS, U3 MCP2562-E-P, U4 MCP6286T-E/OT, U5 UA78M05QDCYRG4Q1, U6 MCP6286T-E/OT, U7 MCP6286T-E/OT, U8 J115F11AH12VDCS61.5U

Commit message: Done! Serg Ed have looked at relay circ
Parts:
- moved D7 5.69 mm to (209.9, 45.0)
- moved TP4 2.41 mm to (222.6, 48.8)
- moved C14 0.35 mm to (105.6, 61.8)
Routing:
- net +5V: track 69.9 -> 63.6 mm
- net GND: vias 148 -> 160
Changed lines of the file:
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@@
 	(footprint "SMV_Passives:DO-41_DIO"
 		(layer "F.Cu")
-		(at 215.6 45)
+		(at 209.9105 44.995376)
 		(tags "SB1100-T ")
 		(property "Reference" "D7"
@@
 	(footprint "SMV_Misc:ValueTestPoint_Pad_D1.0mm"
 		(layer "F.Cu")
-		(at 224.2 50.6 -90)
+		(at 222.6 48.8 -90)
 		(descr "SMD pad as test Point, diameter 1.0mm")
 		(tags "test point SMD pad")
@@
 	(footprint "Capacitor_SMD:C_0805_2012Metric"
 		(layer "F.Cu")
-		(at 105.25 61.75)
+		(at 105.6 61.8)
 		(descr "Capacitor SMD 0805 (2012 Metric), square (rectangular) end terminal, IPC-7351 nominal, (Body size source: IPC-SM-782 page 76, https://www.pcb-3d.com/wordpress/wp-content/uploads/ipc-sm-782a_amendment_1_and_2.pdf, https://docs.google.com/spreadsheets/d/1BsfQQcO9C6DZCsRaXUlFlo91Tg2WpOkGARC1WS5S8t0/edit?usp=sharing), generated with kicad-footprint-generator")
 		(tags "capacitor")
@@
 	(footprint "SMV_ICs:SOT-23-5_MC_MCH"
 		(layer "F.Cu")
-		(at 107.5 65.754801 90)
+		(at 107.500001 65.754801 90)
 		(tags "MCP6286T-E/OT ")
 		(property "Reference" "U7"
@@
 	(gr_poly
 		(pts
+			(xy 219.2 33.8) (xy 222.8 33.8) (xy 222.8 52.2) (xy 217.8 52.2) (xy 217.8 47.8) (xy 219.2 47.8)
+		)
+		(stroke
+			(width 0.2)
+			(type solid)
+		)
+		(fill yes)
+		(layer "F.Cu")
+		(net 102)
+	)
+	(gr_poly
+		(pts
 			(xy 227.191866 109.6) (xy 227.191866 113.6) (xy 221.191866 113.6) (xy 221.191866 115.6) (xy 229.691866 115.6)
 			(xy 229.691866 109.6)
@@
 		(net 107)
 	)
-	(gr_poly
-		(pts
-			(xy 219.372905 34.448653) (xy 217.8 52.2) (xy 223.8 52.2) (xy 228.946556 43.920757) (xy 222.436843 34.268421)
-		)
-		(stroke
-			(width 0.2)
-			(type solid)
-		)
-		(fill yes)
-		(layer "F.Cu")
-		(net 102)
-	)
 	(gr_rect
 		(start 225.2 95.4)
@@
 	)
 	(via
+		(at 208 111.4)
+		(size 0.6)
+		(drill 0.3)
+		(layers "F.Cu" "B.Cu")
+		(free yes)
+		(net 1)
+	)
+	(via
 		(at 200.5 98)
 		(size 0.6)
@@
 	)
 	(via
+		(at 118.8 47.4)
+		(size 0.6)
+		(drill 0.3)
+		(layers "F.Cu" "B.Cu")
+		(free yes)
+		(net 1)
+	)
+	(via
 		(at 128.5 118)
 		(size 0.6)
@@
 	)
 	(via
+		(at 217.4 60)
+		(size 0.6)
+		(drill 0.3)
+		(layers "F.Cu" "B.Cu")
+		(free yes)
+		(net 1)
+	)
+	(via
 		(at 200.4 51.2)
 		(size 0.6)
@@
 	)
 	(via
+		(at 206.4 113.4)
+		(size 0.6)
+		(drill 0.3)
+		(layers "F.Cu" "B.Cu")
+		(free yes)
+		(net 1)
+	)
+	(via
 		(at 207.2 82.8)
 		(size 0.6)
@@
 	)
 	(via
+		(at 118.8 48.4)
+		(size 0.6)
+		(drill 0.3)
+		(layers "F.Cu" "B.Cu")
+		(free yes)
+		(net 1)
+	)
+	(via
 		(at 208.8 103)
 		(size 0.6)
@@
 	)
 	(via
+		(at 123.4 52.2)
+		(size 0.6)
+		(drill 0.3)
+		(layers "F.Cu" "B.Cu")
+		(free yes)
+		(net 1)
+	)
+	(via
 		(at 177.4 58.8)
 		(size 0.6)
@@
 	)
 	(via
+		(at 215.2 110.2)
+		(size 0.6)
+		(drill 0.3)
+		(layers "F.Cu" "B.Cu")
+		(free yes)
+		(net 1)
+	)
+	(via
 		(at 132.75 66.25)
 		(size 0.6)
@@
 	)
 	(via
+		(at 127.2 52.4)
+		(size 0.6)
+		(drill 0.3)
+		(layers "F.Cu" "B.Cu")
+		(free yes)
+		(net 1)
+	)
+	(via
 		(at 167 75)
 		(size 0.6)
@@
 	)
 	(via
+		(at 125 56.2)
+		(size 0.6)
+		(drill 0.3)
+		(layers "F.Cu" "B.Cu")
+		(free yes)
+		(net 1)
+	)
+	(via
 		(at 146.5 127)
 		(size 0.6)
@@
 	)
 	(via
+		(at 217.4 83.4)
+		(size 0.6)
+		(drill 0.3)
+		(layers "F.Cu" "B.Cu")
+		(free yes)
+		(net 1)
+	)
+	(via
 		(at 135.8 51.8)
 		(size 0.6)
@@
 	)
 	(via
+		(at 217.2 96.2)
+		(size 0.6)
+		(drill 0.3)
+		(layers "F.Cu" "B.Cu")
+		(free yes)
+		(net 1)
+	)
+	(via
 		(at 210 70.6)
 		(size 0.6)
@@
 	)
 	(via
+		(at 217 71.4)
+		(size 0.6)
+		(drill 0.3)
+		(layers "F.Cu" "B.Cu")
+		(free yes)
+		(net 1)
+	)
+	(via
 		(at 116.099999 78.450001)
 		(size 0.6)
@@
 	)
 	(segment
-		(start 119.599998 58.199998)
-		(end 119.599998 64.459602)
-		(width 1)
-		(layer "F.Cu")
-		(net 6)
-	)
-	(segment
 		(start 186.165 128.55)
 		(end 186.165 126.315)
@@
 	)
 	(segment
-		(start 132.75 76)
-		(end 131.712448 76)
+		(start 135.9 71.24)
+		(end 135.9 72.541552)
 		(width 0.2)
 		(layer "F.Cu")
@@
 	)
 	(segment
-		(start 135.9 72.541552)
-		(end 134.891552 73.55)
+		(start 134.4 69.74)
+		(end 135.9 71.24)
 		(width 0.2)
 		(layer "F.Cu")
@@
 	)
 	(segment
-		(start 134.4 69.74)
-		(end 135.9 71.24)
+		(start 133.15 75.6)
+		(end 132.75 76)
 		(width 0.2)
 		(layer "F.Cu")
@@
 	)
 	(segment
-		(start 126 85.237498)
-		(end 121.512499 89.724999)
+		(start 132.75 76)
+		(end 131.712448 76)
 		(width 0.2)
 		(layer "F.Cu")
@@
 	)
 	(segment
-		(start 131.712448 76)
-		(end 126 81.712448)
+		(start 126.8 84.437498)
+		(end 121.512499 89.724999)
 		(width 0.2)
 		(layer "F.Cu")
@@
 	)
 	(segment
-		(start 133.15 74.35)
-		(end 133.15 75.6)
+		(start 134.891552 73.55)
+		(end 133.95 73.55)
 		(width 0.2)
 		(layer "F.Cu")
@@
 	)
 	(segment
-		(start 135.9 71.24)
-		(end 135.9 72.541552)
+		(start 133.95 73.55)
+		(end 133.15 74.35)
 		(width 0.2)
 		(layer "F.Cu")
@@
 	)
 	(segment
-		(start 133.95 73.55)
-		(end 133.15 74.35)
+		(start 135.9 72.541552)
+		(end 134.891552 73.55)
 		(width 0.2)
 		(layer "F.Cu")
@@
 	)
 	(segment
-		(start 134.891552 73.55)
-		(end 133.95 73.55)
+		(start 131.712448 76)
+		(end 126.8 80.912448)
 		(width 0.2)
 		(layer "F.Cu")
@@
 	)
 	(segment
-		(start 133.15 75.6)
-		(end 132.75 76)
+		(start 126.8 80.912448)
+		(end 126.8 84.437498)
 		(width 0.2)
 		(layer "F.Cu")
@@
 	)
 	(segment
-		(start 126 81.712448)
-		(end 126 85.237498)
+		(start 133.15 74.35)
+		(end 133.15 75.6)
 		(width 0.2)
 		(layer "F.Cu")
@@
 		(priority 9)
 		(connect_pads
-			(clearance 0.5)
+			(clearance 0.3)
 		)
 		(min_thickness 0.25)
