File: SafetySchematicChenR/Safety Schematic.kicad_sch (KiCad schematic)
At the start: 68 parts, among them J1 XT60-M, J2 430450200, J3 Conn_01x04_Pin, J4 22035035, J6 430450200, J7 XT60-M, Q1 IRLML6344TRPBF, U1 74AHC1G32, U10 74LVC1GU04DRL, U12 MCP6286T-E/OT, U14 J115F11AH12VDCS61.5U, U15 MCP2562-E-P, U2 74LVC1GU04DRL, U3 LT1962-3, U4 MAX603, U5 LT1962-3.3, U7 74LS279, U8 74LVC1GU04DRL

Commit message: gurt
Parts:
- removed D5: 7.5V, Diode_SMD:D_MiniMELF, symbol Diode:BZV55C7V5
- removed J3: Conn_01x04_Pin, symbol Connector:Conn_01x04_Pin
- added C13, C14: 0.1 uF, symbol Device:C_Small
- added C15: 0.01 uF, symbol Device:C_Small
- added D5: 5V, symbol Device:D_Zener_Small
- added J5: Molex Micro-Fit 4 Pin, SMV_Connectors:4_pin0430450401, symbol SMV_Custom:Molex Micro-Fit 4 Pin
- added R1, R3, R7: 0.1k ohms, symbol Device:R_Small
- added R15, R4: 1.2k ohms, symbol Device:R_Small
- added RV1: 100 ohms, symbol Device:R_Potentiometer
- added TP12, TP24: TestPoint, symbol Connector:TestPoint
- added U11: LT1962-1.5, Package_SO:MSOP-8_3x3mm_P0.65mm, symbol Regulator_Linear:LT1962-1.5
- added U6: MCP6286T-E/OT, SOT-23-5_MC_MCH, symbol SMV_Custom:MCP6286T-E_OT
- R9: value 100,000k ohms -> 68k Ohms
Connections:
- net +3V0: now also C13.2, J5.1, R4.1; no longer C8.2
- net +3V3: now also C8.1, U9.16 (+3V3), U11.5 (~{SHDN}), U11.8 (IN), U6.5 (VDD)
- net GND: now also C8.2, C13.1, C14.2, J5.4, R1.1, R15.2, R3.1, R7.1, U11.4 (GND), U6.2 (VSS); no longer C8.1
- net HSENSOR: now also J5.2, R3.2, TP12.1, U6.3 (VIN+); no longer TP4.1, U12.3 (VIN+)
- net OPAMPOUT: now also D5.2 (A)
- net at R14.1, R9.2, TP11.1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: now also D5.1 (K)
- net HSENSEBASEDIF: now reaches U9.49 (PA5)
- net HDIF: now reaches U9.51 (PA6)
- net HDIF: now also U6.1 (VOUT)
- new net: C15.2, U11.3 (BYP)
- new net: R15.1, RV1.1
- new net: R4.2, RV1.3
- new net +1V5: C14.1, C15.1, TP24.1, TP4.1, U11.1 (OUT), U11.2 (SENSE)
- new net ADJHDIF: R1.2, U12.3 (VIN+)
- new net POTENTIOMETER: R7.2, RV1.2, U6.4 (VIN-)
- no-connect marks 55 -> 53
Other:
- moved on the sheet: C1, C2, J2, J4, R10, R2, TP18, TP19, TP5, TP7, TP8, U15

Commit message: gurt
Parts:
- removed C14, C8: 0.1 uF, symbol Device:C_Small
- removed C15: 0.01 uF, symbol Device:C_Small
- removed R1, R8: 0.1k ohms, symbol Device:R_Small
- removed R14: 10k ohms, symbol Device:R_Small
- removed R9: 68k Ohms, symbol Device:R_Small
- removed TP11, TP24, TP4: TestPoint, symbol Connector:TestPoint
- removed U11: LT1962-1.5, Package_SO:MSOP-8_3x3mm_P0.65mm, symbol Regulator_Linear:LT1962-1.5
- removed U12: MCP6286T-E/OT, SOT-23-5_MC_MCH, symbol SMV_Custom:MCP6286T-E_OT
- added R16, R17: 0.1k ohms, symbol Device:R_Small
- R3, R7: value 0.1k ohms -> 68k ohms
Connections:
- net GND: no longer R3.1
- net HDIF: now also D5.1 (K), R3.1; no longer U9.51 (PA6)
- net HSENSOR: now also R17.1; no longer R3.2, U6.3 (VIN+)
- net POTENTIOMETER: now also TP3.1, R16.1; no longer R7.2, U6.4 (VIN-)
- net HSENSEBASEDIF: no longer names the net of U9.49 (PA5)
- new net: R16.2, R7.2, U6.3 (VIN+)
- new net: R17.2, R3.2, U6.4 (VIN-)
- no-connect marks 53 -> 56
Other:
- moved on the sheet: D5, R3, R7, U6

Commit message: changes
Parts:
- removed C10, C11, C3, C5, C6: 0.1 uF, symbol Device:C_Small
- removed C12, C7: 0.01 uF, symbol Device:C_Small
- removed C9: 0.33 uF, symbol Device:C_Small
- removed R13: 5k ohms, symbol Device:R_Small
- removed R2: 10k ohms, symbol Device:R_Small
- removed TP13, TP14, TP2, TP20, TP21, TP22, TP6, TP9: TestPoint, symbol Connector:TestPoint
- removed U1: 74AHC1G32, symbol 74xGxx:74AHC1G32
- removed U3: LT1962-3, Package_SO:MSOP-8_3x3mm_P0.65mm, symbol Regulator_Linear:LT1962-3
- removed U4: MAX603, symbol Regulator_Linear:MAX603
- removed U5: LT1962-3.3, Package_SO:MSOP-8_3x3mm_P0.65mm, symbol Regulator_Linear:LT1962-3.3
- removed U7: 74LS279, symbol 74xx:74LS279
- removed U8: 74LVC1GU04DRL, Package_TO_SOT_SMD:SOT-553, symbol 74xGxx:74LVC1GU04DRL
- added D10, D8, D9: LED, LED_SMD:LED-APA102-2020, symbol Device:LED
- added R1: 5k ohms, Resistor_SMD:R_0603_1608Metric_Pad0.98x0.95mm_HandSolder, symbol Device:R_Small
- added U1: CD4043BPWR, SMV_ICs:PW16, symbol SMV_Custom:CD4043BPWR
- added U7, U8: 74AHC1G32, symbol 74xGxx:74AHC1G32
- C1, C13, C2, C4: footprint (none) -> Capacitor_SMD:C_0805_2012Metric_Pad1.18x1.45mm_HandSolder
- D1, D2, D3: footprint (none) -> LED_SMD:LED_0805_2012Metric_Pad1.15x1.40mm_HandSolder
- D5: footprint (none) -> Diode_SMD:D_MiniMELF
- Q1: footprint IRLML6344TRPBF:TRANS_IRLML6344TRPBF -> SMV_ICs:TRANS_IRLML6344TRPBF
- R10, R11, R12, R15, R16, R17, R3, R4, R5, R6, R7, RV1: footprint (none) -> Resistor_SMD:R_0603_1608Metric_Pad0.98x0.95mm_HandSolder
- TP1, TP10, TP12, TP15, TP16, TP17, TP18, TP19, TP23, TP3, TP5, TP7, TP8: footprint (none) -> TestPoint:TestPoint_Pad_D1.0mm
- U14: footprint SMV_ICs:J115F11AH12VDCS615U -> SMV_Passives:J115F11AH12VDCS615U
- U6: footprint SOT-23-5_MC_MCH -> SMV_ICs:SOT-23-5_MC_MCH
Connections:
- net +12V: now also U6.5 (VDD)
- net +3V3: no longer U6.5 (VDD)
- net +5V: now also U1.16 (VDD), U1.5 (ENABLE), U7.5 (VCC), U8.5 (VCC)
- net EXTESTOP: now also J2.1
- net GND: now also R1.2, U1.8 (VSS), U7.3 (GND), U8.3 (GND)
- net OPAMPOUT: no longer U2.2
- net RESET: now also R1.1, U1.12 (S3), U1.14 (S4), U1.6 (S2)
- net at D1.1 (K), R12.1: now also U1.7 (R2)
- net at D3.2 (A): now also U10.4
- net at U2.4: now also U1.11 (R3)
- net at D2.1 (K), R6.1: now also U2.2; no longer U10.2
- new net: U1.1 (Q4), U7.1
- new net: U7.4, U8.1
- new net: D10.1 (K), D8.1 (K), D9.1 (K), U1.15 (R4)
- new net: U10.2, U8.4
- new net EXTESTOPSR: U1.9 (Q2), U8.2
- new net HSENSE2: D9.2 (A)
- new net HSENSE3: D10.2 (A)
- new net INTESTOPSR: U1.10 (Q3), U7.2
- new net OPAMPLDO: D8.2 (A)
- no-connect marks 56 -> 58
Other:
- added sheet Hydrogen Sensors (hydrogenSensors.kicad_sch)
- added sheet LDOs (LDOs.kicad_sch)
- moved on the sheet: C4, D1, D2, D3, D4, J1, J2, J7, Q1, R11, R12, R5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
